File: mtg_life_counter/mtg_life_counter.sch (KiCad schematic (older format))
At the start: 66 parts

Commit message: Get schematic more complete
Parts:
- removed R?: 1k, symbol Device:R
- removed SW? (x9): SW_Push, symbol Switch:SW_Push
- removed SW?: SW_SPDT, symbol Switch:SW_SPDT
- removed U? (x2): TPIC6595, symbol Interface_Expansion:TPIC6595
- added B10, B2, B3, B4, B5, B6, B7, B8, B9: SW_Push, symbol Switch:SW_Push
- added C1, C2, C3, C4: 0.1uF, symbol Device:C_Small
- added R33: R, symbol Device:R
- added R34: 10k, symbol Device:R
- added SW1: SW_SPST, symbol Switch:SW_SPST
- added U3: TLC5916, symbol Driver_LED:STP08CP05
- added U4: TPIC6595, symbol Interface_Expansion:TPIC6595
- C5, C6, C7: renamed from C?; value C_Small -> 0.1uF
- gave numbers to parts that had none: 50
Connections:
- net SPI_CLK is gone; now on net SER_CLK: A1.16 (D13)
- net SPI_OUT is gone; now on net SER_DATA: A1.14 (D11)
- net +5V: now also U1.10 (~SRCLR), U1.16 (VCC), U2.10 (~SRCLR), U2.16 (VCC), C1.2, C2.2, C3.2, C4.2, R34.2, U3.16 (VDD), U4.2 (VCC)
- net BTN_RB: now also A1.23 (A4)
- net GND: now also B1.2, U1.8 (GND), U2.8 (GND), B10.2, B2.2, B3.2, B4.2, B5.2, B6.2, B7.2, B8.2, B9.2, C1.1, C2.1, C3.1, C4.1, R33.2, SW1.2 (B), U3.1 (GND), U4.1 (PGND), U4.10 (PGND), U4.11 (PGND), U4.19 (LGND), U4.20 (PGND)
- net SEL_0: now also A1.24 (A5)
- net SEL_1: now also A1.25 (A6)
- net SEL_2: now also A1.26 (A7)
- net SW_RB_1: now also A1.22 (A3)
- net SW_RB_2: now also A1.21 (A2)
- net RESET_BTN: now reaches A1.10 (D7)
- net RESET_BTN: now also B1.1
- net NENABLE: now reaches A1.11 (D8)
- net NENABLE: now also U1.13 (~OE), U2.13 (~OE), U3.13 (~OE), U4.9 (~G)
- net SER_LATCH: now reaches A1.12 (D9)
- net SER_LATCH: now also U1.12 (RCLK), U2.12 (RCLK), U3.4 (LE), U4.12 (RCLK)
- net RNG_WIRE: now reaches A1.19 (A0)
- net MODE_SW: now reaches A1.20 (A1)
- net MODE_SW: now also SW1.1 (A)
- net ROLL_BTN: now reaches A1.9 (D6)
- net ROLL_BTN: now also B2.1
- net SER_CLK: now reaches U1.11 (SRCLK)
- net SER_CLK: now also U2.11 (SRCLK), U3.3 (CLK), U4.13 (SRCK)
- net SER_DATA: now reaches U1.14 (SER)
- net at U1.9 (QH'): now also U2.14 (SER)
- net at D2.14 (CC1): now also U3.9 (OUT4)
- net at D2.11 (CC2): now also U3.10 (OUT5)
- net at D2.10 (CC3): now also U3.11 (OUT6)
- net at D2.6 (CC4): now also U3.12 (OUT7)
- net at D1.14 (CC1): now also U3.5 (OUT0)
- net at D1.11 (CC2): now also U3.6 (OUT1)
- net at D1.10 (CC3): now also U3.7 (OUT2)
- net at D1.6 (CC4): now also U3.8 (OUT3)
- net at RN3.5 (R4), U7.1 (I3): now also B6.1
- net at RN3.9 (R8), U7.12 (I7): now also B10.1
- net at RN3.8 (R7), U7.13 (I6): now also B9.1
- net at RN3.7 (R6), U7.14 (I5): now also B8.1
- net at RN3.6 (R5), U7.15 (I4): now also B7.1
- net at RN3.4 (R3), U7.2 (I2): now also B5.1
- net at RN3.3 (R2), U7.3 (I1): now also B4.1
- net at RN3.2 (R1), U7.4 (I0): now also B3.1
- net at D4.14 (CC1): now also U4.14 (DRAIN4)
- net at D4.11 (CC2): now also U4.15 (DRAIN5)
- net at D4.10 (CC3): now also U4.16 (DRAIN6)
- net at D4.6 (CC4): now also U4.17 (DRAIN7)
- net at D3.14 (CC1): now also U4.4 (DRAIN0)
- net at D3.11 (CC2): now also U4.5 (DRAIN1)
- net at D3.10 (CC3): now also U4.6 (DRAIN2)
- net at D3.6 (CC4): now also U4.7 (DRAIN3)
- net SER_XTEND: now reaches U2.9 (QH')
- net SER_XTEND: now also U3.2 (SDI)
- new net: R33.1, U3.15 (R-EXT)
- new net: U3.14 (SDO), U4.3 (SER_IN)
- new net: R34.1, U4.8 (~SRCLR)
- no-connect marks 12 -> 24
Other:
- note added: "Arduino"
- note added: "Button Sense"
- note added: "Display Bank 1"
- note added: "Display Bank 2"
- note added: "Switch Sense 1"
- note added: "Switch Sense 2"
- note added: "TPIC vs TLC?\n-----------------\nTPIC\n- Needs current limiting resistors\n on all segments of all displays\n- Values will be manually adjusted\n- Each segment will have a\n constant brightness\nTLC\n- Constant current driver\n- \n- Can use special function mode to\n adjust current around the point\n set by single external resistor\n- Group 2 brightest displays on\n 1 chip, 2 dimmest on another"
- moved on the sheet: A1, B1, C5, C6, C7, D1, D2, D3, D4, R1, R10, R11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

Commit message: Complete PCB layout
Parts:
- removed C3: 0.1uF, symbol Device:C_Small
- removed U3: TLC5916, symbol Driver_LED:STP08CP05
- added C2: 0.1uF, Capacitor_THT:C_Disc_D3.0mm_W1.6mm_P2.50mm, symbol Device:C_Small
- added H1, H2, H3, H4: MountingHole_Pad, MountingHole:MountingHole_3.2mm_M3_Pad_Via, symbol Mechanical:MountingHole_Pad
- added R35: 100, Resistor_THT:R_Axial_DIN0207_L6.3mm_D2.5mm_P10.16mm_Horizontal, symbol Device:R
- added SW1: SW_SPDT, Button_Switch_THT:SW_Slide_1P2T_CK_OS102011MS2Q, symbol Switch:SW_SPDT
- added U2: TPIC6595, Package_DIP:DIP-20_W7.62mm, symbol Interface_Expansion:TPIC6595
- B1, B10, B2, B3, B4, B5, B6, B7, B8, B9: footprint (none) -> mtg_life_counter:B3F_12mm
- C1, C4, C5, C6, C7: footprint (none) -> Capacitor_THT:C_Disc_D3.0mm_W1.6mm_P2.50mm
- C3: renamed from C2; footprint (none) -> Capacitor_THT:C_Disc_D3.0mm_W1.6mm_P2.50mm
- D1, D2, D3, D4: footprint Display_7Segment:CA56-12EWA -> mtg_life_counter:KW4-56NX
- R1, R10, R11, R12, R13, R14, R15, R16, R17, R18, R19, R2, R20, R21, R22, R23, R24, R25, R26, R27, R28, R29, R3, R30, R31, R32, R34, R4, R5, R6, R7, R8, R9: footprint (none) -> Resistor_THT:R_Axial_DIN0207_L6.3mm_D2.5mm_P10.16mm_Horizontal
- R33: value R -> 10k; footprint (none) -> Resistor_THT:R_Axial_DIN0207_L6.3mm_D2.5mm_P10.16mm_Horizontal
- SW2: renamed from SW1; footprint (none) -> Button_Switch_THT:SW_Slide_1P2T_CK_OS102011MS2Q
- SW3: renamed from SW2; footprint (none) -> mtg_life_counter:CK_RM10x77
- SW4: renamed from SW3; footprint (none) -> mtg_life_counter:CK_RM10x77
- SW5: renamed from SW4; footprint (none) -> mtg_life_counter:CK_RM10x77
- SW6: renamed from SW5; footprint (none) -> mtg_life_counter:CK_RM10x77
- U1, U5, U6, U7: footprint (none) -> Package_DIP:DIP-16_W7.62mm
- U3: renamed from U2; footprint (none) -> Package_DIP:DIP-16_W7.62mm
- U4: footprint (none) -> Package_DIP:DIP-20_W7.62mm
Connections:
- net +5V: now also A1.5 (D2), R33.2, C2.2, SW1.2 (B), U2.2 (VCC); no longer A1.27 (+5V)
- net GND: now also C2.1, H1.1, H2.1, H3.1, H4.1, R35.1, U2.1 (PGND), U2.10 (PGND), U2.11 (PGND), U2.19 (LGND), U2.20 (PGND); no longer R33.2
- net NENABLE: now also U2.9 (~G)
- net SER_CLK: now also U2.13 (SRCK)
- net SER_LATCH: now also U2.12 (RCLK)
- net INT_1: now reaches A1.6 (D3)
- net SER_CASCADE_1: now reaches U1.9 (QH'), U3.14 (SER)
- net at RN1.9 (R8), U5.12 (I7): now also SW3.5; no longer SW4.5
- net at RN1.8 (R7), U5.13 (I6): now also SW3.4; no longer SW4.4
- net at RN1.7 (R6), U5.14 (I5): now also SW3.3; no longer SW4.3
- net at RN1.6 (R5), U5.15 (I4): now also SW3.2; no longer SW4.2
- net at RN2.9 (R8), U6.12 (I7): now also SW5.5; no longer SW6.5
- net at RN2.8 (R7), U6.13 (I6): now also SW5.4; no longer SW6.4
- net at RN2.7 (R6), U6.14 (I5): now also SW5.3; no longer SW6.3
- net at RN2.6 (R5), U6.15 (I4): now also SW5.2; no longer SW6.2
- net at B6.1, RN3.5 (R4): now also U7.12 (I7); no longer U7.1 (I3)
- net at B5.1, RN3.4 (R3): now also U7.13 (I6); no longer U7.2 (I2)
- net at B4.1, RN3.3 (R2): now also U7.14 (I5); no longer U7.3 (I1)
- net at B3.1, RN3.2 (R1): now also U7.15 (I4); no longer U7.4 (I0)
- net at D1.10 (CC3): now also U2.6 (DRAIN2)
- net at D1.11 (CC2): now also U2.5 (DRAIN1)
- net at D1.14 (CC1): now also U2.4 (DRAIN0)
- net at D1.6 (CC4): now also U2.7 (DRAIN3)
- net at D2.10 (CC3): now also U2.16 (DRAIN6)
- net at D2.11 (CC2): now also U2.15 (DRAIN5)
- net at D2.14 (CC1): now also U2.14 (DRAIN4)
- net at D2.6 (CC4): now also U2.17 (DRAIN7)
- net at D3.10 (CC3): now also U4.16 (DRAIN6); no longer U4.6 (DRAIN2)
- net at D3.11 (CC2): now also U4.15 (DRAIN5); no longer U4.5 (DRAIN1)
- net at D3.14 (CC1): now also U4.14 (DRAIN4); no longer U4.4 (DRAIN0)
- net at D3.6 (CC4): now also U4.17 (DRAIN7); no longer U4.7 (DRAIN3)
- net at D4.10 (CC3): now also U4.6 (DRAIN2); no longer U4.16 (DRAIN6)
- net at D4.11 (CC2): now also U4.5 (DRAIN1); no longer U4.15 (DRAIN5)
- net at D4.14 (CC1): now also U4.4 (DRAIN0); no longer U4.14 (DRAIN4)
- net at D4.6 (CC4): now also U4.7 (DRAIN3); no longer U4.17 (DRAIN7)
- net at R33.1: now also U2.8 (~SRCLR)
- net SER_CASCADE_3: now reaches U4.3 (SER_IN)
- net SER_CASCADE_3: now also U2.18 (SER_OUT)
- net SER_XTEND renamed SER_CASCADE_2
- net SER_CASCADE_2: now also U2.3 (SER_IN)
- new net: RN1.2 (R1), SW4.2, U5.1 (I3)
- new net: RN1.3 (R2), SW4.3, U5.2 (I2)
- new net: RN1.4 (R3), SW4.4, U5.3 (I1)
- new net: RN1.5 (R4), SW4.5, U5.4 (I0)
- new net: RN2.2 (R1), SW6.2, U6.1 (I3)
- new net: RN2.3 (R2), SW6.3, U6.2 (I2)
- new net: RN2.4 (R3), SW6.4, U6.3 (I1)
- new net: RN2.5 (R4), SW6.5, U6.4 (I0)
- new net: B9.1, RN3.6 (R5), U7.1 (I3)
- new net: B10.1, RN3.7 (R6), U7.2 (I2)
- new net: B8.1, RN3.8 (R7), U7.3 (I1)
- new net: B7.1, RN3.9 (R8), U7.4 (I0)
- new net 5V_SRC: A1.27 (+5V), SW1.1 (A)
- new net OFF: R35.2, SW1.3 (C)
- no-connect marks 24 -> 25
Other:
- note removed: "TPIC vs TLC?\n-----------------\nTPIC\n- Needs current limiting resistors\n on all segments of all displays\n- Values will be manually adjusted\n- Each segment will have a\n constant brightness\nTLC\n- Constant current driver\n- \n- Can use special function mode to\n adjust current around the point\n set by single external resistor\n- Group 2 brightest displays on\n 1 chip, 2 dimmest on another"
- moved on the sheet: B10, B3, B4, B5, B6, B7, B8, B9, D3, D4, R17, R18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

Commit message: Fix TPIC pinout
Parts:
- removed U2, U4: TPIC6595, Package_DIP:DIP-20_W7.62mm, symbol Interface_Expansion:TPIC6595
- added U2, U4: TPIC6595, Package_DIP:DIP-20_W7.62mm, symbol mtg_life_counter:TPIC6595
Connections:
- net +5V: now also U2.2 (VCC), U4.2 (VCC)
- net GND: now also U2.10 (GND), U2.11 (GND), U2.19 (GND), U4.10 (GND), U4.11 (GND), U4.19 (GND)
- net NENABLE: now also U2.9 (~G), U4.9 (~G)
- net SER_CASCADE_2: now also U2.3 (SER_IN)
- net SER_CASCADE_3: now also U2.18 (SER_OUT), U4.3 (SER_IN)
- net SER_CLK: now also U2.13 (SRCK), U4.13 (SRCK)
- net SER_LATCH: now also U2.12 (RCLK), U4.12 (RCLK)
- net at D1.10 (CC3): now also U2.6 (DRAIN2)
- net at D1.11 (CC2): now also U2.5 (DRAIN1)
- net at D1.14 (CC1): now also U2.4 (DRAIN0)
- net at D1.6 (CC4): now also U2.7 (DRAIN3)
- net at D2.10 (CC3): now also U2.16 (DRAIN6)
- net at D2.11 (CC2): now also U2.15 (DRAIN5)
- net at D2.14 (CC1): now also U2.14 (DRAIN4)
- net at D2.6 (CC4): now also U2.17 (DRAIN7)
- net at D3.10 (CC3): now also U4.16 (DRAIN6)
- net at D3.11 (CC2): now also U4.15 (DRAIN5)
- net at D3.14 (CC1): now also U4.14 (DRAIN4)
- net at D3.6 (CC4): now also U4.17 (DRAIN7)
- net at D4.10 (CC3): now also U4.6 (DRAIN2)
- net at D4.11 (CC2): now also U4.5 (DRAIN1)
- net at D4.14 (CC1): now also U4.4 (DRAIN0)
- net at D4.6 (CC4): now also U4.7 (DRAIN3)
- net at R33.1: now also U2.8 (~SRCLR)
- net at R34.1: now also U4.8 (~SRCLR)
Changed lines of the file:
@@
 $EndComp
 Wire Wire Line
-	10650 6250 10850 6250
+	10650 6250 10750 6250
 Wire Wire Line
 	10650 6250 10650 6350
-Connection ~ 10650 6250
-$Comp
-L Interface_Expansion:TPIC6595 U4
-U 1 1 61791AA4
-P 10550 5550
-F 0 "U4" H 10850 6150 50  0000 C CNN
-F 1 "TPIC6595" H 10750 4850 50  0000 C CNN
-F 2 "Package_DIP:DIP-20_W7.62mm" H 11200 4900 50  0001 C CNN
-F 3 "http://www.ti.com/lit/ds/symlink/tpic6595.pdf" H 10550 5500 50  0001 C CNN
-	1    10550 5550
-	-1   0    0    -1
-$EndComp
 Wire Wire Line
 	11050 5150 11150 5150
@@
 $EndComp
 Wire Wire Line
-	10650 3100 10850 3100
+	10650 3100 10750 3100
 Wire Wire Line
 	10650 3100 10650 3200
-Connection ~ 10650 3100
-$Comp
-L Interface_Expansion:TPIC6595 U2
-U 1 1 5F96845D
-P 10550 2400
-F 0 "U2" H 10850 3000 50  0000 C CNN
-F 1 "TPIC6595" H 10750 1700 50  0000 C CNN
-F 2 "Package_DIP:DIP-20_W7.62mm" H 11200 1750 50  0001 C CNN
-F 3 "http://www.ti.com/lit/ds/symlink/tpic6595.pdf" H 10550 2350 50  0001 C CNN
-	1    10550 2400
-	-1   0    0    -1
-$EndComp
 Wire Wire Line
 	11700 2000 11050 2000
@@
 Text Label 2650 7150 0    50   ~ 0
 OFF
+$Comp
+L mtg_life_counter:TPIC6595 U4
+U 1 1 60554267
+P 10550 5550
+F 0 "U4" H 10850 6150 50  0000 C CNN
+F 1 "TPIC6595" H 10750 4850 50  0000 C CNN
+F 2 "Package_DIP:DIP-20_W7.62mm" H 11200 4900 50  0001 C CNN
+F 3 "http://www.ti.com/lit/ds/symlink/tpic6595.pdf" H 10550 5500 50  0001 C CNN
+	1    10550 5550
+	-1   0    0    -1
+$EndComp
+Connection ~ 10650 6250
+$Comp
+L mtg_life_counter:TPIC6595 U2
+U 1 1 6055710C
+P 10550 2400
+F 0 "U2" H 10850 3000 50  0000 C CNN
+F 1 "TPIC6595" H 10750 1700 50  0000 C CNN
+F 2 "Package_DIP:DIP-20_W7.62mm" H 11200 1750 50  0001 C CNN
+F 3 "http://www.ti.com/lit/ds/symlink/tpic6595.pdf" H 10550 2350 50  0001 C CNN
+	1    10550 2400
+	-1   0    0    -1
+$EndComp
+Connection ~ 10650 3100
+Wire Wire Line
+	10750 3100 10850 3100
+Connection ~ 10750 3100
+Wire Wire Line
+	10750 6250 10850 6250
+Connection ~ 10750 6250
 $EndSCHEMATC
