File: mtg_life_counter/mtg_life_counter.kicad_pcb (KiCad board)
At the start: 2 copper layers, 208.3 x 127 mm, 77 parts, among them SW1 SW_SPDT, SW2 SW_SPST, SW3 SW_SP4T, SW4 SW_SP4T, SW5 SW_SP4T, SW6 SW_SP4T, U1 74HC595, U2 TPIC6595, U3 74HC595, U4 TPIC6595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

Commit message: Fix TPIC pinout
Parts:
- moved B2 12.7 mm to (154.8, 88.9)
- moved C1 12.7 mm to (233.7, 73.7)
- moved C5 12.7 mm to (153.7, 76.2)
- moved C6 12.7 mm to (130.8, 101.6)
- moved C7 12.7 mm to (177.8, 85.0)
- moved H2 12.7 mm to (241.3, 30.5)
- moved H3 12.7 mm to (241.3, 147.3)
- moved R13 12.7 mm to (201.9, 58.4)
- moved R15 12.7 mm to (184.2, 58.4)
- moved R16 12.7 mm to (191.8, 58.4)
- moved R21 12.7 mm to (184.2, 119.4)
- moved R22 12.7 mm to (191.8, 119.4)
- moved R23 12.7 mm to (201.9, 119.4)
- moved RN1 12.7 mm to (152.4, 58.4)
- moved RN2 12.7 mm to (132.1, 119.4)
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Connections:
- U2 pad 1: GND -> Net-(U2-Pad1)
- U2 pad 20: GND -> Net-(U2-Pad20)
- U4 pad 1: GND -> Net-(U4-Pad1)
- U4 pad 20: GND -> Net-(U4-Pad20)
Routing:
- net Net-(D3-Pad6): track 190.4 -> 166.6 mm, vias 3 -> 1
- net Net-(D3-Pad10): track 176.6 -> 160.6 mm, vias 3 -> 1
- net Net-(D4-Pad10): track 47.5 -> 59.5 mm, vias 1 -> 2
- net Net-(D3-Pad14): track 145.8 -> 141.8 mm, vias 3 -> 1
- net Net-(D4-Pad6): track 59.8 -> 55.8 mm
- net Net-(D4-Pad14): track 42.4 -> 38.4 mm
- net Net-(D3-Pad11): track 157.7 -> 153.8 mm, vias 3 -> 1
- net Net-(B10-Pad1): track 194.5 -> 197.5 mm, vias 1 -> 2
- net Net-(D4-Pad11): track 44.2 -> 42.7 mm
- net /SER_CASCADE_3: track 42.3 -> 43.0 mm, vias 1 -> 2
- net /SER_CLK: track 377.5 -> 377.0 mm, vias 1 -> 0
- net GND: vias 928 -> 924

Commit message: Complete PCB layout. Purchased version
Parts:
- moved RN2 1.27 mm to (130.8, 119.4)
- moved RN1 1.27 mm to (153.7, 58.4)
- turned SW3 to 292.5 degrees
- turned SW4 to 292.5 degrees
- turned SW5 to 112.5 degrees
- turned SW6 to 112.5 degrees
Routing:
- net Net-(RN1-Pad5): track 10.7 -> 33.3 mm
- net Net-(RN2-Pad5): track 10.7 -> 33.3 mm
- net Net-(RN1-Pad6): track 21.5 -> 44.0 mm
- net Net-(RN2-Pad6): track 21.5 -> 44.0 mm
- net Net-(RN1-Pad9): track 21.5 -> 42.8 mm
- net Net-(RN2-Pad9): track 21.5 -> 42.8 mm
- net Net-(RN1-Pad2): track 10.7 -> 32.1 mm
- net Net-(RN2-Pad2): track 10.7 -> 32.1 mm
- net Net-(RN1-Pad7): track 21.5 -> 42.2 mm
- net Net-(RN2-Pad7): track 21.5 -> 42.2 mm
- net Net-(RN2-Pad4): track 10.7 -> 31.4 mm
- net Net-(RN1-Pad4): track 10.7 -> 31.4 mm
- net Net-(RN1-Pad3): track 10.7 -> 31.2 mm
- net Net-(RN2-Pad3): track 10.7 -> 31.2 mm
- net Net-(RN1-Pad8): track 21.5 -> 41.9 mm
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