File: pcb/mtg_life_counter.sch (KiCad schematic (older format))
At the start: 77 parts, among them SW1 SW_SPDT, SW2 SW_SPST, SW3 SW_SP4T, SW4 SW_SP4T, SW5 SW_SP4T, SW6 SW_SP4T, U1 74HC595, U2 TPIC6595, U3 74HC595, U4 TPIC6595, U5 74LS151, U6 74LS151, U7 74LS151

Commit message: Fix A6 A7 digital mode bug (SCHEMATIC ONLY)
Parts:
- A1: symbol MCU_Module:Arduino_Nano_v3.x -> mtg_life_counter-rescue:Arduino_Nano_v3.x-MCU_Module
Changed lines of the file:
@@
 EESchema Schematic File Version 4
-LIBS:mtg_life_counter-cache
 EELAYER 30 0
 EELAYER END
@@
 $EndDescr
 $Comp
-L MCU_Module:Arduino_Nano_v3.x A1
+L mtg_life_counter-rescue:Arduino_Nano_v3.x-MCU_Module A1
 U 1 1 5F28B68A
 P 2450 8550
@@
 Text Label 3450 9050 2    50   ~ 0
 SEL_0
-Text Label 3450 9150 2    50   ~ 0
+Text Label 3450 8550 2    50   ~ 0
 SEL_1
-Text Label 3450 9250 2    50   ~ 0
+Text Label 1450 8950 0    50   ~ 0
 SEL_2
 Text Label 3450 8950 2    50   ~ 0
@@
 	2950 9050 3450 9050
 Wire Wire Line
-	2950 9150 3450 9150
-Wire Wire Line
 	2950 9250 3450 9250
 Wire Wire Line
@@
 Wire Wire Line
 	2950 8750 3450 8750
-NoConn ~ 1950 8950
-Text Label 3450 8550 2    50   ~ 0
+Text Label 3450 9250 2    50   ~ 0
 RNG_WIRE
 Wire Wire Line
@@
 INT_0
 NoConn ~ 1950 9150
-NoConn ~ 2950 8550
 NoConn ~ 1950 8250
 $Comp
@@
 	10750 6250 10850 6250
 Connection ~ 10750 6250
+NoConn ~ 2950 9250
+NoConn ~ 2950 9150
+Wire Wire Line
+	1450 8950 1950 8950
 $EndSCHEMATC

Commit message: Update resistor values for displays. Remove power switch resistor
Parts:
- removed R35: 100, Resistor_THT:R_Axial_DIN0207_L6.3mm_D2.5mm_P10.16mm_Horizontal, symbol Device:R
- D1: value KW4-56NX -> KW4-56NX RED
- D2: value KW4-56NX -> KW4-56NX GREEN
- D3: value KW4-56NX -> KW4-56NX YELLOW
- D4: value KW4-56NX -> KW4-56NX BLUE
- R1, R2, R3, R4, R5, R6, R7, R8: value R -> 330
- R10, R11, R12, R13, R14, R15, R16, R9: value R -> 22
- R17, R18, R19, R20, R21, R22, R23, R24: value R -> 100
- R25, R26, R27, R28, R29, R30, R31, R32: value R -> 390
Connections:
- wire segments 350 -> 349

Commit message: begin design plan for mini
Parts:
- removed B10, B3, B4, B5, B6, B7, B8, B9: SW_Push, mtg_life_counter:B3F_12mm, symbol Switch:SW_Push
- removed C6, C7: 0.1uF, Capacitor_THT:C_Disc_D3.0mm_W1.6mm_P2.50mm, symbol Device:C_Small
- removed RN2, RN3: 1000, Resistor_THT:R_Array_SIP9, symbol Device:R_Network08_US
- removed SW3, SW4, SW5, SW6: SW_SP4T, mtg_life_counter:CK_RM10x77, symbol mtg_life_counter:SW_SP4T
- removed U6, U7: 74LS151, Package_DIP:DIP-16_W7.62mm, symbol 74xx:74LS151
- added U?: ATmega328P-AU, Package_QFP:TQFP-32_7x7mm_P0.8mm, symbol MCU_Microchip_ATmega:ATmega328P-AU
- added Y?: Crystal_Small, symbol Device:Crystal_Small
- R10, R11, R12, R13, R14, R15, R16, R9: value 22 -> 33
Connections:
- net labels added: ENCODER_RB
- wire segments 349 -> 269
- no-connect marks 25 -> 23
Other:
- note removed: "Button Sense"
- note removed: "Switch Sense 2"
- moved on the sheet: C1, C2, C3, C4, C5, D1, D2, D3, D4, R1, R10, R11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

Commit message: Sketch out mini pcb
Parts:
- removed RN1: 1000, Resistor_THT:R_Array_SIP9, symbol Device:R_Network08_US
- added E1, E2, E3, E4: Rotary_Encoder_Switch, Rotary_Encoder:RotaryEncoder_Alps_EC11E-Switch_Vertical_H20mm, symbol Device:Rotary_Encoder_Switch
- added J1: USB_B_Micro, Connector_USB:USB_Micro-B_Molex-105017-0001, symbol Connector:USB_B_Micro
- added R35, R36, R37, R38, R39, R40, R41, R42: 10k, Resistor_SMD:R_1206_3216Metric_Pad1.42x1.75mm_HandSolder, symbol Device:R
- added U2: FT232RL, Package_SO:SSOP-28_5.3x10.2mm_P0.65mm, symbol Interface_USB:FT232RL
- C1, C2, C3, C4, C5: footprint Capacitor_THT:C_Disc_D3.0mm_W1.6mm_P2.50mm -> Capacitor_SMD:C_1206_3216Metric_Pad1.42x1.75mm_HandSolder
- R1, R10, R11, R12, R13, R14, R15, R16, R17, R18, R19, R2, R20, R21, R22, R23, R24, R25, R26, R27, R28, R29, R3, R30, R31, R32, R33, R34, R4, R5, R6, R7, R8, R9: footprint Resistor_THT:R_Axial_DIN0207_L6.3mm_D2.5mm_P10.16mm_Horizontal -> Resistor_SMD:R_1206_3216Metric_Pad1.42x1.75mm_HandSolder
- U1: renamed from U?; symbol MCU_Microchip_ATmega:ATmega328P-AU -> mtg_life_counter-rescue:ATmega328P-AU-MCU_Microchip_ATmega
- U3: renamed from U5; footprint Package_DIP:DIP-16_W7.62mm -> Package_SO:SOIC-16_3.9x9.9mm_P1.27mm
- U4: renamed from U1; footprint Package_DIP:DIP-16_W7.62mm -> Package_SO:SOIC-16_3.9x9.9mm_P1.27mm
- U5: renamed from U3; footprint Package_DIP:DIP-16_W7.62mm -> Package_SO:SOIC-16_3.9x9.9mm_P1.27mm
- U6: renamed from U2; value TPIC6595 -> TPIC6C596; footprint Package_DIP:DIP-20_W7.62mm -> Package_SO:SOIC-16_3.9x9.9mm_P1.27mm
- U7: renamed from U4; value TPIC6595 -> TPIC6C596; footprint Package_DIP:DIP-20_W7.62mm -> Package_SO:SOIC-16_3.9x9.9mm_P1.27mm
- gave numbers to parts that had none: 1
Connections:
- net labels added: MUX_RB, MUX_SEL_0, MUX_SEL_1, MUX_SEL_2
- net labels removed: ENCODER_RB
- wire segments 269 -> 272
Other:
- note added: "Encoder Multiplexing"
- note removed: "Switch Sense 1"
- moved on the sheet: B1, B2, C5, H1, H2, H3, H4, SW2, U3, Y1

Commit message: Continue updating schematic
Parts:
- removed A1: Arduino_Nano_v3.x, Module:Arduino_Nano, symbol mtg_life_counter-rescue:Arduino_Nano_v3.x-MCU_Module
- removed SW1: SW_SPDT, Button_Switch_THT:SW_Slide_1P2T_CK_OS102011MS2Q, symbol Switch:SW_SPDT
- removed U1: ATmega328P-AU, Package_QFP:TQFP-32_7x7mm_P0.8mm, symbol mtg_life_counter-rescue:ATmega328P-AU-MCU_Microchip_ATmega
- added C6, C7: 0.1uF, Capacitor_SMD:C_1206_3216Metric_Pad1.42x1.75mm_HandSolder, symbol Device:C_Small
- added C?: 100nF, Capacitor_SMD:C_1206_3216Metric_Pad1.42x1.75mm_HandSolder, symbol Device:C_Small
- added J?: ICSP, symbol Connector_Generic:Conn_02x03_Odd_Even
- added R? (x2): 1k, Resistor_SMD:R_1206_3216Metric_Pad1.42x1.75mm_HandSolder, symbol Device:R
- added SW1: SW_SPST, Button_Switch_THT:SW_Slide_1P2T_CK_OS102011MS2Q, symbol Switch:SW_SPST
- added U1: ATmega328P-AU, Package_QFP:TQFP-32_7x7mm_P0.8mm, symbol mtg_life_counter:ATmega328P-AU
- Y1: value Crystal_Small -> 16MHz
Connections:
- net labels added: A0, A1, A2, A3, A4, A5, A6, A7, AREF, D0(RX), D1(TX), D10, D11(MOSI), D12(MISO), D13(SCK), D2, D3, D4, D5, D6, D7, D8, D9, E1_CLK, E1_DIR, E1_SW, E2_CLK, E2_DIR, E2_SW, E3_CLK, E3_DIR, E3_SW, E4_CLK, E4_DIR, E4_SW, SER_LINK_1, SER_LINK_2, SER_LINK_3, USB_DM, USB_DP, ~ENABLE, ~RESET
- net labels removed: 5V_SRC, BTN_RB, INT_0, INT_1, NENABLE, OFF, RNG_WIRE, SEL_0, SEL_1, SEL_2, SER_CASCADE_1, SER_CASCADE_2, SER_CASCADE_3, SPI_IN, SW_RB_1, SW_RB_2
- wire segments 272 -> 343
- no-connect marks 23 -> 28
Other:
- note added: "DNP"
- moved on the sheet: D3, D4, E1, J1, R17, R18, R19, R20, R21, R22, R23, R24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

Commit message: Continue work on mini PCB
Parts:
- removed R18, R19: 100, Resistor_SMD:R_1206_3216Metric_Pad1.42x1.75mm_HandSolder, symbol Device:R
- removed R2, R3, R4, R5, R6, R7, R8: 330, Resistor_SMD:R_1206_3216Metric_Pad1.42x1.75mm_HandSolder, symbol Device:R
- removed R28, R29: 390, Resistor_SMD:R_1206_3216Metric_Pad1.42x1.75mm_HandSolder, symbol Device:R
- removed R38, R39: 10k, Resistor_SMD:R_1206_3216Metric_Pad1.42x1.75mm_HandSolder, symbol Device:R
- removed R9: 33, Resistor_SMD:R_1206_3216Metric_Pad1.42x1.75mm_HandSolder, symbol Device:R
- removed U6, U7: TPIC6C596, Package_SO:SOIC-16_3.9x9.9mm_P1.27mm, symbol mtg_life_counter:TPIC6595
- added C3, C4: 0.1uF, Capacitor_SMD:C_1206_3216Metric_Pad1.42x1.75mm_HandSolder, symbol Device:C_Small
- added R33, R34: 100, Resistor_SMD:R_1206_3216Metric_Pad1.42x1.75mm_HandSolder, symbol Device:R
- added R43, R44, R45, R46, R47: 390, Resistor_SMD:R_1206_3216Metric_Pad1.42x1.75mm_HandSolder, symbol Device:R
- added R50, R51, R52, R53, R54, R55, R56, R57: 10k, Resistor_SMD:R_1206_3216Metric_Pad1.42x1.75mm_HandSolder, symbol Device:R
- added U4, U5: TPIC6596, Package_SO:SOIC-16_3.9x9.9mm_P1.27mm, symbol mtg_life_counter:TPIC6596
- C1: renamed from C6; value 0.1uF -> 18pF; footprint Capacitor_SMD:C_1206_3216Metric_Pad1.42x1.75mm_HandSolder -> Capacitor_SMD:C_0805_2012Metric_Pad1.15x1.40mm_HandSolder
- C2: renamed from C7; value 0.1uF -> 18pF; footprint Capacitor_SMD:C_1206_3216Metric_Pad1.42x1.75mm_HandSolder -> Capacitor_SMD:C_0805_2012Metric_Pad1.15x1.40mm_HandSolder
- J2: renamed from J?; footprint (none) -> Connector:Tag-Connect_TC2030-IDC-NL_2x03_P1.27mm_Vertical
- R1: value 330 -> 1k
- R10, R11, R12, R13, R14, R15, R16: value 33 -> 330
- R17: value 100 -> 330
- R20, R21, R22, R23, R24: value 100 -> 33
- R25, R26, R27: value 390 -> 33
- R30, R31, R32: value 390 -> 100
- R35, R36, R37: value 10k -> 100
- R40, R41, R42: value 10k -> 390
- Y1: footprint (none) -> Crystal:Crystal_HC49-U_Vertical
- gave numbers to parts that had none: 3
- renumbered C1 to C5, C3 to C6, C2 to C7, C4 to C8, C5 to C9, R33 to R2, R34 to R3, U4 to U2, U5 to U3, U3 to U6, U2 to U7
Connections:
- net labels added: VBUS
- wire segments 343 -> 347
Other:
- moved on the sheet: SW1

Commit message: Continue work on mini version
Parts:
- removed C2: 18pF, Capacitor_SMD:C_0805_2012Metric_Pad1.15x1.40mm_HandSolder, symbol Device:C_Small
- removed J1: USB_B_Micro, Connector_USB:USB_Micro-B_Molex-105017-0001, symbol Connector:USB_B_Micro
- removed U4, U5: TPIC6596, Package_SO:SOIC-16_3.9x9.9mm_P1.27mm, symbol mtg_life_counter:TPIC6596
- removed Y1: 16MHz, Crystal:Crystal_HC49-U_Vertical, symbol Device:Crystal_Small
- added J1: USB_C_Receptacle_USB2.0, Connector_USB:USB_C_Receptacle_GCT_USB4085, symbol Connector:USB_C_Receptacle_USB2.0
- added U4, U5: TPIC6B595, Package_SO:SOIC-20W_7.5x12.8mm_P1.27mm, symbol mtg_life_counter:TPIC6B595
- added Y1: 16MHz, Crystal:Resonator_muRata_CSTLSxxxX-3Pin_W5.5mm_H3.0mm, symbol Device:Resonator_Small
- C1: value 18pF -> 4.7uF
- C10: value 100nF -> 0.1uF; footprint Capacitor_SMD:C_1206_3216Metric_Pad1.42x1.75mm_HandSolder -> Capacitor_SMD:C_0805_2012Metric_Pad1.15x1.40mm_HandSolder
- C3, C5, C6, C7, C8, C9: footprint Capacitor_SMD:C_1206_3216Metric_Pad1.42x1.75mm_HandSolder -> Capacitor_SMD:C_0805_2012Metric_Pad1.15x1.40mm_HandSolder
- C4: value 0.1uF -> 1uF; footprint Capacitor_SMD:C_1206_3216Metric_Pad1.42x1.75mm_HandSolder -> Capacitor_SMD:C_0805_2012Metric_Pad1.15x1.40mm_HandSolder
- R1, R10, R11, R12, R13, R14, R15, R16, R17, R2, R20, R21, R22, R23, R24, R25, R26, R27, R3, R30, R31, R32, R33, R34, R35, R36, R37, R4, R40, R41, R42, R43, R44, R45, R46, R47, R5, R50, R51, R52, R53, R54, R55, R56, R57: footprint Resistor_SMD:R_1206_3216Metric_Pad1.42x1.75mm_HandSolder -> Resistor_SMD:R_0805_2012Metric_Pad1.15x1.40mm_HandSolder
Connections:
- net A0 is gone; now on net E1_SW: U1.23 (PC0(ADC0))
- net A1 is gone; now on net E2_SW: U1.24 (PC1(ADC1))
- net A2 is gone; now on net E3_SW: U1.25 (PC2(ADC2))
- net A3 is gone; now on net E4_SW: U1.26 (PC3(ADC3))
- net A4 is gone; now on net ROLL_BTN: U1.27 (PC4(SDA/ADC4))
- net A5 is gone; now on net RESET_BTN: U1.28 (PC5(SCL/ADC5))
- net D10 is gone; now on net SER_LATCH: U1.14 (PB2(CS))
- net D4 is gone; now on net MUX_SEL_0: U1.2 (PD4)
- net D5 is gone; now on net MUX_SEL_1: U1.9 (PD5)
- net D6 is gone; now on net MUX_SEL_2: U1.10 (PD6)
- net D7 is gone; now on net MUX_RB: U1.11 (PD7)
- net D8 is gone; now on net ~ENABLE: U1.12 (PB0(ICP))
- net D9 is gone; now on net MODE_SW: U1.13 (PB1)
- net +5V: now also R1.2, U4.2 (VCC), U5.2 (VCC)
- net D11(MOSI): no longer U1.15 (PB3(MOSI))
- net D12(MISO): no longer U1.16 (PB4(MISO))
- net D13(SCK): no longer U1.17 (PB5(SCK)), U2.11 (SRCLK), U3.11 (SRCLK)
- net GND: now also J1.A1 (GND), J1.A12 (GND), J1.B1 (GND), J1.B12 (GND), J1.S1 (SHIELD), U4.1 (NC), U4.10 (GND), U4.11 (GND), U4.19 (GND), U4.20 (NC), U5.1 (NC), U5.10 (GND), U5.11 (GND), U5.19 (GND), U5.20 (NC), Y1.2; no longer C1.2
- net SER_LATCH: now also U4.12 (RCLK), U5.12 (RCLK)
- net SER_LINK_1: now also U4.3 (SER_IN), U5.18 (SER_OUT)
- net SER_LINK_2: now also U4.18 (SER_OUT)
- net USB_DM: now also J1.A7 (D-), J1.B7 (D-)
- net USB_DP: now also J1.A6 (D+), J1.B6 (D+)
- net VBUS: now also J1.A4 (VBUS), J1.A9 (VBUS), J1.B4 (VBUS), J1.B9 (VBUS)
- net ~ENABLE: now also U4.9 (~G), U5.9 (~G)
- net ~RESET: now also R1.1
- net at D1.10 (CC3): now also U4.6 (DRAIN2)
- net at D1.11 (CC2): now also U4.5 (DRAIN1)
- net at D1.14 (CC1): now also U4.4 (DRAIN0)
- net at D1.6 (CC4): now also U4.7 (DRAIN3)
- net at D2.10 (CC3): now also U4.16 (DRAIN6)
- net at D2.11 (CC2): now also U4.15 (DRAIN5)
- net at D2.14 (CC1): now also U4.14 (DRAIN4)
- net at D2.6 (CC4): now also U4.17 (DRAIN7)
- net at D3.10 (CC3): now also U5.6 (DRAIN2)
- net at D3.11 (CC2): now also U5.5 (DRAIN1)
- net at D3.14 (CC1): now also U5.4 (DRAIN0)
- net at D3.6 (CC4): now also U5.7 (DRAIN3)
- net at D4.10 (CC3): now also U5.16 (DRAIN6)
- net at D4.11 (CC2): now also U5.15 (DRAIN5)
- net at D4.14 (CC1): now also U5.14 (DRAIN4)
- net at D4.6 (CC4): now also U5.17 (DRAIN7)
- net at U1.7 (XTAL1(PB6)): now also Y1.1; no longer C1.1
- net at U1.8 (XTAL2(PB7)): now also Y1.3
- net +3V3: now reaches U7.17 (3V3OUT)
- net at R2.1: now also U4.8 (~SRCLR)
- net at R3.1: now also U5.8 (~SRCLR)
- net D2: no longer names the net of U1.32 (PD2(INT0))
- net D3: no longer names the net of U1.1 (PD3(INT1))
- new net SER_CLK: U1.17 (PB5(SCK)), U2.11 (SRCLK), U3.11 (SRCLK), U4.13 (SRCK), U5.13 (SRCK)
- new net SER_DATA: U1.15 (PB3(MOSI)), U5.3 (SER_IN)
- no-connect marks 28 -> 34
Other:
- note added: "A0"
- note added: "A1"
- note added: "A2"
- note added: "A3"
- note added: "A4"
- note added: "A5"
- note added: "D10"
- note added: "D11(MOSI)"
- note added: "D12(MISO)"
- note added: "D13(SCK)"
- note added: "D2(INT0)"
- note added: "D3(INT1)"
- note added: "D4"
- note added: "D5"
- note added: "D6"
- note added: "D7"
- note added: "D8"
- note added: "D9"
- moved on the sheet: B1, B2, C10, C3, C4, C9, E1, E2, E3, E4, H1, H2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

Commit message: Tweak layout
Parts:
- J1: symbol Connector:USB_C_Receptacle_USB2.0 -> mtg_life_counter-rescue:USB_C_Receptacle_USB2.0-Connector
- U7: symbol Interface_USB:FT232RL -> mtg_life_counter-rescue:FT232RL-Interface_USB
Connections:
- net USB_DM renamed USB_D_N
- net USB_DP renamed USB_D_P
Changed lines of the file:
@@
 $EndComp
 $Comp
-L Interface_USB:FT232RL U7
+L mtg_life_counter-rescue:FT232RL-Interface_USB U7
 U 1 1 5F77F9F3
 P 6000 5450
@@
 ~ENABLE
 Text Label 3500 5500 2    50   ~ 0
-USB_DP
+USB_D_P
 Text Label 3500 5300 2    50   ~ 0
-USB_DM
+USB_D_N
 $Comp
 L power:GND #PWR0101
@@
 Wire Wire Line
 	3500 5300 3000 5300
-Text Label 4850 5050 0    50   ~ 0
-USB_DP
 Wire Wire Line
 	4850 5050 5200 5050
 Wire Wire Line
 	4850 5150 5200 5150
-Text Label 4850 5150 0    50   ~ 0
-USB_DM
 NoConn ~ 5200 4750
 $Comp
@@
 	2400 6300 2400 6400
 $Comp
-L Connector:USB_C_Receptacle_USB2.0 J1
+L mtg_life_counter-rescue:USB_C_Receptacle_USB2.0-Connector J1
 U 1 1 5F6AF0EA
 P 2400 5400
@@
 Text Notes 3150 2900 0    50   ~ 0
 D4
+Text Label 4850 5050 0    50   ~ 0
+USB_D_P
+Text Label 4850 5150 0    50   ~ 0
+USB_D_N
 $EndSCHEMATC
