File: pcb/mtg_life_counter.sch (KiCad schematic (older format))
At the start: 80 parts, among them J1 USB_C_Receptacle_USB2.0, J2 ICSP, SW1 SW_SPST, SW2 SW_SPST, U1 ATmega328P-AU, U2 74HC595, U3 74HC595, U4 TPIC6B595, U5 TPIC6B595, U6 74LS151, U7 FT232RL, Y1 16MHz

Commit message: complete electrical layout
Parts:
- removed C10: 0.1uF, Capacitor_SMD:C_0805_2012Metric_Pad1.15x1.40mm_HandSolder, symbol Device:C_Small
- removed D1: KW4-56NX RED, mtg_life_counter:KW4-56NX, symbol mtg_life_counter:KW4-56NX
- removed D2: KW4-56NX GREEN, mtg_life_counter:KW4-56NX, symbol mtg_life_counter:KW4-56NX
- removed D3: KW4-56NX YELLOW, mtg_life_counter:KW4-56NX, symbol mtg_life_counter:KW4-56NX
- removed D4: KW4-56NX BLUE, mtg_life_counter:KW4-56NX, symbol mtg_life_counter:KW4-56NX
- removed R4, R5: 1k, Resistor_SMD:R_0805_2012Metric_Pad1.15x1.40mm_HandSolder, symbol Device:R
- removed U7: FT232RL, Package_SO:SSOP-28_5.3x10.2mm_P0.65mm, symbol mtg_life_counter-rescue:FT232RL-Interface_USB
- added C5, C7: 0.1uF, Capacitor_SMD:C_0805_2012Metric_Pad1.15x1.40mm_HandSolder, symbol Device:C_Small
- added D1: KW4-566CVB RED, mtg_life_counter:KW4-566xxB_THT, symbol mtg_life_counter:KW4-566CxB
- added D2: KW4-566CVB GREEN, mtg_life_counter:KW4-566xxB_THT, symbol mtg_life_counter:KW4-566CxB
- added D3: KW4-566CVB YELLOW, mtg_life_counter:KW4-566xxB_THT, symbol mtg_life_counter:KW4-566CxB
- added D4: KW4-566CVB BLUE, mtg_life_counter:KW4-566xxB_THT, symbol mtg_life_counter:KW4-566CxB
- added TP1: INT0, TestPoint:TestPoint_Pad_D1.0mm, symbol Connector:TestPoint
- added TP2: Debug, TestPoint:TestPoint_Pad_D1.0mm, symbol Connector:TestPoint
- added U3, U5: 74HC595, Package_SO:SOIC-16_3.9x9.9mm_P1.27mm, symbol 74xx:74HC595
- renumbered C3 to C1, C9 to C10, C1 to C2, C4 to C3, C5 to C4, C7 to C8, C8 to C9, U3 to U4, U4 to U6, U5 to U7, U6 to U8
Connections:
- net labels added: D2(INT0), DEBUG_PIN, SER_LINK_4, SER_LINK_5
- net labels removed: +3.3V, D11(MOSI), D13(SCK), USB_D_N, USB_D_P
- wire segments 345 -> 331
- no-connect marks 34 -> 14
Other:
- note added: "D0(RX)"
- note added: "D1(TX)"
- note added: "Seven Segement Displays"
- note removed: "DNP"
- note removed: "Display Bank 1"
- note removed: "Display Bank 2"
- moved on the sheet: B1, B2, C1, C10, C2, C3, C4, C6, C8, C9, E1, E2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

Commit message: Switch to 74x165. Optimize pin assignments
Parts:
- removed U8: 74LS151, Package_SO:SOIC-16_3.9x9.9mm_P1.27mm, symbol 74xx:74LS151
- added TP1: TX, TestPoint:TestPoint_Pad_D1.5mm, symbol Connector:TestPoint
- added TP2: RX, TestPoint:TestPoint_Pad_D1.5mm, symbol Connector:TestPoint
- added U8: 74HC165, Package_SO:SOIC-16_3.9x9.9mm_P1.27mm, symbol mtg_life_counter:74HC165
- TP3: renamed from TP1; footprint TestPoint:TestPoint_Pad_D1.0mm -> TestPoint:TestPoint_Pad_D1.5mm
- TP4: renamed from TP2; footprint TestPoint:TestPoint_Pad_D1.0mm -> TestPoint:TestPoint_Pad_D1.5mm
Connections:
- net labels added: SER_IN, SER_MISO, SER_MOSI
- net labels removed: D12(MISO), MUX_RB, MUX_SEL_0, MUX_SEL_1, MUX_SEL_2, SER_DATA
- no-connect marks 14 -> 17
Changed lines of the file:
@@
 Sheet 1 1
 Title "Magic: The Gathering Life Counter"
-Date "2020-09-03"
+Date "2021-02-10"
 Rev "2.0"
 Comp "Max Proskauer"
@@
 $EndComp
 $Comp
-L 74xx:74LS151 U8
-U 1 1 5F293C96
-P 2500 8850
-F 0 "U8" H 2750 9600 50  0000 C CNN
-F 1 "74LS151" H 2300 9600 50  0000 C CNN
-F 2 "Package_SO:SOIC-16_3.9x9.9mm_P1.27mm" H 2500 8850 50  0001 C CNN
-F 3 "http://www.ti.com/lit/gpn/sn74LS151" H 2500 8850 50  0001 C CNN
-	1    2500 8850
-	-1   0    0    -1
-$EndComp
-$Comp
 L power:+5V #PWR029
 U 1 1 5F2A4AB1
@@
 	1    0    0    -1
 $EndComp
-Text Label 3750 9150 2    50   ~ 0
-MUX_SEL_0
-Text Label 3750 9250 2    50   ~ 0
-MUX_SEL_1
-Text Label 3750 9350 2    50   ~ 0
-MUX_SEL_2
-Wire Wire Line
-	3750 9150 3000 9150
-Wire Wire Line
-	3000 9250 3750 9250
-Wire Wire Line
-	3000 9350 3750 9350
 $Comp
 L power:GND #PWR026
 U 1 1 5F2E233A
-P 3000 9850
-F 0 "#PWR026" H 3000 9600 50  0001 C CNN
-F 1 "GND" H 3005 9677 50  0000 C CNN
-F 2 "" H 3000 9850 50  0001 C CNN
-F 3 "" H 3000 9850 50  0001 C CNN
-	1    3000 9850
-	1    0    0    -1
-$EndComp
-Wire Wire Line
-	2500 9850 3000 9850
-Wire Wire Line
-	3000 9550 3000 9850
-Connection ~ 3000 9850
+P 5050 10050
+F 0 "#PWR026" H 5050 9800 50  0001 C CNN
+F 1 "GND" H 5055 9877 50  0000 C CNN
+F 2 "" H 5050 10050 50  0001 C CNN
+F 3 "" H 5050 10050 50  0001 C CNN
+	1    5050 10050
+	1    0    0    -1
+$EndComp
+Wire Wire Line
+	4550 10050 5050 10050
+Wire Wire Line
+	5050 9750 5050 10050
+Connection ~ 5050 10050
 $Comp
 L power:+5V #PWR023
@@
 Wire Wire Line
 	2100 7850 2200 7850
-Text Label 1500 8250 0    50   ~ 0
-MUX_RB
 Wire Wire Line
 	14300 2550 14400 2550
@@
 Text Label 15900 3350 2    50   ~ 0
 SER_LINK_2
-NoConn ~ 2000 8350
-Wire Wire Line
-	1500 8250 2000 8250
 $Comp
 L Device:Rotary_Encoder_Switch E1
@@
 	1    0    0    -1
 $EndComp
-Text Label 15900 6400 2    50   ~ 0
-SER_DATA
 Wire Wire Line
 	15400 6400 15900 6400
@@
 Wire Wire Line
 	3550 1800 4500 1800
-Text Label 7300 2700 2    50   ~ 0
-SER_DATA
 Text Label 5800 2700 0    50   ~ 0
 SER_CLK
-Text Label 4500 1800 2    50   ~ 0
-D12(MISO)
+Text Label 5800 2600 0    50   ~ 0
+SER_MISO
 Wire Wire Line
 	5900 1900 6400 1900
 $Comp
-L Connector:TestPoint TP2
+L Connector:TestPoint TP4
 U 1 1 608B6D51
 P 6400 1900
-F 0 "TP2" V 6400 2100 50  0000 L CNN
+F 0 "TP4" V 6400 2100 50  0000 L CNN
 F 1 "Debug" V 6400 2300 50  0000 L CNN
-F 2 "TestPoint:TestPoint_Pad_D1.0mm" H 6600 1900 50  0001 C CNN
+F 2 "TestPoint:TestPoint_Pad_D1.5mm" H 6600 1900 50  0001 C CNN
 F 3 "~" H 6600 1900 50  0001 C CNN
 	1    6400 1900
@@
 	3550 3600 4500 3600
 $Comp
-L Connector:TestPoint TP1
+L Connector:TestPoint TP3
 U 1 1 60802308
 P 6400 1750
-F 0 "TP1" V 6400 1950 50  0000 L CNN
+F 0 "TP3" V 6400 1950 50  0000 L CNN
 F 1 "INT0" V 6400 2150 50  0000 L CNN
-F 2 "TestPoint:TestPoint_Pad_D1.0mm" H 6600 1750 50  0001 C CNN
+F 2 "TestPoint:TestPoint_Pad_D1.5mm" H 6600 1750 50  0001 C CNN
 F 3 "~" H 6600 1750 50  0001 C CNN
 	1    6400 1750
@@
 Text Notes 3600 3500 0    50   ~ 0
 D3(INT1)
-Text Notes 4950 1600 2    50   ~ 0
-D12(MISO)
 Text Notes 3600 2900 0    50   ~ 0
 A0
@@
 Wire Wire Line
 	3550 2100 4500 2100
-Wire Wire Line
-	3550 2500 4500 2500
-Text Label 4500 2900 2    50   ~ 0
+Text Label 4500 3200 2    50   ~ 0
 ROLL_BTN
 Text Label 4500 2100 2    50   ~ 0
 MODE_SW
 Wire Wire Line
-	3550 3400 4500 3400
-Wire Wire Line
-	3550 3300 4500 3300
-Wire Wire Line
-	3550 3200 4500 3200
-Wire Wire Line
-	3550 3100 4500 3100
-Wire Wire Line
-	3550 2900 4500 2900
-Wire Wire Line
 	3550 2800 4500 2800
 Wire Wire Line
 	3550 2700 4500 2700
-Wire Wire Line
-	3550 2600 4500 2600
 Text Label 4500 2200 2    50   ~ 0
 E3_SW
-Text Label 4500 3400 2    50   ~ 0
+Text Label 4500 3300 2    50   ~ 0
 E4_SW
 Text Label 4500 2800 2    50   ~ 0
@@
 Text Label 4500 2700 2    50   ~ 0
 E1_SW
-Text Label 4500 3300 2    50   ~ 0
-MUX_SEL_2
-Text Label 4500 3200 2    50   ~ 0
-MUX_SEL_1
-Text Label 4500 3100 2    50   ~ 0
-MUX_SEL_0
-Text Label 4500 2600 2    50   ~ 0
-MUX_RB
 Wire Wire Line
 	1550 3400 1650 3400
@@
 Text Label 5800 2800 0    50   ~ 0
 ~RESET
-Text Label 5800 2600 0    50   ~ 0
-D12(MISO)
 $Comp
 L power:GND #PWR0118
@@
 D1(TX)
 Text Label 4500 1900 2    50   ~ 0
-SER_DATA
+SER_MOSI
 Text Label 4500 1700 2    50   ~ 0
 SER_CLK
@@
 	1    0    0    -1
 $EndComp
-NoConn ~ 4500 2500
+Text Label 15900 6400 2    50   ~ 0
+SER_MOSI
+Text Label 1300 8250 0    50   ~ 0
+SER_IN
+Text Notes 3600 1800 0    50   ~ 0
+D12(MISO)
+Text Label 1300 8650 0    50   ~ 0
+SER_LATCH
+$Comp
+L mtg_life_counter:74HC165 U8
+U 1 1 603BF06B
+P 2500 8850
+F 0 "U8" H 2250 9750 50  0000 C CNN
+F 1 "74HC165" H 2250 9650 50  0000 C CNN
+F 2 "Package_SO:SOIC-16_3.9x9.9mm_P1.27mm" H 2500 8850 50  0001 C CNN
+F 3 "http://www.ti.com/lit/gpn/sn74LS165" H 2500 8850 50  0001 C CNN
+	1    2500 8850
+	-1   0    0    -1
+$EndComp
+$Comp
+L power:GND #PWR01
+U 1 1 603EBE82
+P 2500 9350
+F 0 "#PWR01" H 2500 9100 50  0001 C CNN
+F 1 "GND" H 2505 9177 50  0000 C CNN
+F 2 "" H 2500 9350 50  0001 C CNN
+F 3 "" H 2500 9350 50  0001 C CNN
+	1    2500 9350
+	1    0    0    -1
+$EndComp
+Wire Wire Line
+	2500 9250 2500 9350
+Connection ~ 2500 9250
+Text Label 1300 8850 0    50   ~ 0
+SER_CLK
+Wire Wire Line
+	1300 8850 2000 8850
+Wire Wire Line
+	1300 8250 2000 8250
+Wire Wire Line
+	1300 8650 2000 8650
+Wire Wire Line
+	2000 8550 1900 8550
+Wire Wire Line
+	1900 8550 1900 8950
+Wire Wire Line
+	2000 8950 1900 8950
+Connection ~ 1900 8950
+Wire Wire Line
+	1900 8950 1900 9250
+Wire Wire Line
+	1900 9250 2500 9250
+$Comp
+L Connector:TestPoint TP2
+U 1 1 60642369
+P 4500 3800
+F 0 "TP2" V 4500 4000 50  0000 L CNN
+F 1 "RX" V 4500 4200 50  0000 L CNN
+F 2 "TestPoint:TestPoint_Pad_D1.5mm" H 4700 3800 50  0001 C CNN
+F 3 "~" H 4700 3800 50  0001 C CNN
+	1    4500 3800
+	0    1    1    0
+$EndComp
+$Comp
+L Connector:TestPoint TP1
+U 1 1 60642AD4
+P 4500 3700
+F 0 "TP1" V 4500 3900 50  0000 L CNN
+F 1 "TX" V 4500 4100 50  0000 L CNN
+F 2 "TestPoint:TestPoint_Pad_D1.5mm" H 4700 3700 50  0001 C CNN
+F 3 "~" H 4700 3700 50  0001 C CNN
+	1    4500 3700
+	0    1    1    0
+$EndComp
+NoConn ~ 3550 2500
+NoConn ~ 3550 2600
+NoConn ~ 3550 3400
+Text Label 4500 1800 2    50   ~ 0
+SER_MISO
+Text Label 7300 2700 2    50   ~ 0
+SER_MOSI
+Wire Wire Line
+	4500 3300 3550 3300
+Wire Wire Line
+	4500 3200 3550 3200
+NoConn ~ 3550 2900
+NoConn ~ 3550 3100
 $EndSCHEMATC

Commit message: Finish routing
Connections:
- net SER_IN is gone; now on net SER_MISO: U8.9 (Q7)
- net E1_CLK: now also U8.13 (D2); no longer U8.12 (D1)
- net E1_DIR: now also U8.14 (D3); no longer U8.11 (D0)
- net E1_SW: now also U1.27 (PC4(SDA/ADC4)); no longer U1.25 (PC2(ADC2))
- net E2_CLK: now also U8.11 (D0); no longer U8.14 (D3)
- net E2_DIR: now also U8.12 (D1); no longer U8.13 (D2)
- net E2_SW: now also E2.S2, U1.26 (PC3(ADC3)); no longer E2.S1, U1.24 (PC1(ADC1))
- net E3_CLK: now also U8.5 (D6); no longer U8.4 (D5)
- net E3_DIR: now also U8.6 (D7); no longer U8.3 (D4)
- net E4_CLK: now also U8.3 (D4); no longer U8.6 (D7)
- net E4_DIR: now also U8.4 (D5); no longer U8.5 (D6)
- net GND: now also E2.S1; no longer E2.S2
- no-connect marks 17 -> 18
Other:
- moved on the sheet: R50, R51, R52, R53, R54, R55, R56, R57
Changed lines of the file:
@@
 Wire Wire Line
 	3000 8650 3450 8650
-Wire Wire Line
-	3450 8150 3450 8650
-Connection ~ 3450 8650
-Wire Wire Line
-	3550 8150 3550 8750
-Connection ~ 3550 8750
-Wire Wire Line
-	3650 8150 3650 8850
-Connection ~ 3650 8850
-Wire Wire Line
-	3750 8150 3750 8950
-Connection ~ 3750 8950
 Text Label 15900 7200 2    50   ~ 0
 SER_LINK_1
@@
 Wire Wire Line
 	6100 8350 6400 8350
-Text Label 7300 8150 2    50   ~ 0
+Text Label 7300 8350 2    50   ~ 0
 E2_SW
 $Comp
@@
 $EndComp
 Wire Wire Line
-	7000 8150 7300 8150
+	7000 8350 7300 8350
 Wire Wire Line
 	6000 8250 6000 8550
@@
 	6000 8550 7000 8550
 Wire Wire Line
-	7000 8550 7000 8350
-Wire Wire Line
 	6000 8250 6400 8250
-Connection ~ 7000 8550
 $Comp
 L Device:Rotary_Encoder_Switch E3
@@
 Wire Wire Line
 	6000 9250 6400 9250
-Text Label 4150 8350 2    50   ~ 0
+Text Label 4150 8450 2    50   ~ 0
 E1_CLK
 Text Label 4150 8250 2    50   ~ 0
-E1_DIR
-Text Label 4150 8550 2    50   ~ 0
 E2_CLK
-Text Label 4150 8450 2    50   ~ 0
+Text Label 4150 8350 2    50   ~ 0
 E2_DIR
-Text Label 4150 8750 2    50   ~ 0
-E3_CLK
-Text Label 4150 8650 2    50   ~ 0
-E3_DIR
-Text Label 4150 8950 2    50   ~ 0
-E4_CLK
-Text Label 4150 8850 2    50   ~ 0
-E4_DIR
-Wire Wire Line
-	3450 8650 4150 8650
-Wire Wire Line
-	3550 8750 4150 8750
-Wire Wire Line
-	3650 8850 4150 8850
-Wire Wire Line
-	3750 8950 4150 8950
 Wire Wire Line
 	6000 9550 7000 9550
@@
 Wire Wire Line
 	3050 8150 3050 8250
-Connection ~ 3050 8250
-Wire Wire Line
-	3050 8250 4150 8250
 Wire Wire Line
 	3150 8150 3150 8350
-Connection ~ 3150 8350
-Wire Wire Line
-	3150 8350 4150 8350
 Wire Wire Line
 	3250 8150 3250 8450
-Connection ~ 3250 8450
-Wire Wire Line
-	3250 8450 4150 8450
 Wire Wire Line
 	3350 8150 3350 8550
-Connection ~ 3350 8550
-Wire Wire Line
-	3350 8550 4150 8550
 Wire Wire Line
 	3750 7750 3750 7850
@@
 Wire Wire Line
 	3350 7750 3450 7750
-Wire Wire Line
-	3250 7850 3250 7750
 Connection ~ 3250 7750
 Wire Wire Line
@@
 	15900 7200 15400 7200
 $Comp
-L Device:R R50
-U 1 1 5FC9A634
+L Device:R R51
+U 1 1 5FCF8D4C
+P 3250 8000
+F 0 "R51" V 3250 7650 50  0000 C CNN
+F 1 "10k" V 3250 8000 50  0000 C CNN
+F 2 "Resistor_SMD:R_0805_2012Metric_Pad1.15x1.40mm_HandSolder" V 3180 8000 50  0001 C CNN
+F 3 "~" H 3250 8000 50  0001 C CNN
+	1    3250 8000
+	-1   0    0    1
+$EndComp
+$Comp
+L Device:R R52
+U 1 1 5FCF907B
+P 3150 8000
+F 0 "R52" V 3150 7650 50  0000 C CNN
+F 1 "10k" V 3150 8000 50  0000 C CNN
+F 2 "Resistor_SMD:R_0805_2012Metric_Pad1.15x1.40mm_HandSolder" V 3080 8000 50  0001 C CNN
+F 3 "~" H 3150 8000 50  0001 C CNN
+	1    3150 8000
+	-1   0    0    1
+$EndComp
+$Comp
+L Device:R R53
+U 1 1 5FCF927C
 P 3050 8000
-F 0 "R50" V 3050 7650 50  0000 C CNN
+F 0 "R53" V 3050 7650 50  0000 C CNN
 F 1 "10k" V 3050 8000 50  0000 C CNN
 F 2 "Resistor_SMD:R_0805_2012Metric_Pad1.15x1.40mm_HandSolder" V 2980 8000 50  0001 C CNN
@@
 $EndComp
 $Comp
-L Device:R R51
-U 1 1 5FCF8D4C
-P 3150 8000
-F 0 "R51" V 3150 7650 50  0000 C CNN
-F 1 "10k" V 3150 8000 50  0000 C CNN
-F 2 "Resistor_SMD:R_0805_2012Metric_Pad1.15x1.40mm_HandSolder" V 3080 8000 50  0001 C CNN
-F 3 "~" H 3150 8000 50  0001 C CNN
-	1    3150 8000
-	-1   0    0    1
-$EndComp
-$Comp
-L Device:R R52
-U 1 1 5FCF907B
-P 3250 8000
-F 0 "R52" V 3250 7650 50  0000 C CNN
-F 1 "10k" V 3250 8000 50  0000 C CNN
-F 2 "Resistor_SMD:R_0805_2012Metric_Pad1.15x1.40mm_HandSolder" V 3180 8000 50  0001 C CNN
-F 3 "~" H 3250 8000 50  0001 C CNN
-	1    3250 8000
-	-1   0    0    1
-$EndComp
-$Comp
-L Device:R R53
-U 1 1 5FCF927C
-P 3350 8000
-F 0 "R53" V 3350 7650 50  0000 C CNN
-F 1 "10k" V 3350 8000 50  0000 C CNN
-F 2 "Resistor_SMD:R_0805_2012Metric_Pad1.15x1.40mm_HandSolder" V 3280 8000 50  0001 C CNN
-F 3 "~" H 3350 8000 50  0001 C CNN
-	1    3350 8000
-	-1   0    0    1
-$EndComp
-$Comp
 L Device:R R54
 U 1 1 5FCF9481
+P 3750 8000
+F 0 "R54" V 3750 7650 50  0000 C CNN
+F 1 "10k" V 3750 8000 50  0000 C CNN
+F 2 "Resistor_SMD:R_0805_2012Metric_Pad1.15x1.40mm_HandSolder" V 3680 8000 50  0001 C CNN
+F 3 "~" H 3750 8000 50  0001 C CNN
+	1    3750 8000
+	-1   0    0    1
+$EndComp
+$Comp
+L Device:R R55
+U 1 1 5FCF96F4
+P 3650 8000
+F 0 "R55" V 3650 7650 50  0000 C CNN
+F 1 "10k" V 3650 8000 50  0000 C CNN
+F 2 "Resistor_SMD:R_0805_2012Metric_Pad1.15x1.40mm_HandSolder" V 3580 8000 50  0001 C CNN
+F 3 "~" H 3650 8000 50  0001 C CNN
+	1    3650 8000
+	-1   0    0    1
+$EndComp
+$Comp
+L Device:R R56
+U 1 1 5FCF9B90
+P 3550 8000
+F 0 "R56" V 3550 7650 50  0000 C CNN
+F 1 "10k" V 3550 8000 50  0000 C CNN
+F 2 "Resistor_SMD:R_0805_2012Metric_Pad1.15x1.40mm_HandSolder" V 3480 8000 50  0001 C CNN
+F 3 "~" H 3550 8000 50  0001 C CNN
+	1    3550 8000
+	-1   0    0    1
+$EndComp
+$Comp
+L Device:R R57
+U 1 1 5FCF9DA1
 P 3450 8000
-F 0 "R54" V 3450 7650 50  0000 C CNN
+F 0 "R57" V 3450 7650 50  0000 C CNN
 F 1 "10k" V 3450 8000 50  0000 C CNN
 F 2 "Resistor_SMD:R_0805_2012Metric_Pad1.15x1.40mm_HandSolder" V 3380 8000 50  0001 C CNN
@@
 	-1   0    0    1
 $EndComp
-$Comp
-L Device:R R55
-U 1 1 5FCF96F4
-P 3550 8000
-F 0 "R55" V 3550 7650 50  0000 C CNN
-F 1 "10k" V 3550 8000 50  0000 C CNN
-F 2 "Resistor_SMD:R_0805_2012Metric_Pad1.15x1.40mm_HandSolder" V 3480 8000 50  0001 C CNN
-F 3 "~" H 3550 8000 50  0001 C CNN
-	1    3550 8000
-	-1   0    0    1
-$EndComp
-$Comp
-L Device:R R56
-U 1 1 5FCF9B90
-P 3650 8000
-F 0 "R56" V 3650 7650 50  0000 C CNN
-F 1 "10k" V 3650 8000 50  0000 C CNN
-F 2 "Resistor_SMD:R_0805_2012Metric_Pad1.15x1.40mm_HandSolder" V 3580 8000 50  0001 C CNN
-F 3 "~" H 3650 8000 50  0001 C CNN
-	1    3650 8000
-	-1   0    0    1
-$EndComp
-$Comp
-L Device:R R57
-U 1 1 5FCF9DA1
-P 3750 8000
-F 0 "R57" V 3750 7650 50  0000 C CNN
-F 1 "10k" V 3750 8000 50  0000 C CNN
-F 2 "Resistor_SMD:R_0805_2012Metric_Pad1.15x1.40mm_HandSolder" V 3680 8000 50  0001 C CNN
-F 3 "~" H 3750 8000 50  0001 C CNN
-	1    3750 8000
-	-1   0    0    1
-$EndComp
-Wire Wire Line
-	3050 7850 3050 7750
 Connection ~ 3050 7750
 Wire Wire Line
@@
 MODE_SW
 Wire Wire Line
-	3550 2800 4500 2800
-Wire Wire Line
-	3550 2700 4500 2700
+	3550 2600 4500 2600
+Wire Wire Line
+	3550 2500 4500 2500
 Text Label 4500 2200 2    50   ~ 0
 E3_SW
 Text Label 4500 3300 2    50   ~ 0
 E4_SW
-Text Label 4500 2800 2    50   ~ 0
+Text Label 4500 2600 2    50   ~ 0
 E2_SW
-Text Label 4500 2700 2    50   ~ 0
+Text Label 4500 2500 2    50   ~ 0
 E1_SW
 Wire Wire Line
@@
 Text Label 15900 6400 2    50   ~ 0
 SER_MOSI
-Text Label 1300 8250 0    50   ~ 0
-SER_IN
 Text Notes 3600 1800 0    50   ~ 0
 D12(MISO)
@@
 	0    1    1    0
 $EndComp
-NoConn ~ 3550 2500
-NoConn ~ 3550 2600
 NoConn ~ 3550 3400
 Text Label 4500 1800 2    50   ~ 0
@@
 NoConn ~ 3550 2900
 NoConn ~ 3550 3100
+Text Label 4150 8550 2    50   ~ 0
+E1_DIR
+Text Label 4150 8750 2    50   ~ 0
+E4_DIR
+Text Label 4150 8650 2    50   ~ 0
+E4_CLK
+Text Label 4150 8950 2    50   ~ 0
+E3_DIR
+Text Label 4150 8850 2    50   ~ 0
+E3_CLK
+Wire Wire Line
+	3450 8150 3450 8250
+Wire Wire Line
+	3550 8150 3550 8350
+Wire Wire Line
+	3750 8150 3750 8550
+Wire Wire Line
+	3650 8150 3650 8450
+Connection ~ 3050 8250
+Wire Wire Line
+	3450 8250 3450 8650
+Connection ~ 3150 8350
+Wire Wire Line
+	3550 8350 3550 8750
+Connection ~ 3250 8450
+Wire Wire Line
+	3650 8450 3650 8850
+Connection ~ 3350 8550
+Wire Wire Line
+	3750 8550 3750 8950
+Wire Wire Line
+	3250 8450 4150 8450
+Wire Wire Line
+	3350 8550 4150 8550
+Wire Wire Line
+	3150 8350 4150 8350
+Wire Wire Line
+	3050 8250 4150 8250
+Wire Wire Line
+	3450 8650 4150 8650
+Connection ~ 3450 8650
+Wire Wire Line
+	4150 8750 3550 8750
+Connection ~ 3550 8750
+Wire Wire Line
+	3650 8850 4150 8850
+Connection ~ 3650 8850
+Wire Wire Line
+	4150 8950 3750 8950
+Connection ~ 3750 8950
+Wire Wire Line
+	3250 7850 3250 7750
+$Comp
+L Device:R R50
+U 1 1 5FC9A634
+P 3350 8000
+F 0 "R50" V 3350 7650 50  0000 C CNN
+F 1 "10k" V 3350 8000 50  0000 C CNN
+F 2 "Resistor_SMD:R_0805_2012Metric_Pad1.15x1.40mm_HandSolder" V 3280 8000 50  0001 C CNN
+F 3 "~" H 3350 8000 50  0001 C CNN
+	1    3350 8000
+	-1   0    0    1
+$EndComp
+Wire Wire Line
+	3050 7750 3050 7850
+NoConn ~ 3550 2700
+NoConn ~ 3550 2800
+NoConn ~ 2000 8350
+Text Label 1300 8250 0    50   ~ 0
+SER_MISO
+Connection ~ 7000 8550
+Wire Wire Line
+	7400 8150 7400 8550
+Wire Wire Line
+	7400 8550 7000 8550
+Wire Wire Line
+	7000 8150 7400 8150
 $EndSCHEMATC

Commit message: Add comments from design review
Parts:
- C4, C5, C6, C7, C8, C9: value 0.1uF -> 1uF
Other:
- note added: "Encoder Readback"
- note removed: "Encoder Multiplexing"
- moved on the sheet: TP1, TP2
Changed lines of the file:
@@
 EESchema Schematic File Version 4
-LIBS:mtg_life_counter-cache
 EELAYER 30 0
 EELAYER END
@@
 $EndComp
 $Comp
-L power:GND #PWR026
-U 1 1 5F2E233A
-P 5050 10050
-F 0 "#PWR026" H 5050 9800 50  0001 C CNN
-F 1 "GND" H 5055 9877 50  0000 C CNN
-F 2 "" H 5050 10050 50  0001 C CNN
-F 3 "" H 5050 10050 50  0001 C CNN
-	1    5050 10050
-	1    0    0    -1
-$EndComp
-Wire Wire Line
-	4550 10050 5050 10050
-Wire Wire Line
-	5050 9750 5050 10050
-Connection ~ 5050 10050
-$Comp
 L power:+5V #PWR023
 U 1 1 5F2E3AF9
@@
 P 9100 6600
 F 0 "C6" V 8950 6600 50  0000 C CNN
-F 1 "0.1uF" V 9000 6800 50  0000 C CNN
+F 1 "1uF" V 9000 6800 50  0000 C CNN
 F 2 "Capacitor_SMD:C_0805_2012Metric_Pad1.15x1.40mm_HandSolder" H 9100 6600 50  0001 C CNN
 F 3 "~" H 9100 6600 50  0001 C CNN
@@
 P 9100 2750
 F 0 "C4" V 8950 2750 50  0000 C CNN
-F 1 "0.1uF" V 9000 2950 50  0000 C CNN
+F 1 "1uF" V 9000 2950 50  0000 C CNN
 F 2 "Capacitor_SMD:C_0805_2012Metric_Pad1.15x1.40mm_HandSolder" H 9100 2750 50  0001 C CNN
 F 3 "~" H 9100 2750 50  0001 C CNN
@@
 	8700 2150 9400 2150
 Text Notes 4300 7650 0    100  ~ 20
-Encoder Multiplexing
+Encoder Readback
 Text Label 15900 6600 2    50   ~ 0
 SER_CLK
@@
 P 15100 6100
 F 0 "C9" V 14871 6100 50  0000 C CNN
-F 1 "0.1uF" V 14962 6100 50  0000 C CNN
+F 1 "1uF" V 14962 6100 50  0000 C CNN
 F 2 "Capacitor_SMD:C_0805_2012Metric_Pad1.15x1.40mm_HandSolder" H 15100 6100 50  0001 C CNN
 F 3 "~" H 15100 6100 50  0001 C CNN
@@
 P 15100 2250
 F 0 "C8" V 14871 2250 50  0000 C CNN
-F 1 "0.1uF" V 14962 2250 50  0000 C CNN
+F 1 "1uF" V 14962 2250 50  0000 C CNN
 F 2 "Capacitor_SMD:C_0805_2012Metric_Pad1.15x1.40mm_HandSolder" H 15100 2250 50  0001 C CNN
 F 3 "~" H 15100 2250 50  0001 C CNN
@@
 P 9100 4600
 F 0 "C5" V 8950 4600 50  0000 C CNN
-F 1 "0.1uF" V 9000 4800 50  0000 C CNN
+F 1 "1uF" V 9000 4800 50  0000 C CNN
 F 2 "Capacitor_SMD:C_0805_2012Metric_Pad1.15x1.40mm_HandSolder" H 9100 4600 50  0001 C CNN
 F 3 "~" H 9100 4600 50  0001 C CNN
@@
 P 9100 8600
 F 0 "C7" V 8950 8600 50  0000 C CNN
-F 1 "0.1uF" V 9000 8800 50  0000 C CNN
+F 1 "1uF" V 9000 8800 50  0000 C CNN
 F 2 "Capacitor_SMD:C_0805_2012Metric_Pad1.15x1.40mm_HandSolder" H 9100 8600 50  0001 C CNN
 F 3 "~" H 9100 8600 50  0001 C CNN
@@
 L Connector:TestPoint TP2
 U 1 1 60642369
-P 4500 3800
-F 0 "TP2" V 4500 4000 50  0000 L CNN
-F 1 "RX" V 4500 4200 50  0000 L CNN
-F 2 "TestPoint:TestPoint_Pad_D1.5mm" H 4700 3800 50  0001 C CNN
-F 3 "~" H 4700 3800 50  0001 C CNN
-	1    4500 3800
+P 6400 1600
+F 0 "TP2" V 6400 1800 50  0000 L CNN
+F 1 "RX" V 6400 2000 50  0000 L CNN
+F 2 "TestPoint:TestPoint_Pad_D1.5mm" H 6600 1600 50  0001 C CNN
+F 3 "~" H 6600 1600 50  0001 C CNN
+	1    6400 1600
 	0    1    1    0
 $EndComp
@@
 L Connector:TestPoint TP1
 U 1 1 60642AD4
-P 4500 3700
-F 0 "TP1" V 4500 3900 50  0000 L CNN
-F 1 "TX" V 4500 4100 50  0000 L CNN
-F 2 "TestPoint:TestPoint_Pad_D1.5mm" H 4700 3700 50  0001 C CNN
-F 3 "~" H 4700 3700 50  0001 C CNN
-	1    4500 3700
+P 6400 1450
+F 0 "TP1" V 6400 1650 50  0000 L CNN
+F 1 "TX" V 6400 1850 50  0000 L CNN
+F 2 "TestPoint:TestPoint_Pad_D1.5mm" H 6600 1450 50  0001 C CNN
+F 3 "~" H 6600 1450 50  0001 C CNN
+	1    6400 1450
 	0    1    1    0
 $EndComp
@@
 Wire Wire Line
 	7000 8150 7400 8150
+Text Label 5900 1600 0    50   ~ 0
+D0(RX)
+Text Label 5900 1450 0    50   ~ 0
+D1(TX)
+Wire Wire Line
+	5900 1450 6400 1450
+Wire Wire Line
+	6400 1600 5900 1600
+Wire Notes Line
+	14400 3800 14400 3000
+Wire Notes Line
+	14400 3000 9400 3000
+Wire Notes Line
+	9400 3000 9400 2800
+Wire Notes Line
+	14400 3800 15000 3800
 $EndSCHEMATC
