File: pcb/mtg_life_counter.sch (KiCad schematic (older format))
At the start: 84 parts, among them J1 USB_C_Receptacle_USB2.0, J2 ICSP, SW1 SW_SPST, SW2 SW_SPST, U1 ATmega328P-AU, U2 74HC595, U3 74HC595, U4 74HC595, U5 74HC595, U6 TPIC6B595, U7 TPIC6B595, U8 74HC165, Y1 16MHz

Commit message: Switch to SMD 7segs
Parts:
- removed D1: KW4-566CVB RED, mtg_life_counter:KW4-566xxB_THT, symbol mtg_life_counter:KW4-566CxB
- removed D2: KW4-566CVB GREEN, mtg_life_counter:KW4-566xxB_THT, symbol mtg_life_counter:KW4-566CxB
- removed D3: KW4-566CVB YELLOW, mtg_life_counter:KW4-566xxB_THT, symbol mtg_life_counter:KW4-566CxB
- removed D4: KW4-566CVB BLUE, mtg_life_counter:KW4-566xxB_THT, symbol mtg_life_counter:KW4-566CxB
- added D1: KW4-S561CxB RED SMD, mtg_life_counter:KW4-S561xxB_SMD, symbol mtg_life_counter:KW4-S561CxB
- added D2: KW4-S561CxB GREEN SMD, mtg_life_counter:KW4-S561xxB_SMD, symbol mtg_life_counter:KW4-S561CxB
- added D3: KW4-S561CxB YELLOW SMD, mtg_life_counter:KW4-S561xxB_SMD, symbol mtg_life_counter:KW4-S561CxB
- added D4: KW4-S561CxB BLUE SMD, mtg_life_counter:KW4-S561xxB_SMD, symbol mtg_life_counter:KW4-S561CxB
Connections:
- net GND: no longer U2.13 (~OE), U3.13 (~OE), U4.13 (~OE), U5.13 (~OE), U6.9 (~G), U7.9 (~G), U8.15 (~CEN)
- net at R40.2: now also D4.11 (a)
- net at R41.2: now also D4.7 (b)
- net at R42.2: now also D4.4 (c)
- net at R43.2: now also D4.2 (d)
- net at R44.2: now also D4.1 (e)
- net at R45.2: now also D4.10 (f)
- net at R46.2: now also D4.5 (g)
- net at R47.2: now also D4.3 (DP)
- net at U6.14 (DRAIN4): now also D2.12 (CC1)
- net at U6.15 (DRAIN5): now also D2.9 (CC2)
- net at U6.16 (DRAIN6): now also D2.8 (CC3)
- net at U6.17 (DRAIN7): now also D2.6 (CC4)
- net at U6.4 (DRAIN0): now also D1.12 (CC1)
- net at U6.5 (DRAIN1): now also D1.9 (CC2)
- net at U6.6 (DRAIN2): now also D1.8 (CC3)
- net at U6.7 (DRAIN3): now also D1.6 (CC4)
- net at U7.14 (DRAIN4): now also D4.12 (CC1)
- net at U7.15 (DRAIN5): now also D4.9 (CC2)
- net at U7.16 (DRAIN6): now also D4.8 (CC3)
- net at U7.17 (DRAIN7): now also D4.6 (CC4)
- net at U7.4 (DRAIN0): now also D3.12 (CC1)
- net at U7.5 (DRAIN1): now also D3.9 (CC2)
- net at U7.6 (DRAIN2): now also D3.8 (CC3)
- net at U7.7 (DRAIN3): now also D3.6 (CC4)
- net at R30.2: now also D3.11 (a)
- net at R31.2: now also D3.7 (b)
- net at R32.2: now also D3.4 (c)
- net at R33.2: now also D3.2 (d)
- net at R34.2: now also D3.1 (e)
- net at R35.2: now also D3.10 (f)
- net at R36.2: now also D3.5 (g)
- net at R37.2: now also D3.3 (DP)
- net at R20.2: now also D2.11 (a)
- net at R21.2: now also D2.7 (b)
- net at R22.2: now also D2.4 (c)
- net at R23.2: now also D2.2 (d)
- net at R24.2: now also D2.1 (e)
- net at R25.2: now also D2.10 (f)
- net at R26.2: now also D2.5 (g)
- net at R27.2: now also D2.3 (DP)
- net at R10.2: now also D1.11 (a)
- net at R11.2: now also D1.7 (b)
- net at R12.2: now also D1.4 (c)
- net at R13.2: now also D1.2 (d)
- net at R14.2: now also D1.1 (e)
- net at R15.2: now also D1.10 (f)
- net at R16.2: now also D1.5 (g)
- net at R17.2: now also D1.3 (DP)
- new net ~ENABLE: U2.13 (~OE), U3.13 (~OE), U4.13 (~OE), U5.13 (~OE), U6.9 (~G), U7.9 (~G), U8.15 (~CEN)
Changed lines of the file:
@@
 EESchema Schematic File Version 4
+LIBS:mtg_life_counter-cache
 EELAYER 30 0
 EELAYER END
@@
 	-1   0    0    -1
 $EndComp
-Text Label 14800 4950 0    50   ~ 0
-~ENABLE
 Wire Wire Line
 	15100 3650 15000 3650
@@
 Text Notes 11850 1300 0    100  ~ 20
 Seven Segement Displays
-$Comp
-L mtg_life_counter:KW4-566CxB D2
-U 1 1 60A3B26F
-P 12800 4050
-F 0 "D2" H 12800 4667 50  0000 C CNN
-F 1 "KW4-566CVB GREEN" H 12800 4576 50  0000 C CNN
-F 2 "mtg_life_counter:KW4-566xxB_THT" H 12800 3550 50  0001 C CNN
-F 3 "" H 12370 4080 50  0001 C CNN
-	1    12800 4050
-	1    0    0    -1
-$EndComp
-$Comp
-L mtg_life_counter:KW4-566CxB D1
-U 1 1 60A35AC0
-P 12800 2200
-F 0 "D1" H 12800 2817 50  0000 C CNN
-F 1 "KW4-566CVB RED" H 12800 2726 50  0000 C CNN
-F 2 "mtg_life_counter:KW4-566xxB_THT" H 12800 1700 50  0001 C CNN
-F 3 "" H 12370 2230 50  0001 C CNN
-	1    12800 2200
-	1    0    0    -1
-$EndComp
 Wire Wire Line
 	14000 2350 13900 2350
@@
 Wire Wire Line
 	13900 4100 14200 4100
-$Comp
-L mtg_life_counter:KW4-566CxB D3
-U 1 1 60C9EF14
-P 12800 6050
-F 0 "D3" H 12800 6667 50  0000 C CNN
-F 1 "KW4-566CVB YELLOW" H 12800 6576 50  0000 C CNN
-F 2 "mtg_life_counter:KW4-566xxB_THT" H 12800 5550 50  0001 C CNN
-F 3 "" H 12370 6080 50  0001 C CNN
-	1    12800 6050
-	1    0    0    -1
-$EndComp
-$Comp
-L mtg_life_counter:KW4-566CxB D4
-U 1 1 60CC9F0E
-P 12800 8050
-F 0 "D4" H 12800 8667 50  0000 C CNN
-F 1 "KW4-566CVB BLUE" H 12800 8576 50  0000 C CNN
-F 2 "mtg_life_counter:KW4-566xxB_THT" H 12800 7550 50  0001 C CNN
-F 3 "" H 12370 8080 50  0001 C CNN
-	1    12800 8050
-	1    0    0    -1
-$EndComp
 Wire Wire Line
 	13900 6200 14000 6200
@@
 Wire Wire Line
 	13900 8200 14300 8200
-$Comp
-L power:GND #PWR0136
-U 1 1 610D747B
-P 15300 4950
-F 0 "#PWR0136" H 15300 4700 50  0001 C CNN
-F 1 "GND" H 15305 4777 50  0000 C CNN
-F 2 "" H 15300 4950 50  0001 C CNN
-F 3 "" H 15300 4950 50  0001 C CNN
-	1    15300 4950
-	1    0    0    -1
-$EndComp
-Wire Wire Line
-	14800 4950 15300 4950
 Wire Wire Line
 	7300 9350 7000 9350
@@
 Text Notes 3600 1800 0    50   ~ 0
 D12(MISO)
-Text Label 1300 8650 0    50   ~ 0
+Text Label 1500 8650 0    50   ~ 0
 SER_LATCH
 $Comp
@@
 Wire Wire Line
 	2500 9250 2500 9350
-Connection ~ 2500 9250
-Text Label 1300 8850 0    50   ~ 0
+Text Label 1500 8850 0    50   ~ 0
 SER_CLK
 Wire Wire Line
-	1300 8850 2000 8850
-Wire Wire Line
-	1300 8250 2000 8250
-Wire Wire Line
-	1300 8650 2000 8650
-Wire Wire Line
-	2000 8550 1900 8550
-Wire Wire Line
-	1900 8550 1900 8950
-Wire Wire Line
-	2000 8950 1900 8950
-Connection ~ 1900 8950
-Wire Wire Line
-	1900 8950 1900 9250
-Wire Wire Line
-	1900 9250 2500 9250
+	1500 8850 2000 8850
+Wire Wire Line
+	1500 8250 2000 8250
+Wire Wire Line
+	1500 8650 2000 8650
 $Comp
 L Connector:TestPoint TP2
@@
 NoConn ~ 3550 2800
 NoConn ~ 2000 8350
-Text Label 1300 8250 0    50   ~ 0
+Text Label 1500 8250 0    50   ~ 0
 SER_MISO
 Connection ~ 7000 8550
@@
 Wire Wire Line
 	6400 1600 5900 1600
-Wire Notes Line
-	14400 3800 14400 3000
-Wire Notes Line
-	14400 3000 9400 3000
-Wire Notes Line
-	9400 3000 9400 2800
-Wire Notes Line
-	14400 3800 15000 3800
+$Comp
+L mtg_life_counter:KW4-S561CxB D1
+U 1 1 61A0F869
+P 12800 2200
+F 0 "D1" H 12800 2817 50  0000 C CNN
+F 1 "KW4-S561CxB RED SMD" H 12800 2726 50  0000 C CNN
+F 2 "mtg_life_counter:KW4-S561xxB_SMD" H 12800 1700 50  0001 C CNN
+F 3 "" H 12370 2230 50  0001 C CNN
+	1    12800 2200
+	1    0    0    -1
+$EndComp
+$Comp
+L mtg_life_counter:KW4-S561CxB D2
+U 1 1 61A171D8
+P 12800 4050
+F 0 "D2" H 12800 4667 50  0000 C CNN
+F 1 "KW4-S561CxB GREEN SMD" H 12800 4576 50  0000 C CNN
+F 2 "mtg_life_counter:KW4-S561xxB_SMD" H 12800 3550 50  0001 C CNN
+F 3 "" H 12370 4080 50  0001 C CNN
+	1    12800 4050
+	1    0    0    -1
+$EndComp
+$Comp
+L mtg_life_counter:KW4-S561CxB D3
+U 1 1 61A185C0
+P 12800 6050
+F 0 "D3" H 12800 6667 50  0000 C CNN
+F 1 "KW4-S561CxB YELLOW SMD" H 12800 6576 50  0000 C CNN
+F 2 "mtg_life_counter:KW4-S561xxB_SMD" H 12800 5550 50  0001 C CNN
+F 3 "" H 12370 6080 50  0001 C CNN
+	1    12800 6050
+	1    0    0    -1
+$EndComp
+$Comp
+L mtg_life_counter:KW4-S561CxB D4
+U 1 1 61A1971E
+P 12800 8050
+F 0 "D4" H 12800 8667 50  0000 C CNN
+F 1 "KW4-S561CxB BLUE SMD" H 12800 8576 50  0000 C CNN
+F 2 "mtg_life_counter:KW4-S561xxB_SMD" H 12800 7550 50  0001 C CNN
+F 3 "" H 12370 8080 50  0001 C CNN
+	1    12800 8050
+	1    0    0    -1
+$EndComp
+Text Label 1500 8950 0    50   ~ 0
+~ENABLE
+Wire Wire Line
+	2000 8950 1500 8950
+$Comp
+L power:GND #PWR?
+U 1 1 61BA45A0
+P 1250 8550
+F 0 "#PWR?" H 1250 8300 50  0001 C CNN
+F 1 "GND" H 1255 8377 50  0000 C CNN
+F 2 "" H 1250 8550 50  0001 C CNN
+F 3 "" H 1250 8550 50  0001 C CNN
+	1    1250 8550
+	1    0    0    -1
+$EndComp
+Wire Wire Line
+	1250 8550 2000 8550
 $EndSCHEMATC

Commit message: Complete layout. Use new USB-C connector
Parts:
- removed J1: USB_C_Receptacle_USB2.0, Connector_USB:USB_C_Receptacle_GCT_USB4085, symbol mtg_life_counter-rescue:USB_C_Receptacle_USB2.0-Connector
- removed TP4: Debug, TestPoint:TestPoint_Pad_D1.5mm, symbol Connector:TestPoint
- added C11, C12: 1uF, Capacitor_SMD:C_0805_2012Metric_Pad1.15x1.40mm_HandSolder, symbol Device:C_Small
- added J1: USB C 4907, mtg_life_counter:4907_USB_C_PowerOnly, symbol mtg_life_counter:USB_C_Receptacle_USB2.0-Connector
- added JP1: Jumper_2_Open, Jumper:SolderJumper-2_P1.3mm_Open_TrianglePad1.0x1.5mm, symbol Jumper:Jumper_2_Open
- added R4: 10k, Resistor_SMD:R_0805_2012Metric_Pad1.15x1.40mm_HandSolder, symbol Device:R
- added R5, R6: 5.1k, Resistor_SMD:R_0805_2012Metric_Pad1.15x1.40mm_HandSolder, symbol Device:R
- C4, C5, C6, C7, C8, C9: value 1uF -> 0.1uF
- R1: value 1k -> 10k
- R20, R21, R22, R23, R24, R25, R26, R27: value 33 -> 10
- TP1, TP2: footprint TestPoint:TestPoint_Pad_D1.5mm -> TestPoint:TestPoint_Keystone_5015_Micro-Minature
- TP3: value INT0 -> GND; footprint TestPoint:TestPoint_Pad_D1.5mm -> TestPoint:TestPoint_Keystone_5015_Micro-Minature
Connections:
- net DEBUG_PIN is gone; now on net E1_SW: U1.28 (PC5(SCL/ADC5))
- net ~ENABLE is gone; now on net GND: U2.13 (~OE), U3.13 (~OE), U4.13 (~OE), U5.13 (~OE), U6.9 (~G), U7.9 (~G), U8.15 (~CEN)
- net +5V: now also R4.1
- net E1_CLK: now also R50.1, U8.14 (D3); no longer R51.1, U8.13 (D2)
- net E1_DIR: now also R51.1, U8.13 (D2); no longer R50.1, U8.14 (D3)
- net E1_SW: no longer U1.27 (PC4(SDA/ADC4))
- net E2_CLK: now also R52.1, U8.12 (D1); no longer R53.1, U8.11 (D0)
- net E2_DIR: now also R53.1, U8.11 (D0); no longer R52.1, U8.12 (D1)
- net E2_SW: now also U1.25 (PC2(ADC2)); no longer U1.26 (PC3(ADC3))
- net E3_CLK: now also R54.1, U8.6 (D7); no longer R55.1, U8.5 (D6)
- net E3_DIR: now also R55.1, U8.5 (D6); no longer R54.1, U8.6 (D7)
- net E3_SW: now also E3.S1, U1.9 (PD5); no longer E3.S2, U1.12 (PB0(ICP))
- net E4_CLK: now also R56.1, U8.4 (D5); no longer R57.1, U8.3 (D4)
- net E4_DIR: now also R57.1, U8.3 (D4); no longer R56.1, U8.4 (D5)
- net E4_SW: now also U1.1 (PD3(INT1)); no longer U1.9 (PD5)
- net GND: now also E3.S2, TP3.1, C11.1, C12.1, J1.A12 (GND), J1.B12 (GND), R5.2, R6.2; no longer E3.S1, H1.1, H2.1, H3.1, H4.1
- net RESET_BTN: now also U1.12 (PB0(ICP)); no longer U1.1 (PD3(INT1))
- net ROLL_BTN: now also U1.11 (PD7); no longer U1.10 (PD6)
- net SER_LATCH: now also R4.2
- net SER_MISO: now also JP1.2 (B); no longer U8.9 (Q7)
- net VBUS: now also C11.2, C12.2, J1.A9 (VBUS), J1.B9 (VBUS)
- net D2(INT0): no longer names the net of U1.32 (PD2(INT0))
- net D2(INT0): no longer TP3.1
- new net: J1.A5 (CC1), R5.1
- new net: J1.B5 (CC2), R6.1
- new net SR_OUT: JP1.1 (A), U8.9 (Q7)
- no-connect marks 18 -> 16
Other:
- moved on the sheet: SW1

Commit message: Tweak encoder footprint. Add more via stitching
Parts:
- E1, E2, E3, E4: footprint Rotary_Encoder:RotaryEncoder_Alps_EC11E-Switch_Vertical_H20mm -> mtg_life_counter:TT_EN11-HSB
Changed lines of the file:
@@
 EESchema Schematic File Version 4
-LIBS:mtg_life_counter-cache
 EELAYER 30 0
 EELAYER END
@@
 F 0 "E1" H 5200 8617 50  0000 C CNN
 F 1 "Rotary_Encoder_Switch" H 5200 8526 50  0000 C CNN
-F 2 "Rotary_Encoder:RotaryEncoder_Alps_EC11E-Switch_Vertical_H20mm" H 5050 8410 50  0001 C CNN
+F 2 "mtg_life_counter:TT_EN11-HSB" H 5050 8410 50  0001 C CNN
 F 3 "~" H 5200 8510 50  0001 C CNN
 	1    5200 8250
@@
 F 0 "E2" H 6700 8617 50  0000 C CNN
 F 1 "Rotary_Encoder_Switch" H 6700 8526 50  0000 C CNN
-F 2 "Rotary_Encoder:RotaryEncoder_Alps_EC11E-Switch_Vertical_H20mm" H 6550 8410 50  0001 C CNN
+F 2 "mtg_life_counter:TT_EN11-HSB" H 6550 8410 50  0001 C CNN
 F 3 "~" H 6700 8510 50  0001 C CNN
 	1    6700 8250
@@
 F 0 "E3" H 5200 9617 50  0000 C CNN
 F 1 "Rotary_Encoder_Switch" H 5200 9526 50  0000 C CNN
-F 2 "Rotary_Encoder:RotaryEncoder_Alps_EC11E-Switch_Vertical_H20mm" H 5050 9410 50  0001 C CNN
+F 2 "mtg_life_counter:TT_EN11-HSB" H 5050 9410 50  0001 C CNN
 F 3 "~" H 5200 9510 50  0001 C CNN
 	1    5200 9250
@@
 F 0 "E4" H 6700 9617 50  0000 C CNN
 F 1 "Rotary_Encoder_Switch" H 6700 9526 50  0000 C CNN
-F 2 "Rotary_Encoder:RotaryEncoder_Alps_EC11E-Switch_Vertical_H20mm" H 6550 9410 50  0001 C CNN
+F 2 "mtg_life_counter:TT_EN11-HSB" H 6550 9410 50  0001 C CNN
 F 3 "~" H 6700 9510 50  0001 C CNN
 	1    6700 9250

Commit message: Begin updating firmware to match new hardware
Other:
- note added: "TODO: Confirm latch pull-up/down direction"
Changed lines of the file:
@@
 NoConn ~ 4850 5650
 NoConn ~ 5100 5650
+Text Notes 600  4400 0    50   ~ 0
+TODO: Confirm latch pull-up/down direction
 $EndSCHEMATC
