File: pcb/mtg_life_counter.sch (KiCad schematic (older format))
At the start: 89 parts, among them J1 USB C 4907, J2 ICSP, SW1 SW_SPST, SW2 SW_SPST, U1 ATmega328P-AU, U2 74HC595, U3 74HC595, U4 74HC595, U5 74HC595, U6 TPIC6B595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

Commit message: Separate display and encoder latch lines
Parts:
- added R2: 10k, Resistor_SMD:R_0805_2012Metric_Pad1.15x1.40mm_HandSolder, symbol Device:R
- renumbered R4 to R3, R2 to R4, R3 to R5, R5 to R60, R6 to R61
Connections:
- net +5V: now also R2.1; no longer R3.1
- net E4_SW: now also U1.32 (PD2(INT0)); no longer U1.1 (PD3(INT1))
- net GND: now also R3.1
- net SER_LATCH renamed DISP_LATCH
- net DISP_LATCH: no longer U8.1 (~LOAD)
- new net ENC_LATCH: R2.2, U1.1 (PD3(INT1)), U8.1 (~LOAD)
- no-connect marks 16 -> 15
Changed lines of the file:
@@
 Text Label 10700 8600 2    50   ~ 0
 SER_LINK_3
-Text Label 8900 6200 0    50   ~ 0
-SER_LATCH
 Wire Wire Line
 	8900 6200 9400 6200
-Text Label 8900 2350 0    50   ~ 0
-SER_LATCH
 Wire Wire Line
 	8900 2350 9400 2350
@@
 Wire Wire Line
 	15400 6600 15900 6600
-Text Label 15900 6900 2    50   ~ 0
-SER_LATCH
 Wire Wire Line
 	15900 6900 15400 6900
@@
 	15900 7000 15400 7000
 $Comp
-L Device:R R3
+L Device:R R5
 U 1 1 617ED900
 P 15700 6700
-F 0 "R3" V 15700 6300 50  0000 C CNN
+F 0 "R5" V 15700 6300 50  0000 C CNN
 F 1 "10k" V 15700 6700 50  0000 C CNN
 F 2 "Resistor_SMD:R_0805_2012Metric_Pad1.15x1.40mm_HandSolder" V 15630 6700 50  0001 C CNN
@@
 Wire Wire Line
 	15400 2750 15900 2750
-Text Label 15900 3050 2    50   ~ 0
-SER_LATCH
 Wire Wire Line
 	15900 3050 15400 3050
@@
 	15900 3150 15400 3150
 $Comp
-L Device:R R2
+L Device:R R4
 U 1 1 5F968430
 P 15700 2850
-F 0 "R2" V 15700 2450 50  0000 C CNN
+F 0 "R4" V 15700 2450 50  0000 C CNN
 F 1 "10k" V 15700 2850 50  0000 C CNN
 F 2 "Resistor_SMD:R_0805_2012Metric_Pad1.15x1.40mm_HandSolder" V 15630 2850 50  0001 C CNN
@@
 Wire Wire Line
 	8900 7900 9400 7900
-Text Label 8900 8200 0    50   ~ 0
-SER_LATCH
 Wire Wire Line
 	8900 8200 9400 8200
@@
 Wire Wire Line
 	8900 3900 9400 3900
-Text Label 8900 4200 0    50   ~ 0
-SER_LATCH
 Wire Wire Line
 	8900 4200 9400 4200
@@
 $EndComp
 Wire Wire Line
-	3550 3500 4500 3500
+	3550 3600 4500 3600
 Text Label 4500 2200 2    50   ~ 0
 RESET_BTN
@@
 	3550 2000 4500 2000
 Text Label 4500 2000 2    50   ~ 0
-SER_LATCH
+DISP_LATCH
 Wire Wire Line
 	3550 2100 4500 2100
@@
 Text Label 4500 3300 2    50   ~ 0
 E3_SW
-Text Label 4500 3500 2    50   ~ 0
+Text Label 4500 3600 2    50   ~ 0
 E4_SW
 Text Label 4500 2700 2    50   ~ 0
@@
 D12(MISO)
 Text Label 1500 8650 0    50   ~ 0
-SER_LATCH
+ENC_LATCH
 $Comp
 L mtg_life_counter:74HC165 U8
@@
 NoConn ~ 3550 2500
 $Comp
-L Device:R R4
+L Device:R R3
 U 1 1 62408EA5
 P 1150 4200
-F 0 "R4" V 1250 4200 50  0000 C CNN
+F 0 "R3" V 1250 4200 50  0000 C CNN
 F 1 "10k" V 1150 4200 50  0000 C CNN
 F 2 "Resistor_SMD:R_0805_2012Metric_Pad1.15x1.40mm_HandSolder" V 1080 4200 50  0001 C CNN
@@
 	0    -1   -1   0
 $EndComp
-Text Label 1800 4200 2    50   ~ 0
-SER_LATCH
 $Comp
 L power:+5V #PWR0117
 U 1 1 6240AF10
-P 800 4200
-F 0 "#PWR0117" H 800 4050 50  0001 C CNN
-F 1 "+5V" H 815 4373 50  0000 C CNN
-F 2 "" H 800 4200 50  0001 C CNN
-F 3 "" H 800 4200 50  0001 C CNN
-	1    800  4200
+P 750 3900
+F 0 "#PWR0117" H 750 3750 50  0001 C CNN
+F 1 "+5V" H 765 4073 50  0000 C CNN
+F 2 "" H 750 3900 50  0001 C CNN
+F 3 "" H 750 3900 50  0001 C CNN
+	1    750  3900
 	1    0    0    -1
 $EndComp
@@
 	1800 4200 1300 4200
 Wire Wire Line
-	1000 4200 800  4200
+	1000 4200 750  4200
 Wire Wire Line
 	3300 4500 3800 4500
@@
 Wire Wire Line
 	6900 2600 7300 2600
-NoConn ~ 3550 3200
 $Comp
 L mtg_life_counter:USB_C_Receptacle_USB2.0-Connector J1
@@
 	2150 5550 2150 5650
 $Comp
-L Device:R R5
+L Device:R R60
 U 1 1 6286452B
 P 2300 5850
-F 0 "R5" V 2400 5850 50  0000 C CNN
+F 0 "R60" V 2400 5850 50  0000 C CNN
 F 1 "5.1k" V 2300 5850 50  0000 C CNN
 F 2 "Resistor_SMD:R_0805_2012Metric_Pad1.15x1.40mm_HandSolder" V 2230 5850 50  0001 C CNN
@@
 $EndComp
 $Comp
-L Device:R R6
+L Device:R R61
 U 1 1 62864ACD
 P 2300 5950
-F 0 "R6" V 2200 5950 50  0000 C CNN
+F 0 "R61" V 2200 5950 50  0000 C CNN
 F 1 "5.1k" V 2300 5950 50  0000 C CNN
 F 2 "Resistor_SMD:R_0805_2012Metric_Pad1.15x1.40mm_HandSolder" V 2230 5950 50  0001 C CNN
@@
 Wire Wire Line
 	2150 5950 2050 5950
-NoConn ~ 3550 3600
 $Comp
 L power:GND #PWR0139
@@
 NoConn ~ 4850 5650
 NoConn ~ 5100 5650
-Text Notes 600  4400 0    50   ~ 0
+Text Notes 600  4850 0    50   ~ 0
 TODO: Confirm latch pull-up/down direction
+Text Label 1800 4200 2    50   ~ 0
+DISP_LATCH
+Text Label 8900 2350 0    50   ~ 0
+DISP_LATCH
+Text Label 8900 4200 0    50   ~ 0
+DISP_LATCH
+Text Label 8900 6200 0    50   ~ 0
+DISP_LATCH
+Text Label 8900 8200 0    50   ~ 0
+DISP_LATCH
+Text Label 15900 6900 2    50   ~ 0
+DISP_LATCH
+Text Label 15900 3050 2    50   ~ 0
+DISP_LATCH
+Text Label 1800 3900 2    50   ~ 0
+ENC_LATCH
+$Comp
+L Device:R R2
+U 1 1 61DCE226
+P 1150 3900
+F 0 "R2" V 1250 3900 50  0000 C CNN
+F 1 "10k" V 1150 3900 50  0000 C CNN
+F 2 "Resistor_SMD:R_0805_2012Metric_Pad1.15x1.40mm_HandSolder" V 1080 3900 50  0001 C CNN
+F 3 "~" H 1150 3900 50  0001 C CNN
+	1    1150 3900
+	0    -1   -1   0
+$EndComp
+$Comp
+L power:GND #PWR012
+U 1 1 61DCE57C
+P 750 4200
+F 0 "#PWR012" H 750 3950 50  0001 C CNN
+F 1 "GND" H 755 4027 50  0000 C CNN
+F 2 "" H 750 4200 50  0001 C CNN
+F 3 "" H 750 4200 50  0001 C CNN
+	1    750  4200
+	1    0    0    -1
+$EndComp
+Wire Wire Line
+	750  3900 1000 3900
+Wire Wire Line
+	1300 3900 1800 3900
+Text Label 4500 3500 2    50   ~ 0
+ENC_LATCH
+Wire Wire Line
+	4500 3500 3550 3500
+NoConn ~ 3550 3200
 $EndSCHEMATC

Commit message: Add protection diode. Finalize test points + jumpers
Parts:
- added D5: PJSD05W_R1_00001, Diode_SMD:D_SOD-323_HandSoldering, symbol Diode:1.5KExxA
- added J3: TP_UART, mtg_life_counter:TP_Edge_3, symbol Connector_Generic:Conn_01x03
- added JP2: JP_SR, mtg_life_counter:TP_Edge_2, symbol Connector_Generic:Conn_01x02
- added TP4: SCLK, TestPoint:TestPoint_Pad_D2.0mm, symbol Connector:TestPoint
- added TP5: E_LAT, TestPoint:TestPoint_Pad_D2.0mm, symbol Connector:TestPoint
- added TP6: GND, TestPoint:TestPoint_Pad_D2.0mm, symbol Connector:TestPoint
- added TP7: 5V, TestPoint:TestPoint_Pad_D2.0mm, symbol Connector:TestPoint
- C12: value 1uF -> 10uF
- TP1: value TX -> CIPO; footprint TestPoint:TestPoint_Keystone_5015_Micro-Minature -> TestPoint:TestPoint_Pad_D2.0mm
- TP2: value RX -> D_LAT; footprint TestPoint:TestPoint_Keystone_5015_Micro-Minature -> TestPoint:TestPoint_Pad_D2.0mm
- TP3: value GND -> COPI; footprint TestPoint:TestPoint_Keystone_5015_Micro-Minature -> TestPoint:TestPoint_Pad_D2.0mm
Connections:
- net +5V: now also C11.2, C12.2, TP7.1
- net D0(RX): now also J3.1 (Pin_1); no longer TP2.1
- net D1(TX): now also J3.2 (Pin_2); no longer TP1.1
- net DISP_LATCH: now also TP2.1
- net ENC_LATCH: now also TP5.1
- net GND: now also D5.2 (A2), J3.3 (Pin_3), TP6.1; no longer TP3.1
- net SER_CLK: now also TP4.1
- net SR_OUT: now also JP2.2 (Pin_2)
- net VBUS: now also D5.1 (A1); no longer C11.2, C12.2
- net SER_MISO renamed SER_CIPO
- net SER_CIPO: now also TP1.1, JP2.1 (Pin_1)
- net SER_MOSI renamed SER_COPI
- net SER_COPI: now also TP3.1
Other:
- note added: "D11(COPI)"
- note added: "D12(CIPO)"
- note removed: "D11(MOSI)"
- note removed: "D12(MISO)"
- note removed: "TODO: Confirm latch pull-up/down direction"
- moved on the sheet: B1, B2, C1, C10, C11, C12, C2, C3, E1, E2, E3, E4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

Commit message: Resolve design review issues
Parts:
- added R6: 10k, Resistor_SMD:R_0805_2012Metric_Pad1.15x1.40mm_HandSolder, symbol Device:R
Connections:
- net SER_CIPO: now also R6.1
- net SR_OUT: now also R6.2
Other:
- moved on the sheet: JP1, JP2
Changed lines of the file:
@@
 L Jumper:Jumper_2_Open JP1
 U 1 1 61C0859C
-P 1750 6750
-F 0 "JP1" H 1750 6985 50  0000 C CNN
-F 1 "Jumper_2_Open" H 1750 6894 50  0000 C CNN
-F 2 "Jumper:SolderJumper-2_P1.3mm_Open_TrianglePad1.0x1.5mm" H 1750 6750 50  0001 C CNN
-F 3 "~" H 1750 6750 50  0001 C CNN
-	1    1750 6750
+P 1800 6500
+F 0 "JP1" H 1800 6735 50  0000 C CNN
+F 1 "Jumper_2_Open" H 1800 6644 50  0000 C CNN
+F 2 "Jumper:SolderJumper-2_P1.3mm_Open_TrianglePad1.0x1.5mm" H 1800 6500 50  0001 C CNN
+F 3 "~" H 1800 6500 50  0001 C CNN
+	1    1800 6500
 	1    0    0    -1
 $EndComp
@@
 Wire Wire Line
 	1600 8550 2100 8550
-Text Label 1000 6750 0    50   ~ 0
+Text Label 1050 6500 0    50   ~ 0
 SR_OUT
-Text Label 2500 6750 2    50   ~ 0
+Text Label 2550 6500 2    50   ~ 0
 SER_CIPO
 Wire Wire Line
-	1550 6750 1450 6750
+	1600 6500 1500 6500
 Wire Wire Line
 	2000 9250 2000 9550
@@
 	6500 4850 6250 4850
 Wire Wire Line
-	1950 6750 2050 6750
+	2000 6500 2100 6500
 $Comp
 L power:+5V #PWR0136
@@
 L Connector_Generic:Conn_01x02 JP2
 U 1 1 6304655D
-P 2350 6950
-F 0 "JP2" H 2430 6942 50  0000 L CNN
-F 1 "JP_SR" H 2430 6851 50  0000 L CNN
-F 2 "mtg_life_counter:TP_Edge_2" H 2350 6950 50  0001 C CNN
-F 3 "~" H 2350 6950 50  0001 C CNN
-	1    2350 6950
-	1    0    0    -1
-$EndComp
-Wire Wire Line
-	2050 6750 2050 6950
-Wire Wire Line
-	2050 6950 2150 6950
-Connection ~ 2050 6750
-Wire Wire Line
-	2050 6750 2500 6750
-Wire Wire Line
-	1450 6750 1450 7050
-Wire Wire Line
-	1450 7050 2150 7050
-Connection ~ 1450 6750
-Wire Wire Line
-	1450 6750 1000 6750
+P 2400 6750
+F 0 "JP2" H 2480 6742 50  0000 L CNN
+F 1 "JP_SR" H 2480 6651 50  0000 L CNN
+F 2 "mtg_life_counter:TP_Edge_2" H 2400 6750 50  0001 C CNN
+F 3 "~" H 2400 6750 50  0001 C CNN
+	1    2400 6750
+	1    0    0    -1
+$EndComp
+Connection ~ 2100 6500
+Wire Wire Line
+	2100 6500 2550 6500
+Wire Wire Line
+	1500 6500 1500 6750
+Wire Wire Line
+	1500 6850 2200 6850
+Connection ~ 1500 6500
+Wire Wire Line
+	1500 6500 1050 6500
 Wire Wire Line
 	3550 8450 3550 8950
@@
 $EndComp
 $Comp
-L power:+5V #PWR?
+L power:+5V #PWR0139
 U 1 1 63669CBE
 P 6300 2550
-F 0 "#PWR?" H 6300 2400 50  0001 C CNN
+F 0 "#PWR0139" H 6300 2400 50  0001 C CNN
 F 1 "+5V" H 6315 2723 50  0000 C CNN
 F 2 "" H 6300 2550 50  0001 C CNN
@@
 Wire Wire Line
 	6300 2550 6700 2550
+$Comp
+L Device:R R6
+U 1 1 63888C60
+P 1800 6750
+F 0 "R6" V 1700 6750 50  0000 C CNN
+F 1 "10k" V 1800 6750 50  0000 C CNN
+F 2 "Resistor_SMD:R_0805_2012Metric_Pad1.15x1.40mm_HandSolder" V 1730 6750 50  0001 C CNN
+F 3 "~" H 1800 6750 50  0001 C CNN
+	1    1800 6750
+	0    1    1    0
+$EndComp
+Wire Wire Line
+	1650 6750 1500 6750
+Connection ~ 1500 6750
+Wire Wire Line
+	1950 6750 2100 6750
+Wire Wire Line
+	2100 6500 2100 6750
+Connection ~ 2100 6750
+Wire Wire Line
+	2100 6750 2200 6750
+Wire Wire Line
+	1500 6750 1500 6850
 $EndSCHEMATC
