File: pcb/mtg_life_counter.kicad_pcb (KiCad board)
At the start: 2 copper layers, 208.3 x 127 mm, 77 parts, among them SW1 SW_SPDT, SW2 SW_SPST, SW3 SW_SP4T, SW4 SW_SP4T, SW5 SW_SP4T, SW6 SW_SP4T, U1 74HC595, U2 TPIC6595, U3 74HC595, U4 TPIC6595, U5 74LS151, U6 74LS151, U7 74LS151

Commit message: Sketch out mini pcb
Parts:
- removed B10, B3, B4, B5, B6, B7, B8, B9: SW_Push, mtg_life_counter:B3F_12mm
- removed C6, C7: 0.1uF, Capacitor_THT:C_Disc_D3.0mm_W1.6mm_P2.50mm
- removed RN1, RN2, RN3: 1000, Resistor_THT:R_Array_SIP9
- removed SW3, SW4, SW5, SW6: SW_SP4T, mtg_life_counter:CK_RM10x77
- removed the U4 at (50.8, 109.2)
- removed the U5 at (151.1, 68.6)
- added E1: Rotary_Encoder_Switch, Rotary_Encoder:RotaryEncoder_Alps_EC11E-Switch_Vertical_H20mm, F.Cu at (45.7, 132.1)
- added E2: Rotary_Encoder_Switch, Rotary_Encoder:RotaryEncoder_Alps_EC11E-Switch_Vertical_H20mm, F.Cu at (45.7, 66.0)
- added E3: Rotary_Encoder_Switch, Rotary_Encoder:RotaryEncoder_Alps_EC11E-Switch_Vertical_H20mm, F.Cu at (183.0, 132.1)
- added E4: Rotary_Encoder_Switch, Rotary_Encoder:RotaryEncoder_Alps_EC11E-Switch_Vertical_H20mm, F.Cu at (182.9, 66.0)
- added J1: USB_B_Micro, Connector_USB:USB_Micro-B_Molex-105017-0001, F.Cu at (41.9, 101.6)
- added R36: 10k, Resistor_SMD:R_1206_3216Metric_Pad1.42x1.75mm_HandSolder, F.Cu at (184.3, 106.6)
- added R37: 10k, Resistor_SMD:R_1206_3216Metric_Pad1.42x1.75mm_HandSolder, F.Cu at (178.3, 106.6)
- added R38: 10k, Resistor_SMD:R_1206_3216Metric_Pad1.42x1.75mm_HandSolder, F.Cu at (191.7, 105.1)
- added R39: 10k, Resistor_SMD:R_1206_3216Metric_Pad1.42x1.75mm_HandSolder, F.Cu at (172.4, 106.6)
- added R40: 10k, Resistor_SMD:R_1206_3216Metric_Pad1.42x1.75mm_HandSolder, F.Cu at (183.1, -7.80)
- added R41: 10k, Resistor_SMD:R_1206_3216Metric_Pad1.42x1.75mm_HandSolder, F.Cu at (183.1, -4.51)
- added R42: 10k, Resistor_SMD:R_1206_3216Metric_Pad1.42x1.75mm_HandSolder, F.Cu at (197.7, 101.8)
- added U1: ATmega328P-AU, Package_QFP:TQFP-32_7x7mm_P0.8mm, F.Cu at (63.5, 101.6)
- added U3: 74LS151, Package_SO:SOIC-16_3.9x9.9mm_P1.27mm, F.Cu at (162.6, 101.6)
- C1, C2, C3, C4, C5: footprint Capacitor_THT:C_Disc_D3.0mm_W1.6mm_P2.50mm -> Capacitor_SMD:C_1206_3216Metric_Pad1.42x1.75mm_HandSolder
- D1: value KW4-56NX -> KW4-56NX RED
- D2: value KW4-56NX -> KW4-56NX GREEN
- D3: value KW4-56NX -> KW4-56NX YELLOW
- D4: value KW4-56NX -> KW4-56NX BLUE
- R1, R2, R3, R4, R5, R6, R7, R8: value R -> 330; footprint Resistor_THT:R_Axial_DIN0207_L6.3mm_D2.5mm_P10.16mm_Horizontal -> Resistor_SMD:R_1206_3216Metric_Pad1.42x1.75mm_HandSolder
- R10, R11, R12, R13, R14, R15, R16, R9: value R -> 33; footprint Resistor_THT:R_Axial_DIN0207_L6.3mm_D2.5mm_P10.16mm_Horizontal -> Resistor_SMD:R_1206_3216Metric_Pad1.42x1.75mm_HandSolder
- R17, R18, R19, R20, R21, R22, R23, R24: value R -> 100; footprint Resistor_THT:R_Axial_DIN0207_L6.3mm_D2.5mm_P10.16mm_Horizontal -> Resistor_SMD:R_1206_3216Metric_Pad1.42x1.75mm_HandSolder
- R25, R26, R27, R28, R29, R30, R31, R32: value R -> 390; footprint Resistor_THT:R_Axial_DIN0207_L6.3mm_D2.5mm_P10.16mm_Horizontal -> Resistor_SMD:R_1206_3216Metric_Pad1.42x1.75mm_HandSolder
- R33, R34: footprint Resistor_THT:R_Axial_DIN0207_L6.3mm_D2.5mm_P10.16mm_Horizontal -> Resistor_SMD:R_1206_3216Metric_Pad1.42x1.75mm_HandSolder
- R35: value 100 -> 10k; footprint Resistor_THT:R_Axial_DIN0207_L6.3mm_D2.5mm_P10.16mm_Horizontal -> Resistor_SMD:R_1206_3216Metric_Pad1.42x1.75mm_HandSolder
- U2: value TPIC6595 -> FT232RL; footprint Package_DIP:DIP-20_W7.62mm -> Package_SO:SSOP-28_5.3x10.2mm_P0.65mm
- U4: renamed from U1; footprint Package_DIP:DIP-16_W7.62mm -> Package_SO:SOIC-16_3.9x9.9mm_P1.27mm
- U5: renamed from U3; footprint Package_DIP:DIP-16_W7.62mm -> Package_SO:SOIC-16_3.9x9.9mm_P1.27mm
- U6, U7: value 74LS151 -> TPIC6C596; footprint Package_DIP:DIP-16_W7.62mm -> Package_SO:SOIC-16_3.9x9.9mm_P1.27mm
- moved A1 230.9 mm to (308.6, 121.9), turned to 0 degrees
- moved C3 204.0 mm to (411.5, 119.4)
- moved C1 204.0 mm to (436.9, 91.5)
- moved C2 204.0 mm to (276.8, 83.8)
- moved R33 204.0 mm to (261.6, 83.8)
- moved R34 204.0 mm to (269.2, 129.5)
- moved U7 127.3 mm to (53.3, 83.8)
- moved R35 100.6 mm to (191.7, 101.8), turned to 0 degrees
- moved U6 82.3 mm to (51.4, 116.9)
- moved U4 60.4 mm to (175.3, 91.4)
- moved C4 54.7 mm to (100.5, 88.9)
- moved H2 47.9 mm to (200.7, 55.9)
- moved R13 46.6 mm to (161.3, 81.3)
- moved R14 46.6 mm to (153.7, 81.3)
- moved R15 46.6 mm to (143.5, 81.3)
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Connections:
- A1 pad 13: Net-(A1-Pad13) -> /SEL_2
- A1 pad 19: /RNG_WIRE -> /SEL_1
- A1 pad 25: /SEL_1 -> Net-(A1-Pad25)
- A1 pad 26: /SEL_2 -> /RNG_WIRE
- R35 pad 1: GND -> +5V
- R35 pad 2: /OFF -> Net-(R35-Pad2)
- SW1 pad 1: /5V_SRC -> Net-(SW1-Pad1)
- SW1 pad 3: /OFF -> GND
- U2 pad 10: GND -> Net-(U2-Pad10)
- U2 pad 11: GND -> Net-(U2-Pad11)
- U2 pad 12: /SER_LATCH -> Net-(U2-Pad12)
- U2 pad 13: /SER_CLK -> Net-(U2-Pad13)
- U2 pad 14: Net-(D2-Pad14) -> Net-(U2-Pad14)
- U2 pad 15: Net-(D2-Pad11) -> Net-(U2-Pad15)
- U2 pad 16: Net-(D2-Pad10) -> Net-(U2-Pad16)
- U2 pad 17: Net-(D2-Pad6) -> Net-(U2-Pad17)
- U2 pad 18: /SER_CASCADE_3 -> Net-(U2-Pad18)
- U2 pad 19: GND -> Net-(U2-Pad19)
- U2 pad 2: +5V -> Net-(U2-Pad2)
- U2 pad 3: /SER_CASCADE_2 -> Net-(U2-Pad3)
- U2 pad 4: Net-(D1-Pad14) -> Net-(U2-Pad4)
- U2 pad 5: Net-(D1-Pad11) -> Net-(U2-Pad5)
- U2 pad 6: Net-(D1-Pad10) -> Net-(U2-Pad6)
- U2 pad 7: Net-(D1-Pad6) -> Net-(U2-Pad7)
- U2 pad 8: Net-(R33-Pad1) -> (no net)
- U2 pad 9: /NENABLE -> Net-(U2-Pad9)
- U6 pad 10: /SEL_1 -> GND
- U6 pad 11: /SEL_0 -> GND
- U6 pad 12: Net-(RN2-Pad9) -> /SER_LATCH
- U6 pad 13: Net-(RN2-Pad8) -> /SER_CLK
- U6 pad 14: Net-(RN2-Pad7) -> Net-(D2-Pad14)
- U6 pad 15: Net-(RN2-Pad6) -> Net-(D2-Pad11)
- U6 pad 16: +5V -> Net-(D2-Pad10)
- U6 pad 2: Net-(RN2-Pad3) -> +5V
- U6 pad 3: Net-(RN2-Pad4) -> /SER_CASCADE_2
- U6 pad 4: Net-(RN2-Pad5) -> Net-(D1-Pad14)
- U6 pad 5: Net-(U6-Pad5) -> Net-(D1-Pad11)
- U6 pad 6: /SW_RB_2 -> Net-(D1-Pad10)
- U6 pad 7: GND -> Net-(D1-Pad6)
- U6 pad 8: GND -> Net-(R33-Pad1)
- U6 pad 9: /SEL_2 -> /NENABLE
- U7 pad 10: /SEL_1 -> GND
- U7 pad 11: /SEL_0 -> GND
- U7 pad 12: Net-(B6-Pad1) -> /SER_LATCH
- U7 pad 13: Net-(B5-Pad1) -> /SER_CLK
- U7 pad 14: Net-(B4-Pad1) -> Net-(D3-Pad14)
- U7 pad 15: Net-(B3-Pad1) -> Net-(D3-Pad11)
- U7 pad 16: +5V -> Net-(D3-Pad10)
- U7 pad 2: Net-(B10-Pad1) -> +5V
- U7 pad 3: Net-(B8-Pad1) -> /SER_CASCADE_3
- U7 pad 4: Net-(B7-Pad1) -> Net-(D4-Pad14)
- U7 pad 5: Net-(U7-Pad5) -> Net-(D4-Pad11)
- U7 pad 6: /BTN_RB -> Net-(D4-Pad10)
- U7 pad 7: GND -> Net-(D4-Pad6)
- U7 pad 8: GND -> Net-(R34-Pad1)
- U7 pad 9: /SEL_2 -> /NENABLE
Routing:
- net +5V: track 457.8 -> 0.00 mm, vias 5 -> 0
- net /SER_CLK: track 377.0 -> 0.00 mm
- net /NENABLE: track 373.3 -> 0.00 mm, vias 5 -> 0
- net /SER_LATCH: track 357.5 -> 0.00 mm, vias 2 -> 0
- net Net-(B10-Pad1): track 195.2 -> 0.00 mm, vias 1 -> 0
- net /SER_CASCADE_2: track 191.9 -> 0.00 mm, vias 2 -> 0
- net Net-(U7-Pad1): track 181.5 -> 0.00 mm, vias 1 -> 0
- net /SER_DATA: track 179.9 -> 0.00 mm
- net Net-(B3-Pad1): track 175.0 -> 0.00 mm, vias 2 -> 0
- net /SEL_0: track 174.8 -> 0.00 mm, vias 2 -> 0
- net /SEL_1: track 171.3 -> 0.00 mm, vias 4 -> 0
- net Net-(D2-Pad14): track 168.3 -> 0.00 mm, vias 1 -> 0
- net Net-(R10-Pad2): track 168.0 -> 0.00 mm, vias 2 -> 0
- net Net-(D3-Pad6): track 166.6 -> 0.00 mm, vias 1 -> 0
- net /SEL_2: track 165.6 -> 0.00 mm, vias 4 -> 0
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Other:
- board size 208.3 x 127 mm -> 167.6 x 101.6 mm

Commit message: Continue updating schematic
Parts:
- removed A1: Arduino_Nano_v3.x, Module:Arduino_Nano
- added C6: 0.1uF, Capacitor_SMD:C_1206_3216Metric_Pad1.42x1.75mm_HandSolder, F.Cu at (235.7, 115.5)
- added C7: 0.1uF, Capacitor_SMD:C_1206_3216Metric_Pad1.42x1.75mm_HandSolder, F.Cu at (247.6, 109.1)
- SW1: value SW_SPDT -> SW_SPST
- U2: moved to B.Cu
- moved C1 193.0 mm to (243.8, 92.5)
- moved C3 191.6 mm to (226.1, 71.1)
- moved E2 165.2 mm to (210.8, 71.1), turned to 180 degrees
- moved E4 140.9 mm to (58.4, 132.1)
- moved R41 133.5 mm to (247.6, 112.4)
- moved R40 131.1 mm to (265.9, 93.9)
- moved C4 129.1 mm to (229.7, 91.4)
- moved C5 104.7 mm to (237.3, 104.1)
- moved R37 75.9 mm to (254.2, 105.5)
- moved R39 69.8 mm to (241.6, 115.5)
- moved E1 66.8 mm to (72.9, 71.1), turned to 180 degrees
- moved R42 56.4 mm to (253.6, 109.1)
- moved R36 52.8 mm to (235.7, 118.8)
- moved R38 47.1 mm to (235.7, 122.1)
- moved R35 43.1 mm to (234.7, 99.1)
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Connections:
- net /NENABLE renamed /~ENABLE
- net Net-(E1-PadS1) renamed /E1_SW
- net Net-(E2-PadS1) renamed /E2_SW
- net Net-(E3-PadS1) renamed /E3_SW
- net Net-(E4-PadS1) renamed /E4_SW
- net Net-(U1-Pad1) renamed /D3
- net Net-(U1-Pad10) renamed /D6
- net Net-(U1-Pad11) renamed /D7
- net Net-(U1-Pad12) renamed /D8
- net Net-(U1-Pad13) renamed /D9
- net Net-(U1-Pad14) renamed /D10
- net Net-(U1-Pad16) renamed /D12
- net Net-(U1-Pad19) renamed /A6
- net Net-(U1-Pad2) renamed /D4
- net Net-(U1-Pad20) renamed /AREF
- net Net-(U1-Pad22) renamed /A7
- net Net-(U1-Pad23) renamed /A0
- net Net-(U1-Pad24) renamed /A1
- net Net-(U1-Pad25) renamed /A2
- net Net-(U1-Pad26) renamed /A3
- net Net-(U1-Pad27) renamed /A4
- net Net-(U1-Pad28) renamed /A5
- net Net-(U1-Pad29) renamed /~RESET
- net Net-(U1-Pad30) renamed /D0(RX)
- net Net-(U1-Pad31) renamed /D1(TX)
- net Net-(U1-Pad32) renamed /D2
- net Net-(U1-Pad9) renamed /D5
- E1 pad A: Net-(E1-PadA) -> /E1_CLK
- E1 pad B: Net-(E1-PadB) -> /E1_DIR
- E1 pad C: Net-(E1-PadC) -> GND
- E1 pad S2: Net-(E1-PadS2) -> GND
- E2 pad A: Net-(E2-PadA) -> /E2_CLK
- E2 pad B: Net-(E2-PadB) -> /E2_DIR
- E2 pad C: Net-(E2-PadC) -> GND
- E2 pad S2: Net-(E2-PadS2) -> GND
- E3 pad A: Net-(E3-PadA) -> /E3_CLK
- E3 pad B: Net-(E3-PadB) -> /E3_DIR
- E3 pad C: Net-(E3-PadC) -> GND
- E3 pad S2: Net-(E3-PadS2) -> GND
- E4 pad A: Net-(E4-PadA) -> /E4_CLK
- E4 pad B: Net-(E4-PadB) -> /E4_DIR
- E4 pad C: Net-(E4-PadC) -> GND
- E4 pad S2: Net-(E4-PadS2) -> GND
- J1 pad 2: Net-(J1-Pad2) -> /USB_DM
- J1 pad 3: Net-(J1-Pad3) -> /USB_DP
- J1 pad 5: Net-(J1-Pad5) -> GND
- J1 pad 6: Net-(J1-Pad6) -> GND
- R35 pad 2: Net-(R35-Pad2) -> /E1_CLK
- R36 pad 2: Net-(R36-Pad2) -> /E1_DIR
- R37 pad 2: Net-(R37-Pad2) -> /E2_CLK
- R38 pad 2: Net-(R38-Pad2) -> /E2_DIR
- R39 pad 2: Net-(R39-Pad2) -> /E3_CLK
- R40 pad 2: Net-(R40-Pad2) -> /E3_DIR
- R41 pad 2: Net-(R41-Pad2) -> /E4_CLK
- R42 pad 2: Net-(R42-Pad2) -> /E4_DIR
- SW1 pad 1: Net-(SW1-Pad1) -> Net-(J1-Pad1)
- SW1 pad 3: GND -> (no net)
- U1 pad 15: Net-(U1-Pad15) -> /D11
- U1 pad 17: Net-(U1-Pad17) -> /D13
- U1 pad 18: Net-(U1-Pad18) -> +5V
- U1 pad 21: Net-(U1-Pad21) -> GND
- U1 pad 3: Net-(U1-Pad21) -> GND
- U1 pad 4: Net-(U1-Pad4) -> +5V
- U1 pad 5: Net-(U1-Pad21) -> GND
- U1 pad 6: Net-(U1-Pad4) -> +5V
- U2 pad 15: Net-(U2-Pad15) -> /USB_DP
- U2 pad 16: Net-(U2-Pad16) -> /USB_DM
- U3 pad 1: Net-(R35-Pad2) -> /E2_DIR
- U3 pad 12: Net-(R42-Pad2) -> /E4_DIR
- U3 pad 13: Net-(R41-Pad2) -> /E4_CLK
- U3 pad 14: Net-(R40-Pad2) -> /E3_DIR
- U3 pad 15: Net-(R39-Pad2) -> /E3_CLK
- U3 pad 2: Net-(R36-Pad2) -> /E2_CLK
- U3 pad 3: Net-(R37-Pad2) -> /E1_DIR
- U3 pad 4: Net-(R38-Pad2) -> /E1_CLK
- U4 pad 11: /SER_CLK -> /D13
- U4 pad 14: /SER_DATA -> /SER_LINK_3
- U4 pad 9: /SER_CASCADE_1 -> Net-(U4-Pad9)
- U5 pad 11: /SER_CLK -> /D13
- U5 pad 14: /SER_CASCADE_1 -> /SER_LINK_2
- U5 pad 9: /SER_CASCADE_2 -> /SER_LINK_3
- U6 pad 13: /SER_CLK -> /D13
- U6 pad 3: /SER_CASCADE_2 -> /SER_LINK_1
- U7 pad 13: /SER_CLK -> /D13
- U7 pad 14: Net-(D3-Pad14) -> Net-(D4-Pad14)
- U7 pad 15: Net-(D3-Pad11) -> Net-(D4-Pad11)
- U7 pad 16: Net-(D3-Pad10) -> Net-(D4-Pad10)
- U7 pad 3: /SER_CASCADE_3 -> /D11
- U7 pad 4: Net-(D4-Pad14) -> Net-(D3-Pad14)
- U7 pad 5: Net-(D4-Pad11) -> Net-(D3-Pad11)
- U7 pad 6: Net-(D4-Pad10) -> Net-(D3-Pad10)
- U7 pad 7: Net-(D4-Pad6) -> Net-(D3-Pad6)
Other:
- net class Power: trace_width 1 -> 0.5
- board text added: "Max Proskauer v1.0 Oct 2020 github.com/mprosk/mtg_life_counter"
- board text added: "Version 1.0"
- board text removed: "Max Proskauer v0.1 August 2020"

Commit message: Continue work on mini PCB
Parts:
- removed R18, R19: 100, Resistor_SMD:R_1206_3216Metric_Pad1.42x1.75mm_HandSolder
- removed the R2 at (97.8, 81.3)
- removed R28, R29: 390, Resistor_SMD:R_1206_3216Metric_Pad1.42x1.75mm_HandSolder
- removed the R3 at (100.3, 81.3)
- removed R38, R39: 10k, Resistor_SMD:R_1206_3216Metric_Pad1.42x1.75mm_HandSolder
- removed R6, R7, R8: 330, Resistor_SMD:R_1206_3216Metric_Pad1.42x1.75mm_HandSolder
- removed R9: 33, Resistor_SMD:R_1206_3216Metric_Pad1.42x1.75mm_HandSolder
- removed the U6 at (64.1, 116.9)
- removed the U7 at (66.0, 83.8)
- added C10: 100nF, Capacitor_SMD:C_1206_3216Metric_Pad1.42x1.75mm_HandSolder, B.Cu at (67.5, 86.4)
- added C3: 0.1uF, Capacitor_SMD:C_1206_3216Metric_Pad1.42x1.75mm_HandSolder, F.Cu at (73.7, 92.7)
- added C4: 0.1uF, Capacitor_SMD:C_1206_3216Metric_Pad1.42x1.75mm_HandSolder, F.Cu at (73.7, 96.0)
- added J2: ICSP, Connector:Tag-Connect_TC2030-IDC-NL_2x03_P1.27mm_Vertical, F.Cu at (80.0, 89.5)
- added R33: 100, Resistor_SMD:R_1206_3216Metric_Pad1.42x1.75mm_HandSolder, F.Cu at (158.8, 121.7)
- added R34: 100, Resistor_SMD:R_1206_3216Metric_Pad1.42x1.75mm_HandSolder, F.Cu at (156.2, 121.7)
- added R43: 390, Resistor_SMD:R_1206_3216Metric_Pad1.42x1.75mm_HandSolder, F.Cu at (97.8, 121.7)
- added R44: 390, Resistor_SMD:R_1206_3216Metric_Pad1.42x1.75mm_HandSolder, F.Cu at (95.2, 121.7)
- added R45: 390, Resistor_SMD:R_1206_3216Metric_Pad1.42x1.75mm_HandSolder, F.Cu at (102.9, 121.7)
- added R46: 390, Resistor_SMD:R_1206_3216Metric_Pad1.42x1.75mm_HandSolder, F.Cu at (113.0, 121.7)
- added R47: 390, Resistor_SMD:R_1206_3216Metric_Pad1.42x1.75mm_HandSolder, F.Cu at (105.4, 121.7)
- added R50: 10k, Resistor_SMD:R_1206_3216Metric_Pad1.42x1.75mm_HandSolder, F.Cu at (59.5, 78.7)
- added R51: 10k, Resistor_SMD:R_1206_3216Metric_Pad1.42x1.75mm_HandSolder, F.Cu at (71.1, 78.7)
- added R52: 10k, Resistor_SMD:R_1206_3216Metric_Pad1.42x1.75mm_HandSolder, F.Cu at (212.3, 80.0)
- added R53: 10k, Resistor_SMD:R_1206_3216Metric_Pad1.42x1.75mm_HandSolder, F.Cu at (216.1, 66.0)
- added R54: 10k, Resistor_SMD:R_1206_3216Metric_Pad1.42x1.75mm_HandSolder, F.Cu at (210.6, 121.9)
- added R55: 10k, Resistor_SMD:R_1206_3216Metric_Pad1.42x1.75mm_HandSolder, F.Cu at (201.7, 123.2)
- added R56: 10k, Resistor_SMD:R_1206_3216Metric_Pad1.42x1.75mm_HandSolder, F.Cu at (59.5, 123.2)
- added R57: 10k, Resistor_SMD:R_1206_3216Metric_Pad1.42x1.75mm_HandSolder, F.Cu at (73.7, 123.2)
- added U4: TPIC6596, Package_SO:SOIC-16_3.9x9.9mm_P1.27mm, F.Cu at (134.7, 67.9)
- added U5: TPIC6596, Package_SO:SOIC-16_3.9x9.9mm_P1.27mm, F.Cu at (134.6, 134.0)
- added Y1: 16MHz, Crystal:Crystal_HC49-U_Vertical, F.Cu at (123.4, 27.1)
- C1: renamed from C6; value 0.1uF -> 18pF; footprint Capacitor_SMD:C_1206_3216Metric_Pad1.42x1.75mm_HandSolder -> Capacitor_SMD:C_0805_2012Metric_Pad1.15x1.40mm_HandSolder
- C2: renamed from C7; value 0.1uF -> 18pF; footprint Capacitor_SMD:C_1206_3216Metric_Pad1.42x1.75mm_HandSolder -> Capacitor_SMD:C_0805_2012Metric_Pad1.15x1.40mm_HandSolder
- R1: value 330 -> 1k
- R10, R11, R12, R13, R14, R15, R16: value 33 -> 330
- R17: value 100 -> 330
- R20, R21, R22, R23, R24: value 100 -> 33
- R25, R26, R27: value 390 -> 33
- R30, R31, R32: value 390 -> 100
- R35, R36, R37: value 10k -> 100
- R4, R5: value 330 -> 1k; moved to B.Cu
- R40, R41, R42: value 10k -> 390
- moved R40 167.9 mm to (100.3, 121.7), turned to 270 degrees
- moved R42 146.1 mm to (108.0, 121.7), turned to 270 degrees
- moved R41 137.4 mm to (110.5, 121.7), turned to 270 degrees
- moved R3 115.9 mm to (136.1, 142.9)
- moved R37 89.3 mm to (166.4, 121.7), turned to 270 degrees
- moved R25 77.4 mm to (166.4, 81.5)
- moved R35 74.4 mm to (163.8, 121.7), turned to 270 degrees
- moved R12 71.1 mm to (100.3, 81.5), turned to 90 degrees
- moved R17 71.0 mm to (102.9, 81.5)
- moved R27 69.0 mm to (163.8, 81.5)
- moved R16 68.6 mm to (95.2, 81.5), turned to 90 degrees
- moved R13 63.5 mm to (110.5, 81.5), turned to 90 degrees
- moved R32 63.5 mm to (168.9, 121.7), turned to 270 degrees
- moved R11 63.5 mm to (97.8, 81.5), turned to 90 degrees
- moved R36 61.7 mm to (174.0, 121.7), turned to 270 degrees
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- renumbered C1 to C5, C3 to C6, C2 to C7, C4 to C8, C5 to C9, R33 to R2, R34 to R3, U4 to U2, U5 to U3, U3 to U6, U2 to U7
Connections:
- net /D13 renamed /D13(SCK)
- net Net-(J1-Pad1) renamed VBUS
- R1 pad 1: Net-(D1-Pad13) -> Net-(R1-Pad1)
- R10 pad 1: Net-(D2-Pad9) -> Net-(R10-Pad1)
- R10 pad 2: Net-(R10-Pad2) -> Net-(D1-Pad13)
- R11 pad 1: Net-(D2-Pad4) -> Net-(R11-Pad1)
- R11 pad 2: Net-(R11-Pad2) -> Net-(D1-Pad9)
- R12 pad 1: Net-(D2-Pad2) -> Net-(R12-Pad1)
- R12 pad 2: Net-(R12-Pad2) -> Net-(D1-Pad4)
- R13 pad 1: Net-(D2-Pad1) -> Net-(R13-Pad1)
- R13 pad 2: Net-(R13-Pad2) -> Net-(D1-Pad2)
- R14 pad 1: Net-(D2-Pad12) -> Net-(R14-Pad1)
- R14 pad 2: Net-(R14-Pad2) -> Net-(D1-Pad1)
- R15 pad 1: Net-(D2-Pad5) -> Net-(R15-Pad1)
- R15 pad 2: Net-(R15-Pad2) -> Net-(D1-Pad12)
- R16 pad 1: Net-(D2-Pad3) -> Net-(R16-Pad1)
- R16 pad 2: Net-(R16-Pad2) -> Net-(D1-Pad5)
- R17 pad 1: Net-(D3-Pad13) -> Net-(R17-Pad1)
- R17 pad 2: Net-(R17-Pad2) -> Net-(D1-Pad3)
- R20 pad 1: Net-(D3-Pad2) -> Net-(R10-Pad1)
- R20 pad 2: Net-(R20-Pad2) -> Net-(D2-Pad13)
- R21 pad 1: Net-(D3-Pad1) -> Net-(R11-Pad1)
- R21 pad 2: Net-(R21-Pad2) -> Net-(D2-Pad9)
- R22 pad 1: Net-(D3-Pad12) -> Net-(R12-Pad1)
- R22 pad 2: Net-(R22-Pad2) -> Net-(D2-Pad4)
- R23 pad 1: Net-(D3-Pad5) -> Net-(R13-Pad1)
- R23 pad 2: Net-(R23-Pad2) -> Net-(D2-Pad2)
- R24 pad 1: Net-(D3-Pad3) -> Net-(R14-Pad1)
- R24 pad 2: Net-(R24-Pad2) -> Net-(D2-Pad1)
- R25 pad 1: Net-(D4-Pad13) -> Net-(R15-Pad1)
- R25 pad 2: Net-(R17-Pad2) -> Net-(D2-Pad12)
- R26 pad 1: Net-(D4-Pad9) -> Net-(R16-Pad1)
- R26 pad 2: Net-(R18-Pad2) -> Net-(D2-Pad5)
- R27 pad 1: Net-(D4-Pad4) -> Net-(R17-Pad1)
- R27 pad 2: Net-(R19-Pad2) -> Net-(D2-Pad3)
- R30 pad 1: Net-(D4-Pad12) -> Net-(R30-Pad1)
- R30 pad 2: Net-(R22-Pad2) -> Net-(D3-Pad13)
- R31 pad 1: Net-(D4-Pad5) -> Net-(R31-Pad1)
- R31 pad 2: Net-(R23-Pad2) -> Net-(D3-Pad9)
- R32 pad 1: Net-(D4-Pad3) -> Net-(R32-Pad1)
- R32 pad 2: Net-(R24-Pad2) -> Net-(D3-Pad4)
- R35 pad 1: +5V -> Net-(R35-Pad1)
- R35 pad 2: /E1_CLK -> Net-(D3-Pad12)
- R36 pad 1: +5V -> Net-(R36-Pad1)
- R36 pad 2: /E1_DIR -> Net-(D3-Pad5)
- R37 pad 1: +5V -> Net-(R37-Pad1)
- R37 pad 2: /E2_CLK -> Net-(D3-Pad3)
- R4 pad 1: Net-(D1-Pad2) -> /D0(RX)
- R4 pad 2: Net-(R12-Pad2) -> Net-(R4-Pad2)
- R40 pad 1: +5V -> Net-(R30-Pad1)
- R40 pad 2: /E3_DIR -> Net-(D4-Pad13)
- R41 pad 1: +5V -> Net-(R31-Pad1)
- R41 pad 2: /E4_CLK -> Net-(D4-Pad9)
- R42 pad 1: +5V -> Net-(R32-Pad1)
- R42 pad 2: /E4_DIR -> Net-(D4-Pad4)
- R5 pad 1: Net-(D1-Pad1) -> /D1(TX)
- R5 pad 2: Net-(R13-Pad2) -> Net-(R5-Pad2)
- U1 pad 15: /D11 -> /D11(MOSI)
- U1 pad 16: /D12 -> /D12(MISO)
- U2 pad 1: Net-(R10-Pad2) -> Net-(R11-Pad1)
- U2 pad 15: Net-(R1-Pad2) -> Net-(R10-Pad1)
- U2 pad 2: Net-(R11-Pad2) -> Net-(R12-Pad1)
- U2 pad 3: Net-(R12-Pad2) -> Net-(R13-Pad1)
- U2 pad 4: Net-(R13-Pad2) -> Net-(R14-Pad1)
- U2 pad 5: Net-(R14-Pad2) -> Net-(R15-Pad1)
- U2 pad 6: Net-(R15-Pad2) -> Net-(R16-Pad1)
- U2 pad 7: Net-(R16-Pad2) -> Net-(R17-Pad1)
- U3 pad 1: Net-(R18-Pad2) -> Net-(R31-Pad1)
- U3 pad 15: Net-(R17-Pad2) -> Net-(R30-Pad1)
- U3 pad 2: Net-(R19-Pad2) -> Net-(R32-Pad1)
- U3 pad 3: Net-(R20-Pad2) -> Net-(R33-Pad1)
- U3 pad 4: Net-(R21-Pad2) -> Net-(R34-Pad1)
- U3 pad 5: Net-(R22-Pad2) -> Net-(R35-Pad1)
- U3 pad 6: Net-(R23-Pad2) -> Net-(R36-Pad1)
- U3 pad 7: Net-(R24-Pad2) -> Net-(R37-Pad1)
- U7 pad 1: Net-(U2-Pad1) -> Net-(R4-Pad2)
- U7 pad 18: Net-(U2-Pad18) -> GND
- U7 pad 20: Net-(U2-Pad20) -> +5V
- U7 pad 21: Net-(U2-Pad21) -> GND
- U7 pad 25: Net-(U2-Pad25) -> GND
- U7 pad 26: Net-(U2-Pad26) -> GND
- U7 pad 4: Net-(U2-Pad4) -> +5V
- U7 pad 5: Net-(U2-Pad5) -> Net-(R5-Pad2)
- U7 pad 7: Net-(U2-Pad7) -> GND
Routing:
- net Net-(R36-Pad1): track 0.00 -> 92.5 mm, vias 0 -> 3
- net Net-(R31-Pad1): track 0.00 -> 88.7 mm, vias 0 -> 3
- net Net-(R32-Pad1): track 0.00 -> 84.9 mm, vias 0 -> 3
- net Net-(R37-Pad1): track 0.00 -> 81.0 mm, vias 0 -> 3
- net Net-(R30-Pad1): track 0.00 -> 79.4 mm, vias 0 -> 3
- net Net-(R35-Pad1): track 0.00 -> 77.2 mm, vias 0 -> 3
- net Net-(R33-Pad1): track 0.00 -> 69.6 mm, vias 0 -> 3
- net Net-(R34-Pad1): track 0.00 -> 65.8 mm, vias 0 -> 3
- net Net-(D3-Pad6): track 0.00 -> 42.2 mm, vias 0 -> 1
- net Net-(D4-Pad14): track 0.00 -> 40.6 mm, vias 0 -> 2
- net Net-(D3-Pad10): track 0.00 -> 37.0 mm, vias 0 -> 2
- net Net-(D3-Pad11): track 0.00 -> 35.7 mm, vias 0 -> 2
- net Net-(D4-Pad11): track 0.00 -> 34.3 mm, vias 0 -> 2
- net Net-(D4-Pad10): track 0.00 -> 33.0 mm, vias 0 -> 2
- net Net-(D3-Pad14): track 0.00 -> 29.3 mm, vias 0 -> 2
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
Commit message: Continue work on mini version
Parts:
- removed C2: 18pF, Capacitor_SMD:C_0805_2012Metric_Pad1.15x1.40mm_HandSolder
- C1: value 18pF -> 4.7uF
- C10: value 100nF -> 0.1uF; footprint Capacitor_SMD:C_1206_3216Metric_Pad1.42x1.75mm_HandSolder -> Capacitor_SMD:C_0805_2012Metric_Pad1.15x1.40mm_HandSolder
- C3, C5, C6, C7, C8, C9: footprint Capacitor_SMD:C_1206_3216Metric_Pad1.42x1.75mm_HandSolder -> Capacitor_SMD:C_0805_2012Metric_Pad1.15x1.40mm_HandSolder
- C4: value 0.1uF -> 1uF; footprint Capacitor_SMD:C_1206_3216Metric_Pad1.42x1.75mm_HandSolder -> Capacitor_SMD:C_0805_2012Metric_Pad1.15x1.40mm_HandSolder
- J1: value USB_B_Micro -> USB_C_Receptacle_USB2.0; footprint Connector_USB:USB_Micro-B_Molex-105017-0001 -> Connector_USB:USB_C_Receptacle_GCT_USB4085
- R1, R10, R11, R12, R13, R14, R15, R16, R17, R2, R20, R21, R22, R23, R24, R25, R26, R27, R3, R30, R31, R32, R33, R34, R35, R36, R37, R4, R40, R41, R42, R43, R44, R45, R46, R47, R5, R50, R51, R52, R53, R54, R55, R56, R57: footprint Resistor_SMD:R_1206_3216Metric_Pad1.42x1.75mm_HandSolder -> Resistor_SMD:R_0805_2012Metric_Pad1.15x1.40mm_HandSolder
- U4, U5: value TPIC6596 -> TPIC6B595; footprint Package_SO:SOIC-16_3.9x9.9mm_P1.27mm -> Package_SO:SOIC-20W_7.5x12.8mm_P1.27mm
- Y1: footprint Crystal:Crystal_HC49-U_Vertical -> Crystal:Resonator_muRata_CSTLSxxxX-3Pin_W5.5mm_H3.0mm
- moved C9 177.9 mm to (59.4, 110.5)
- moved C1 169.3 mm to (67.3, 97.8)
- moved C5 121.5 mm to (122.9, 80.0), turned to 0 degrees
- moved U6 99.2 mm to (66.0, 106.7)
- moved C6 98.2 mm to (142.0, 121.9), turned to 180 degrees
- moved R1 88.2 mm to (73.9, 88.9)
- moved Y1 68.5 mm to (85.1, 83.8)
- moved R3 67.6 mm to (199.4, 119.0), turned to 90 degrees
- moved U4 59.2 mm to (191.1, 85.9), turned to 270 degrees
- moved U5 59.0 mm to (191.1, 117.3), turned to 270 degrees
- moved C7 57.3 mm to (199.4, 82.9), turned to 270 degrees
- moved R2 42.9 mm to (199.4, 87.9), turned to 90 degrees
- moved C8 37.8 mm to (199.4, 114.1), turned to 270 degrees
- moved R53 19.0 mm to (200.9, 77.5)
- moved SW2 12.9 mm to (99.8, 91.4), turned to 180 degrees
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Connections:
- net /D2 renamed Net-(U1-Pad32)
- net /D3 renamed Net-(U1-Pad1)
- net Net-(U7-Pad17) renamed +3V3
- C1 pad 2: GND -> Net-(C1-Pad2)
- R1 pad 1: Net-(R1-Pad1) -> /~RESET
- R1 pad 2: Net-(R1-Pad2) -> +5V
- U1 pad 10: /D6 -> /MUX_SEL_2
- U1 pad 11: /D7 -> /MUX_RB
- U1 pad 12: /D8 -> /~ENABLE
- U1 pad 13: /D9 -> /MODE_SW
- U1 pad 14: /D10 -> /SER_LATCH
- U1 pad 15: /D11(MOSI) -> /SER_DATA
- U1 pad 16: /D12(MISO) -> Net-(U1-Pad16)
- U1 pad 17: /D13(SCK) -> /SER_CLK
- U1 pad 2: /D4 -> /MUX_SEL_0
- U1 pad 23: /A0 -> /E1_SW
- U1 pad 24: /A1 -> /E2_SW
- U1 pad 25: /A2 -> /E3_SW
- U1 pad 26: /A3 -> /E4_SW
- U1 pad 27: /A4 -> /ROLL_BTN
- U1 pad 28: /A5 -> /RESET_BTN
- U1 pad 7: Net-(C1-Pad1) -> Net-(U1-Pad7)
- U1 pad 8: Net-(C2-Pad1) -> Net-(U1-Pad8)
- U1 pad 9: /D5 -> /MUX_SEL_1
- U2 pad 11: /D13(SCK) -> /SER_CLK
- U3 pad 11: /D13(SCK) -> /SER_CLK
- U4 pad 1: +5V -> GND
- U4 pad 10: /SER_LATCH -> GND
- U4 pad 11: Net-(D2-Pad14) -> GND
- U4 pad 12: Net-(D2-Pad11) -> /SER_LATCH
- U4 pad 13: Net-(D2-Pad10) -> /SER_CLK
- U4 pad 14: Net-(D2-Pad6) -> Net-(D2-Pad14)
- U4 pad 15: /D13(SCK) -> Net-(D2-Pad11)
- U4 pad 16: GND -> Net-(D2-Pad10)
- U4 pad 2: /SER_LINK_1 -> +5V
- U4 pad 3: Net-(D1-Pad14) -> /SER_LINK_1
- U4 pad 4: Net-(D1-Pad11) -> Net-(D1-Pad14)
- U4 pad 5: Net-(D1-Pad10) -> Net-(D1-Pad11)
- U4 pad 6: Net-(D1-Pad6) -> Net-(D1-Pad10)
- U4 pad 7: Net-(R2-Pad1) -> Net-(D1-Pad6)
- U4 pad 8: /~ENABLE -> Net-(R2-Pad1)
- U4 pad 9: /SER_LINK_2 -> /~ENABLE
- U5 pad 1: +5V -> GND
- U5 pad 10: /SER_LATCH -> GND
- U5 pad 11: Net-(D4-Pad14) -> GND
- U5 pad 12: Net-(D4-Pad11) -> /SER_LATCH
- U5 pad 13: Net-(D4-Pad10) -> /SER_CLK
- U5 pad 14: Net-(D4-Pad6) -> Net-(D4-Pad14)
- U5 pad 15: /D13(SCK) -> Net-(D4-Pad11)
- U5 pad 16: GND -> Net-(D4-Pad10)
- U5 pad 2: /D11(MOSI) -> +5V
- U5 pad 3: Net-(D3-Pad14) -> /SER_DATA
- U5 pad 4: Net-(D3-Pad11) -> Net-(D3-Pad14)
- U5 pad 5: Net-(D3-Pad10) -> Net-(D3-Pad11)
- U5 pad 6: Net-(D3-Pad6) -> Net-(D3-Pad10)
- U5 pad 7: Net-(R3-Pad1) -> Net-(D3-Pad6)
- U5 pad 8: /~ENABLE -> Net-(R3-Pad1)
- U5 pad 9: /SER_LINK_1 -> /~ENABLE
- Y1 pad 1: Net-(C1-Pad1) -> Net-(U1-Pad7)
- Y1 pad 2: Net-(C2-Pad1) -> GND
Routing:
- net /SER_CLK: track 0.00 -> 250.2 mm, vias 0 -> 4
- net /~ENABLE: track 4.68 -> 245.8 mm, vias 0 -> 4
- net /SER_LATCH: track 6.63 -> 241.8 mm, vias 0 -> 4
- net +5V: track 0.00 -> 220.3 mm, vias 0 -> 5
- net /E2_DIR: track 0.00 -> 152.7 mm
- net /E2_CLK: track 0.00 -> 146.2 mm
- net /E3_DIR: track 0.00 -> 129.9 mm
- net Net-(D1-Pad10): track 0.00 -> 116.8 mm, vias 0 -> 2
- net /E3_CLK: track 0.00 -> 115.1 mm
- net Net-(D1-Pad11): track 0.00 -> 113.0 mm, vias 0 -> 2
- net Net-(D1-Pad6): track 0.00 -> 109.0 mm, vias 0 -> 1
- net /SER_LINK_2: track 0.00 -> 105.4 mm, vias 0 -> 2
- net Net-(D1-Pad14): track 0.00 -> 104.1 mm, vias 0 -> 2
- net Net-(D4-Pad10): track 33.0 -> 120.7 mm
- net Net-(R10-Pad1): track 0.00 -> 81.7 mm, vias 0 -> 3
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Other:
- board text added: "Max Proskauer v2.0 Oct 2020 github.com/mprosk/mtg_life_counter"
- board text added: "Version 2.0"
- board text removed: "Max Proskauer v1.0 Oct 2020 github.com/mprosk/mtg_life_counter"
- board text removed: "Version 1.0"

Commit message: Tweak layout
Parts:
- moved C5 4.48 mm to (127.2, 81.3)
Connections:
- net /USB_DM renamed /USB_D_N
- net /USB_DP renamed /USB_D_P
Routing:
- net /E3_SW: track 0.00 -> 133.9 mm
- net /E2_SW: track 0.00 -> 118.2 mm
- net /SER_DATA: track 0.00 -> 106.8 mm, vias 0 -> 1
- net +5V: track 220.3 -> 281.0 mm, vias 5 -> 8
- net /USB_D_N: track 0.00 -> 15.0 mm
- net /USB_D_P: track 0.00 -> 13.5 mm
- net /SER_LINK_3: track 52.0 -> 54.7 mm
Other:
- net class USB added: clearance 0.2, trace_width 0.2, via_dia 0.8, via_drill 0.4
