File: pcb/mtg_life_counter.kicad_pcb (KiCad board)
At the start: 2 copper layers, 167.6 x 101.6 mm, 98 parts, among them J1 USB C 4907, J2 ICSP, J3 TP_UART, SW1 SW_SPST, SW2 SW_SPST, U1 ATmega328P-AU, U2 74HC595, U3 74HC595, U4 74HC595, U5 74HC595, U6 TPIC6B595, U7 TPIC6B595, U8 74HC165, Y1 16MHz

Commit message: Update to KiCad 8 and clean up files
Connections:
- net /~RESET renamed /~{RESET}
Other:
- net class Default removed
- net class Power removed
- net class USB removed

Commit message: wip on common cathode with transistors design
Parts:
- removed C10: 0.1uF, Capacitor_SMD:C_0805_2012Metric_Pad1.15x1.40mm_HandSolder
- removed E1, E2, E3, E4: Rotary_Encoder_Switch, mtg_life_counter:TT_EN11-HSB
- removed H4: MountingHole_Pad, MountingHole:MountingHole_3.2mm_M3_Pad_Via
- removed R50, R51, R52, R53, R54, R55, R56, R57: 10k, Resistor_SMD:R_0805_2012Metric_Pad1.15x1.40mm_HandSolder
- removed U8: 74HC165, Package_SO:SOIC-16_3.9x9.9mm_P1.27mm
- added B10: P4 DOWN, mtg_life_counter:B3F_12mm, F.Cu at (64.9, 142.3)
- added B3: P1 UP, mtg_life_counter:B3F_12mm, F.Cu at (43.0, 54.9)
- added B4: P1 DOWN, mtg_life_counter:B3F_12mm, F.Cu at (43.8, 74.7)
- added B5: P2 UP, mtg_life_counter:B3F_12mm, F.Cu at (10.5, 86.0)
- added B6: P2 DOWN, mtg_life_counter:B3F_12mm, F.Cu at (10.5, 99.2)
- added B7: P3 Up, mtg_life_counter:B3F_12mm, F.Cu at (10.5, 112.3)
- added B8: P3 DOWN, mtg_life_counter:B3F_12mm, F.Cu at (26.2, 59.7)
- added B9: P4 UP, mtg_life_counter:B3F_12mm, F.Cu at (64.9, 127.0)
- D1: value KW4-S561CxB RED SMD -> KW4-S561CVB RED SMD
- D2: value KW4-S561CxB GREEN SMD -> KW4-S561CGB GREEN SMD
- D3: value KW4-S561CxB YELLOW SMD -> KW4-S561CAB YELLOW SMD
- D4: value KW4-S561CxB BLUE SMD -> KW4-S561CBB BLUE SMD
- moved R2 13.5 mm to (81.3, 116.8)
Connections:
- net /RESET_BTN renamed /BTN_RESET
- net /ROLL_BTN renamed /BTN_ROLL
- H1 pad 1: Net-(H1-Pad1) -> unconnected-(H1-Pad1)_2
- H2 pad 1: Net-(H2-Pad1) -> unconnected-(H2-Pad1)_3
- H3 pad 1: Net-(H3-Pad1) -> unconnected-(H3-Pad1)_6
- U1 pad 10: Net-(U1-Pad10) -> unconnected-(U1-PD6-Pad10)
- U1 pad 2: Net-(U1-Pad2) -> unconnected-(U1-PD4-Pad2)
- U1 pad 23: Net-(U1-Pad23) -> unconnected-(U1-PC0(ADC0)-Pad23)
- U1 pad 24: Net-(U1-Pad24) -> unconnected-(U1-PC1(ADC1)-Pad24)
- U1 pad 25: /E2_SW -> unconnected-(U1-PC2(ADC2)-Pad25)
- U1 pad 26: Net-(U1-Pad26) -> unconnected-(U1-PC3(ADC3)-Pad26)
- U1 pad 27: Net-(U1-Pad27) -> unconnected-(U1-PC4(SDA/ADC4)-Pad27)
- U1 pad 28: /E1_SW -> unconnected-(U1-PC5(SCL/ADC5)-Pad28)
- U1 pad 32: /E4_SW -> unconnected-(U1-PD2(INT0)-Pad32)
- U1 pad 9: /E3_SW -> unconnected-(U1-PD5-Pad9)
- U2 pad 9: Net-(U2-Pad9) -> unconnected-(U2-QH&apos;-Pad9)
Routing:
- net (no net): track 0.00 -> 484.2 mm, vias 0 -> 4
- net /E4_CLK: track 197.2 -> 0.00 mm, vias 2 -> 0
- net /E1_DIR: track 195.9 -> 0.00 mm, vias 2 -> 0
- net /E4_DIR: track 194.7 -> 0.00 mm, vias 2 -> 0
- net /E1_CLK: track 193.4 -> 0.00 mm, vias 2 -> 0
- net /BTN_P4_DN: track 0.00 -> 184.6 mm, vias 0 -> 2
- net unconnected-(U1-PC2(ADC2)-Pad25): track 0.00 -> 168.9 mm, vias 0 -> 1
- net /E2_SW: track 168.9 -> 0.00 mm, vias 1 -> 0
- net unconnected-(U1-PD5-Pad9): track 0.00 -> 155.3 mm, vias 0 -> 1
- net /E3_SW: track 155.3 -> 0.00 mm, vias 1 -> 0
- net unconnected-(U1-PC5(SCL/ADC5)-Pad28): track 0.00 -> 43.8 mm
- net /E1_SW: track 43.8 -> 0.00 mm
- net /E4_SW: track 40.9 -> 0.00 mm
- net /E3_CLK: track 23.7 -> 0.00 mm
- net /E2_DIR: track 23.7 -> 0.00 mm
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
Commit message: tentative schematic for common cathode
Parts:
- removed the C4 at (114.9, 81.0)
- removed the C5 at (178.4, 81.0)
- removed the D1 at (102.9, 68.6)
- removed JP1: Jumper_2_Open, Jumper:SolderJumper-2_P1.3mm_Open_TrianglePad1.0x1.5mm
- removed JP2: JP_SR, mtg_life_counter:TP_Edge_2
- removed the R2 at (81.3, 116.8)
- removed the R3 at (89.8, 85.1)
- removed U6, U7: TPIC6B595, Package_SO:SOIC-20W_7.5x12.8mm_P1.27mm
- added D5: KW4-S561CBB BLUE SMD, mtg_life_counter:KW4-S561xxB_SMD, F.Cu at (102.9, 134.6)
- added H4: MountingHole_Pad, MountingHole:MountingHole_3.2mm_M3_Pad_Via, F.Cu at (-27.6, 80.2)
- added Q1: 2N7002K, Package_TO_SOT_SMD:SOT-23, F.Cu at (-33.9, 19.4)
- added Q10: BSS84, Package_TO_SOT_SMD:SOT-23, F.Cu at (-19.3, 19.4)
- added Q11: BSS84, Package_TO_SOT_SMD:SOT-23, F.Cu at (-19.3, 24.1)
- added Q12: BSS84, Package_TO_SOT_SMD:SOT-23, F.Cu at (-19.3, 28.7)
- added Q13: 2N7002K, Package_TO_SOT_SMD:SOT-23, F.Cu at (-87.1, 19.4)
- added Q14: 2N7002K, Package_TO_SOT_SMD:SOT-23, F.Cu at (-87.1, 24.1)
- added Q15: 2N7002K, Package_TO_SOT_SMD:SOT-23, F.Cu at (-87.1, 28.7)
- added Q16: 2N7002K, Package_TO_SOT_SMD:SOT-23, F.Cu at (-82.2, 19.4)
- added Q17: BSS84, Package_TO_SOT_SMD:SOT-23, F.Cu at (-82.2, 24.1)
- added Q18: BSS84, Package_TO_SOT_SMD:SOT-23, F.Cu at (-82.2, 28.7)
- added Q19: BSS84, Package_TO_SOT_SMD:SOT-23, F.Cu at (-77.3, 19.4)
- added Q2: 2N7002K, Package_TO_SOT_SMD:SOT-23, F.Cu at (-33.9, 24.1)
- added Q20: BSS84, Package_TO_SOT_SMD:SOT-23, F.Cu at (-77.3, 24.1)
- added Q21: BSS84, Package_TO_SOT_SMD:SOT-23, F.Cu at (-77.3, 28.7)
- added Q22: BSS84, Package_TO_SOT_SMD:SOT-23, F.Cu at (-72.4, 19.4)
- added Q23: BSS84, Package_TO_SOT_SMD:SOT-23, F.Cu at (-72.4, 24.1)
- added Q24: BSS84, Package_TO_SOT_SMD:SOT-23, F.Cu at (-72.4, 28.7)
- added Q25: 2N7002K, Package_TO_SOT_SMD:SOT-23, F.Cu at (-33.9, 61.9)
- added Q26: 2N7002K, Package_TO_SOT_SMD:SOT-23, F.Cu at (-33.9, 66.5)
- added Q27: 2N7002K, Package_TO_SOT_SMD:SOT-23, F.Cu at (-33.9, 71.2)
- added Q28: 2N7002K, Package_TO_SOT_SMD:SOT-23, F.Cu at (-29.0, 61.9)
- added Q29: BSS84, Package_TO_SOT_SMD:SOT-23, F.Cu at (-29.0, 66.5)
- added Q3: 2N7002K, Package_TO_SOT_SMD:SOT-23, F.Cu at (-33.9, 28.7)
- added Q30: BSS84, Package_TO_SOT_SMD:SOT-23, F.Cu at (-29.0, 71.2)
- added Q31: BSS84, Package_TO_SOT_SMD:SOT-23, F.Cu at (-24.1, 61.9)
- added Q32: BSS84, Package_TO_SOT_SMD:SOT-23, F.Cu at (-24.1, 66.5)
- added Q33: BSS84, Package_TO_SOT_SMD:SOT-23, F.Cu at (-24.1, 71.2)
- added Q34: BSS84, Package_TO_SOT_SMD:SOT-23, F.Cu at (-19.3, 61.9)
- added Q35: BSS84, Package_TO_SOT_SMD:SOT-23, F.Cu at (-19.3, 66.5)
- added Q36: BSS84, Package_TO_SOT_SMD:SOT-23, F.Cu at (-19.3, 71.2)
- added Q37: 2N7002K, Package_TO_SOT_SMD:SOT-23, F.Cu at (-87.1, 61.9)
- added Q38: 2N7002K, Package_TO_SOT_SMD:SOT-23, F.Cu at (-87.1, 66.5)
- added Q39: 2N7002K, Package_TO_SOT_SMD:SOT-23, F.Cu at (-87.1, 71.2)
- added Q4: 2N7002K, Package_TO_SOT_SMD:SOT-23, F.Cu at (-29.0, 19.4)
- added Q40: 2N7002K, Package_TO_SOT_SMD:SOT-23, F.Cu at (-82.2, 61.9)
- added Q41: BSS84, Package_TO_SOT_SMD:SOT-23, F.Cu at (-82.2, 66.5)
- added Q42: BSS84, Package_TO_SOT_SMD:SOT-23, F.Cu at (-82.2, 71.2)
- added Q43: BSS84, Package_TO_SOT_SMD:SOT-23, F.Cu at (-77.3, 61.9)
- added Q44: BSS84, Package_TO_SOT_SMD:SOT-23, F.Cu at (-77.3, 66.5)
- added Q45: BSS84, Package_TO_SOT_SMD:SOT-23, F.Cu at (-77.3, 71.2)
- added Q46: BSS84, Package_TO_SOT_SMD:SOT-23, F.Cu at (-72.4, 61.9)
- added Q47: BSS84, Package_TO_SOT_SMD:SOT-23, F.Cu at (-72.4, 66.5)
- added Q48: BSS84, Package_TO_SOT_SMD:SOT-23, F.Cu at (-72.4, 71.2)
- added Q5: BSS84, Package_TO_SOT_SMD:SOT-23, F.Cu at (-29.0, 24.1)
- added Q6: BSS84, Package_TO_SOT_SMD:SOT-23, F.Cu at (-29.0, 28.7)
- added Q7: BSS84, Package_TO_SOT_SMD:SOT-23, F.Cu at (-24.1, 19.4)
- added Q8: BSS84, Package_TO_SOT_SMD:SOT-23, F.Cu at (-24.1, 24.1)
- added Q9: BSS84, Package_TO_SOT_SMD:SOT-23, F.Cu at (-24.1, 28.7)
- added R18: 330R, Resistor_SMD:R_0805_2012Metric_Pad1.20x1.40mm_HandSolder, F.Cu at (-4.93, 18.5)
- added R19: 330R, Resistor_SMD:R_0805_2012Metric_Pad1.20x1.40mm_HandSolder, F.Cu at (-4.93, 21.5)
- added R28: 330R, Resistor_SMD:R_0805_2012Metric_Pad1.20x1.40mm_HandSolder, F.Cu at (-67.6, 18.5)
- added R29: 330R, Resistor_SMD:R_0805_2012Metric_Pad1.20x1.40mm_HandSolder, F.Cu at (-67.6, 21.5)
- added R38: 150R, Resistor_SMD:R_0805_2012Metric_Pad1.20x1.40mm_HandSolder, F.Cu at (-58.1, 18.5)
- added R39: 150R, Resistor_SMD:R_0805_2012Metric_Pad1.20x1.40mm_HandSolder, F.Cu at (-58.1, 21.5)
- added R48: 330R, Resistor_SMD:R_0805_2012Metric_Pad1.20x1.40mm_HandSolder, F.Cu at (-14.4, 61.0)
- added R49: 330R, Resistor_SMD:R_0805_2012Metric_Pad1.20x1.40mm_HandSolder, F.Cu at (-14.4, 63.9)
- added R50: 330R, Resistor_SMD:R_0805_2012Metric_Pad1.20x1.40mm_HandSolder, F.Cu at (-14.4, 66.9)
- added R51: 330R, Resistor_SMD:R_0805_2012Metric_Pad1.20x1.40mm_HandSolder, F.Cu at (-14.4, 69.8)
- added R52: 330R, Resistor_SMD:R_0805_2012Metric_Pad1.20x1.40mm_HandSolder, F.Cu at (-14.4, 72.8)
- added R53: 330R, Resistor_SMD:R_0805_2012Metric_Pad1.20x1.40mm_HandSolder, F.Cu at (-9.69, 61.0)
- added R54: 330R, Resistor_SMD:R_0805_2012Metric_Pad1.20x1.40mm_HandSolder, F.Cu at (-9.69, 63.9)
- added R55: 330R, Resistor_SMD:R_0805_2012Metric_Pad1.20x1.40mm_HandSolder, F.Cu at (-9.69, 66.9)
- added R56: 330R, Resistor_SMD:R_0805_2012Metric_Pad1.20x1.40mm_HandSolder, F.Cu at (-9.69, 69.8)
- added R57: 330R, Resistor_SMD:R_0805_2012Metric_Pad1.20x1.40mm_HandSolder, F.Cu at (-9.69, 72.8)
- added R58: 330R, Resistor_SMD:R_0805_2012Metric_Pad1.20x1.40mm_HandSolder, F.Cu at (-4.93, 61.0)
- added R59: 330R, Resistor_SMD:R_0805_2012Metric_Pad1.20x1.40mm_HandSolder, F.Cu at (-4.93, 63.9)
- added R60: 330R, Resistor_SMD:R_0805_2012Metric_Pad1.20x1.40mm_HandSolder, F.Cu at (-4.93, 66.9)
- added R61: 330R, Resistor_SMD:R_0805_2012Metric_Pad1.20x1.40mm_HandSolder, F.Cu at (-4.93, 69.8)
- added R62: 330R, Resistor_SMD:R_0805_2012Metric_Pad1.20x1.40mm_HandSolder, F.Cu at (-4.93, 72.8)
- added R63: 330R, Resistor_SMD:R_0805_2012Metric_Pad1.20x1.40mm_HandSolder, F.Cu at (-0.18, 61.0)
- added R64: 330R, Resistor_SMD:R_0805_2012Metric_Pad1.20x1.40mm_HandSolder, F.Cu at (-0.18, 63.9)
- added R65: 330R, Resistor_SMD:R_0805_2012Metric_Pad1.20x1.40mm_HandSolder, F.Cu at (-0.18, 66.9)
- added R66: 330R, Resistor_SMD:R_0805_2012Metric_Pad1.20x1.40mm_HandSolder, F.Cu at (-0.18, 69.8)
- added R67: 330R, Resistor_SMD:R_0805_2012Metric_Pad1.20x1.40mm_HandSolder, F.Cu at (-0.18, 72.8)
- added R68: 330R, Resistor_SMD:R_0805_2012Metric_Pad1.20x1.40mm_HandSolder, F.Cu at (-67.6, 61.0)
- added R69: 330R, Resistor_SMD:R_0805_2012Metric_Pad1.20x1.40mm_HandSolder, F.Cu at (-67.6, 63.9)
- added R7: 10k, Resistor_SMD:R_0805_2012Metric_Pad1.20x1.40mm_HandSolder, F.Cu at (-34.0, 86.6)
- added R70: 330R, Resistor_SMD:R_0805_2012Metric_Pad1.20x1.40mm_HandSolder, F.Cu at (-67.6, 66.9)
- added R71: 330R, Resistor_SMD:R_0805_2012Metric_Pad1.20x1.40mm_HandSolder, F.Cu at (-67.6, 69.8)
- added R72: 330R, Resistor_SMD:R_0805_2012Metric_Pad1.20x1.40mm_HandSolder, F.Cu at (-67.6, 72.8)
- added R73: 330R, Resistor_SMD:R_0805_2012Metric_Pad1.20x1.40mm_HandSolder, F.Cu at (-62.8, 61.0)
- added R74: 330R, Resistor_SMD:R_0805_2012Metric_Pad1.20x1.40mm_HandSolder, F.Cu at (-62.8, 63.9)
- added R75: 330R, Resistor_SMD:R_0805_2012Metric_Pad1.20x1.40mm_HandSolder, F.Cu at (-62.8, 66.9)
- added R76: 220R, Resistor_SMD:R_0805_2012Metric_Pad1.20x1.40mm_HandSolder, F.Cu at (-62.8, 69.8)
- added R77: 220R, Resistor_SMD:R_0805_2012Metric_Pad1.20x1.40mm_HandSolder, F.Cu at (-62.8, 72.8)
- added R78: 220R, Resistor_SMD:R_0805_2012Metric_Pad1.20x1.40mm_HandSolder, F.Cu at (-58.1, 61.0)
- added R79: 220R, Resistor_SMD:R_0805_2012Metric_Pad1.20x1.40mm_HandSolder, F.Cu at (-58.1, 63.9)
- added R8: 330R, Resistor_SMD:R_0805_2012Metric_Pad1.20x1.40mm_HandSolder, F.Cu at (-14.4, 18.5)
- added R80: 330R, Resistor_SMD:R_0805_2012Metric_Pad1.20x1.40mm_HandSolder, F.Cu at (-58.1, 66.9)
- added R81: 330R, Resistor_SMD:R_0805_2012Metric_Pad1.20x1.40mm_HandSolder, F.Cu at (-58.1, 69.8)
- added R82: 330R, Resistor_SMD:R_0805_2012Metric_Pad1.20x1.40mm_HandSolder, F.Cu at (-58.1, 72.8)
- added R83: 330R, Resistor_SMD:R_0805_2012Metric_Pad1.20x1.40mm_HandSolder, F.Cu at (-53.3, 61.0)
- added R84: 220R, Resistor_SMD:R_0805_2012Metric_Pad1.20x1.40mm_HandSolder, F.Cu at (-53.3, 63.9)
- added R85: 220R, Resistor_SMD:R_0805_2012Metric_Pad1.20x1.40mm_HandSolder, F.Cu at (-53.3, 66.9)
- added R86: 220R, Resistor_SMD:R_0805_2012Metric_Pad1.20x1.40mm_HandSolder, F.Cu at (-53.3, 69.8)
- added R87: 220R, Resistor_SMD:R_0805_2012Metric_Pad1.20x1.40mm_HandSolder, F.Cu at (-53.3, 72.8)
- added R9: 330R, Resistor_SMD:R_0805_2012Metric_Pad1.20x1.40mm_HandSolder, F.Cu at (-14.4, 21.5)
- C1, C2, C3, C6, C7, C8, C9: footprint Capacitor_SMD:C_0805_2012Metric_Pad1.15x1.40mm_HandSolder -> Capacitor_SMD:C_0805_2012Metric_Pad1.18x1.45mm_HandSolder
- C4: renamed from C11; footprint Capacitor_SMD:C_0805_2012Metric_Pad1.15x1.40mm_HandSolder -> Capacitor_SMD:C_0805_2012Metric_Pad1.18x1.45mm_HandSolder
- C5: renamed from C12; footprint Capacitor_SMD:C_0805_2012Metric_Pad1.15x1.40mm_HandSolder -> Capacitor_SMD:C_0805_2012Metric_Pad1.18x1.45mm_HandSolder
- D2: value KW4-S561CGB GREEN SMD -> KW4-S561CVB RED SMD
- D3: value KW4-S561CAB YELLOW SMD -> KW4-S561CGB GREEN SMD
- D4: value KW4-S561CBB BLUE SMD -> KW4-S561CAB YELLOW SMD
- R1, R4, R5: footprint Resistor_SMD:R_0805_2012Metric_Pad1.15x1.40mm_HandSolder -> Resistor_SMD:R_0805_2012Metric_Pad1.20x1.40mm_HandSolder
- R10, R11, R12, R13, R14, R15, R16, R17: value 330 -> 330R; footprint Resistor_SMD:R_0805_2012Metric_Pad1.15x1.40mm_HandSolder -> Resistor_SMD:R_0805_2012Metric_Pad1.20x1.40mm_HandSolder
- R2: renamed from R60; footprint Resistor_SMD:R_0805_2012Metric_Pad1.15x1.40mm_HandSolder -> Resistor_SMD:R_0805_2012Metric_Pad1.20x1.40mm_HandSolder
- R20, R21, R22, R23, R24, R25, R26, R27: value 10 -> 330R; footprint Resistor_SMD:R_0805_2012Metric_Pad1.15x1.40mm_HandSolder -> Resistor_SMD:R_0805_2012Metric_Pad1.20x1.40mm_HandSolder
- R3: renamed from R61; footprint Resistor_SMD:R_0805_2012Metric_Pad1.15x1.40mm_HandSolder -> Resistor_SMD:R_0805_2012Metric_Pad1.20x1.40mm_HandSolder
- R30, R31, R32, R33, R34, R35: value 100 -> 330R; footprint Resistor_SMD:R_0805_2012Metric_Pad1.15x1.40mm_HandSolder -> Resistor_SMD:R_0805_2012Metric_Pad1.20x1.40mm_HandSolder
- R36, R37: value 100 -> 150R; footprint Resistor_SMD:R_0805_2012Metric_Pad1.15x1.40mm_HandSolder -> Resistor_SMD:R_0805_2012Metric_Pad1.20x1.40mm_HandSolder
- R40, R41, R42, R43: value 390 -> 330R; footprint Resistor_SMD:R_0805_2012Metric_Pad1.15x1.40mm_HandSolder -> Resistor_SMD:R_0805_2012Metric_Pad1.20x1.40mm_HandSolder
- R44, R45, R46, R47: value 390 -> 150R; footprint Resistor_SMD:R_0805_2012Metric_Pad1.15x1.40mm_HandSolder -> Resistor_SMD:R_0805_2012Metric_Pad1.20x1.40mm_HandSolder
- R6: footprint Resistor_SMD:R_0805_2012Metric_Pad1.15x1.40mm_HandSolder -> Resistor_SMD:R_0805_2012Metric_Pad1.20x1.40mm_HandSolder; moved to F.Cu
- SW1, SW2: footprint Button_Switch_THT:SW_Slide_1P2T_CK_OS102011MS2Q -> Button_Switch_THT:SW_Slide_SPDT_Straight_CK_OS102011MS2Q
- Y1: footprint Crystal:Resonator_muRata_CSTLSxxxX-3Pin_W5.5mm_H3.0mm -> Crystal:Resonator_SMD-3Pin_7.2x3.0mm
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- renumbered B3 to B1, B4 to B2, B5 to B3, B6 to B4, B7 to B5, B8 to B6, B1 to B7, B2 to B8, D5 to D1
Connections:
- net /SER_LINK_3 renamed /SHIFT_CARRY_1
- net /SER_LINK_4 renamed /SHIFT_CARRY_2
- net /SER_LINK_5 renamed /SHIFT_CARRY_3
- net Net-(D2-DP) renamed /Player One Display Bank - Red/ANODE_DP
- net Net-(D2-e) renamed /Player One Display Bank - Red/ANODE_E
- net Net-(D2-f) renamed /Player One Display Bank - Red/ANODE_F
- net Net-(D2-g) renamed /Player One Display Bank - Red/ANODE_G
- D2 pad 11: Net-(D2-a) -> /Player One Display Bank - Red/ANODE_A
- D2 pad 12: Net-(D2-CC1) -> /Player One Display Bank - Red/CC1
- D2 pad 2: Net-(D2-d) -> /Player One Display Bank - Red/ANODE_D
- D2 pad 4: Net-(D2-c) -> /Player One Display Bank - Red/ANODE_C
- D2 pad 6: Net-(D2-CC4) -> /Player One Display Bank - Red/CC4
- D2 pad 7: Net-(D2-b) -> /Player One Display Bank - Red/ANODE_B
- D2 pad 8: Net-(D2-CC3) -> /Player One Display Bank - Red/CC3
- D2 pad 9: Net-(D2-CC2) -> /Player One Display Bank - Red/CC2
- D3 pad 1: Net-(D3-e) -> /Player Two Display Bank - Green/ANODE_E
- D3 pad 10: Net-(D3-f) -> /Player Two Display Bank - Green/ANODE_F
- D3 pad 11: Net-(D3-a) -> /Player Two Display Bank - Green/ANODE_A
- D3 pad 12: Net-(D3-CC1) -> /Player Two Display Bank - Green/CC1
- D3 pad 2: Net-(D3-d) -> /Player Two Display Bank - Green/ANODE_D
- D3 pad 3: Net-(D3-DP) -> /Player Two Display Bank - Green/ANODE_DP
- D3 pad 4: Net-(D3-c) -> /Player Two Display Bank - Green/ANODE_C
- D3 pad 5: Net-(D3-g) -> /Player Two Display Bank - Green/ANODE_G
- D3 pad 6: Net-(D3-CC4) -> /Player Two Display Bank - Green/CC4
- D3 pad 7: Net-(D3-b) -> /Player Two Display Bank - Green/ANODE_B
- D3 pad 8: Net-(D3-CC3) -> /Player Two Display Bank - Green/CC3
- D3 pad 9: Net-(D3-CC2) -> /Player Two Display Bank - Green/CC2
- D4 pad 1: Net-(D4-e) -> /Player Three Display Bank - Yellow/ANODE_E
- D4 pad 10: Net-(D4-f) -> /Player Three Display Bank - Yellow/ANODE_F
- D4 pad 11: Net-(D4-a) -> /Player Three Display Bank - Yellow/ANODE_A
- D4 pad 12: Net-(D4-CC1) -> /Player Three Display Bank - Yellow/CC1
- D4 pad 2: Net-(D4-d) -> /Player Three Display Bank - Yellow/ANODE_D
- D4 pad 3: Net-(D4-DP) -> /Player Three Display Bank - Yellow/ANODE_DP
- D4 pad 4: Net-(D4-c) -> /Player Three Display Bank - Yellow/ANODE_C
- D4 pad 5: Net-(D4-g) -> /Player Three Display Bank - Yellow/ANODE_G
- D4 pad 6: Net-(D4-CC4) -> /Player Three Display Bank - Yellow/CC4
- D4 pad 7: Net-(D4-b) -> /Player Three Display Bank - Yellow/ANODE_B
- D4 pad 8: Net-(D4-CC3) -> /Player Three Display Bank - Yellow/CC3
- D4 pad 9: Net-(D4-CC2) -> /Player Three Display Bank - Yellow/CC2
- J2 pad 1: /SER_CIPO -> /CIPO
- J2 pad 3: /SER_CLK -> /SCLK
- J2 pad 4: /SER_COPI -> /COPI
- R10 pad 1: Net-(U2-QA) -> /DIGIT_SEL_3
- R11 pad 1: Net-(U2-QB) -> /DIGIT_SEL_4
- R12 pad 1: Net-(U2-QC) -> /Player One Display Bank - Red/SEG_A
- R13 pad 1: Net-(U2-QD) -> /Player One Display Bank - Red/SEG_B
- R14 pad 1: Net-(U2-QE) -> /Player One Display Bank - Red/SEG_C
- R15 pad 1: Net-(U2-QF) -> /Player One Display Bank - Red/SEG_D
- R16 pad 1: Net-(U2-QG) -> Net-(Q5-S)
- R16 pad 2: Net-(D1-g) -> /Player One Display Bank - Red/ANODE_A
- R17 pad 1: Net-(U2-QH) -> Net-(Q6-S)
- R17 pad 2: Net-(D1-DP) -> /Player One Display Bank - Red/ANODE_B
- R20 pad 1: Net-(U3-QA) -> /Player One Display Bank - Red/SEG_E
- R20 pad 2: Net-(D2-a) -> Net-(Q9-G)
- R21 pad 1: Net-(U3-QB) -> /Player One Display Bank - Red/SEG_F
- R21 pad 2: Net-(D2-b) -> Net-(Q10-G)
- R22 pad 1: Net-(U3-QC) -> /Player One Display Bank - Red/SEG_G
- R22 pad 2: Net-(D2-c) -> Net-(Q11-G)
- R23 pad 1: Net-(U3-QD) -> /Player One Display Bank - Red/SEG_DP
- R23 pad 2: Net-(D2-d) -> Net-(Q12-G)
- R24 pad 1: Net-(U3-QE) -> Net-(Q9-S)
- R25 pad 1: Net-(U3-QF) -> Net-(Q10-S)
- R26 pad 1: Net-(U3-QG) -> Net-(Q11-S)
- R27 pad 1: Net-(U3-QH) -> Net-(Q12-S)
- R30 pad 1: Net-(U4-QA) -> /DIGIT_SEL_3
- R30 pad 2: Net-(D3-a) -> Net-(Q15-G)
- R31 pad 1: Net-(U4-QB) -> /DIGIT_SEL_4
- R31 pad 2: Net-(D3-b) -> Net-(Q16-G)
- R32 pad 1: Net-(U4-QC) -> /Player Two Display Bank - Green/SEG_A
- R32 pad 2: Net-(D3-c) -> Net-(Q17-G)
- R33 pad 1: Net-(U4-QD) -> /Player Two Display Bank - Green/SEG_B
- R33 pad 2: Net-(D3-d) -> Net-(Q18-G)
- R34 pad 1: Net-(U4-QE) -> /Player Two Display Bank - Green/SEG_C
- R34 pad 2: Net-(D3-e) -> Net-(Q19-G)
- R35 pad 1: Net-(U4-QF) -> /Player Two Display Bank - Green/SEG_D
- R35 pad 2: Net-(D3-f) -> Net-(Q20-G)
- R36 pad 1: Net-(U4-QG) -> Net-(Q17-S)
- R36 pad 2: Net-(D3-g) -> /Player Two Display Bank - Green/ANODE_A
- R37 pad 1: Net-(U4-QH) -> Net-(Q18-S)
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Routing:
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
Commit message: common anode schematic
Parts:
- removed C6, C7, C8, C9: 0.1uF, Capacitor_SMD:C_0805_2012Metric_Pad1.18x1.45mm_HandSolder
- removed Q17, Q18, Q19, Q20, Q21, Q22, Q23, Q24, Q29, Q30, Q31, Q32, Q33, Q34, Q35, Q36, Q41, Q42, Q43, Q44, Q45, Q46, Q47, Q48: BSS84, Package_TO_SOT_SMD:SOT-23
- removed Q25, Q26, Q27, Q28, Q37, Q38, Q39, Q40: 2N7002K, Package_TO_SOT_SMD:SOT-23
- removed R60, R61, R62, R63, R64, R65, R66, R67, R68, R69, R70, R71, R72, R73, R74, R75, R80, R81, R82, R83: 330R, Resistor_SMD:R_0805_2012Metric_Pad1.20x1.40mm_HandSolder
- removed R76, R77, R78, R79, R84, R85, R86, R87: 220R, Resistor_SMD:R_0805_2012Metric_Pad1.20x1.40mm_HandSolder
- D2: value KW4-S561CVB RED SMD -> KW4-S561AVB
- D3: value KW4-S561CGB GREEN SMD -> KW4-S561AGB
- D4: value KW4-S561CAB YELLOW SMD -> KW4-S561AAB
- D5: value KW4-S561CBB BLUE SMD -> KW4-S561ABB
- Q1, Q13, Q14, Q15, Q16, Q2, Q3, Q4: value 2N7002K -> DMG2301L
- Q10, Q11, Q12, Q5, Q6, Q7, Q8, Q9: value BSS84 -> DMG2301L
- R20, R33, R59: value 330R -> 10k
- R25, R26, R27, R28, R29, R30, R31, R32: value 330R -> 150R
- R36, R37, R38, R39, R44, R45, R47: value 150R -> 330R
- R46: value 150R -> 10k
- R51, R52, R53, R54, R55, R56, R57, R58: value 330R -> 220R
- U2, U3, U4, U5: value 74HC595 -> TPIC6C596
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- renumbered B8 to B10, B9 to B7, B10 to B8, B7 to B9
Connections:
- D2 pad 1: /Player One Display Bank - Red/ANODE_E -> /Player One Display Bank - Red/AE
- D2 pad 10: /Player One Display Bank - Red/ANODE_F -> /Player One Display Bank - Red/AF
- D2 pad 11: /Player One Display Bank - Red/ANODE_A -> /Player One Display Bank - Red/AA
- D2 pad 12: /Player One Display Bank - Red/CC1 -> /Player One Display Bank - Red/CA1
- D2 pad 2: /Player One Display Bank - Red/ANODE_D -> /Player One Display Bank - Red/AD
- D2 pad 3: /Player One Display Bank - Red/ANODE_DP -> /Player One Display Bank - Red/ADP
- D2 pad 4: /Player One Display Bank - Red/ANODE_C -> /Player One Display Bank - Red/AC
- D2 pad 5: /Player One Display Bank - Red/ANODE_G -> /Player One Display Bank - Red/AG
- D2 pad 6: /Player One Display Bank - Red/CC4 -> /Player One Display Bank - Red/CA4
- D2 pad 7: /Player One Display Bank - Red/ANODE_B -> /Player One Display Bank - Red/AB
- D2 pad 8: /Player One Display Bank - Red/CC3 -> /Player One Display Bank - Red/CA3
- D2 pad 9: /Player One Display Bank - Red/CC2 -> /Player One Display Bank - Red/CA2
- D3 pad 1: /Player Two Display Bank - Green/ANODE_E -> /Player Two Display Bank - Green/AE
- D3 pad 10: /Player Two Display Bank - Green/ANODE_F -> /Player Two Display Bank - Green/AF
- D3 pad 11: /Player Two Display Bank - Green/ANODE_A -> /Player Two Display Bank - Green/AA
- D3 pad 12: /Player Two Display Bank - Green/CC1 -> /Player Two Display Bank - Green/CA1
- D3 pad 2: /Player Two Display Bank - Green/ANODE_D -> /Player Two Display Bank - Green/AD
- D3 pad 3: /Player Two Display Bank - Green/ANODE_DP -> /Player Two Display Bank - Green/ADP
- D3 pad 4: /Player Two Display Bank - Green/ANODE_C -> /Player Two Display Bank - Green/AC
- D3 pad 5: /Player Two Display Bank - Green/ANODE_G -> /Player Two Display Bank - Green/AG
- D3 pad 6: /Player Two Display Bank - Green/CC4 -> /Player Two Display Bank - Green/CA4
- D3 pad 7: /Player Two Display Bank - Green/ANODE_B -> /Player Two Display Bank - Green/AB
- D3 pad 8: /Player Two Display Bank - Green/CC3 -> /Player Two Display Bank - Green/CA3
- D3 pad 9: /Player Two Display Bank - Green/CC2 -> /Player Two Display Bank - Green/CA2
- D4 pad 1: /Player Three Display Bank - Yellow/ANODE_E -> /Player Three Display Bank - Yellow/AE
- D4 pad 10: /Player Three Display Bank - Yellow/ANODE_F -> /Player Three Display Bank - Yellow/AF
- D4 pad 11: /Player Three Display Bank - Yellow/ANODE_A -> /Player Three Display Bank - Yellow/AA
- D4 pad 12: /Player Three Display Bank - Yellow/CC1 -> /Player Three Display Bank - Yellow/CA1
- D4 pad 2: /Player Three Display Bank - Yellow/ANODE_D -> /Player Three Display Bank - Yellow/AD
- D4 pad 3: /Player Three Display Bank - Yellow/ANODE_DP -> /Player Three Display Bank - Yellow/ADP
- D4 pad 4: /Player Three Display Bank - Yellow/ANODE_C -> /Player Three Display Bank - Yellow/AC
- D4 pad 5: /Player Three Display Bank - Yellow/ANODE_G -> /Player Three Display Bank - Yellow/AG
- D4 pad 6: /Player Three Display Bank - Yellow/CC4 -> /Player Three Display Bank - Yellow/CA4
- D4 pad 7: /Player Three Display Bank - Yellow/ANODE_B -> /Player Three Display Bank - Yellow/AB
- D4 pad 8: /Player Three Display Bank - Yellow/CC3 -> /Player Three Display Bank - Yellow/CA3
- D4 pad 9: /Player Three Display Bank - Yellow/CC2 -> /Player Three Display Bank - Yellow/CA2
- D5 pad 1: /Player Four Display Bank - Blue/ANODE_E -> /Player Four Display Bank - Blue/AE
- D5 pad 10: /Player Four Display Bank - Blue/ANODE_F -> /Player Four Display Bank - Blue/AF
- D5 pad 11: /Player Four Display Bank - Blue/ANODE_A -> /Player Four Display Bank - Blue/AA
- D5 pad 12: /Player Four Display Bank - Blue/CC1 -> /Player Four Display Bank - Blue/CA1
- D5 pad 2: /Player Four Display Bank - Blue/ANODE_D -> /Player Four Display Bank - Blue/AD
- D5 pad 3: /Player Four Display Bank - Blue/ANODE_DP -> /Player Four Display Bank - Blue/ADP
- D5 pad 4: /Player Four Display Bank - Blue/ANODE_C -> /Player Four Display Bank - Blue/AC
- D5 pad 5: /Player Four Display Bank - Blue/ANODE_G -> /Player Four Display Bank - Blue/AG
- D5 pad 6: /Player Four Display Bank - Blue/CC4 -> /Player Four Display Bank - Blue/CA4
- D5 pad 7: /Player Four Display Bank - Blue/ANODE_B -> /Player Four Display Bank - Blue/AB
- D5 pad 8: /Player Four Display Bank - Blue/CC3 -> /Player Four Display Bank - Blue/CA3
- D5 pad 9: /Player Four Display Bank - Blue/CC2 -> /Player Four Display Bank - Blue/CA2
- Q1 pad 2: GND -> /Player One Display Bank - Red/CA1
- Q1 pad 3: /Player One Display Bank - Red/CC1 -> +5V
- Q10 pad 2: Net-(Q10-S) -> /Player Three Display Bank - Yellow/CA2
- Q11 pad 2: Net-(Q11-S) -> /Player Three Display Bank - Yellow/CA3
- Q12 pad 2: Net-(Q12-S) -> /Player Three Display Bank - Yellow/CA4
- Q13 pad 2: GND -> /Player Four Display Bank - Blue/CA1
- Q13 pad 3: /Player Two Display Bank - Green/CC1 -> +5V
- Q14 pad 2: GND -> /Player Four Display Bank - Blue/CA2
- Q14 pad 3: /Player Two Display Bank - Green/CC2 -> +5V
- Q15 pad 2: GND -> /Player Four Display Bank - Blue/CA3
- Q15 pad 3: /Player Two Display Bank - Green/CC3 -> +5V
- Q16 pad 2: GND -> /Player Four Display Bank - Blue/CA4
- Q16 pad 3: /Player Two Display Bank - Green/CC4 -> +5V
- Q2 pad 2: GND -> /Player One Display Bank - Red/CA2
- Q2 pad 3: /Player One Display Bank - Red/CC2 -> +5V
- Q3 pad 2: GND -> /Player One Display Bank - Red/CA3
- Q3 pad 3: /Player One Display Bank - Red/CC3 -> +5V
- Q4 pad 2: GND -> /Player One Display Bank - Red/CA4
- Q4 pad 3: /Player One Display Bank - Red/CC4 -> +5V
- Q5 pad 2: Net-(Q5-S) -> /Player Two Display Bank - Green/CA1
- Q6 pad 2: Net-(Q6-S) -> /Player Two Display Bank - Green/CA2
- Q7 pad 2: Net-(Q7-S) -> /Player Two Display Bank - Green/CA3
- Q8 pad 2: Net-(Q8-S) -> /Player Two Display Bank - Green/CA4
- Q9 pad 2: Net-(Q9-S) -> /Player Three Display Bank - Yellow/CA1
- R12 pad 1: /Player One Display Bank - Red/SEG_A -> /Player One Display Bank - Red/AA
- R12 pad 2: Net-(Q5-G) -> /Player One Display Bank - Red/SA
- R13 pad 1: /Player One Display Bank - Red/SEG_B -> /Player One Display Bank - Red/AB
- R13 pad 2: Net-(Q6-G) -> /Player One Display Bank - Red/SB
- R14 pad 1: /Player One Display Bank - Red/SEG_C -> /Player One Display Bank - Red/AC
- R14 pad 2: Net-(Q7-G) -> /Player One Display Bank - Red/SC
- R15 pad 1: /Player One Display Bank - Red/SEG_D -> /Player One Display Bank - Red/AD
- R15 pad 2: Net-(Q8-G) -> /Player One Display Bank - Red/SD
- R16 pad 1: Net-(Q5-S) -> /Player One Display Bank - Red/AE
- R16 pad 2: /Player One Display Bank - Red/ANODE_A -> /Player One Display Bank - Red/SE
- R17 pad 1: Net-(Q6-S) -> /Player One Display Bank - Red/AF
- R17 pad 2: /Player One Display Bank - Red/ANODE_B -> /Player One Display Bank - Red/SF
- R18 pad 1: Net-(Q7-S) -> /Player One Display Bank - Red/AG
- R18 pad 2: /Player One Display Bank - Red/ANODE_C -> /Player One Display Bank - Red/SG
- R19 pad 1: Net-(Q8-S) -> /Player One Display Bank - Red/ADP
- R19 pad 2: /Player One Display Bank - Red/ANODE_D -> /Player One Display Bank - Red/SDP
- R20 pad 1: /Player One Display Bank - Red/SEG_E -> +5V
- R20 pad 2: Net-(Q9-G) -> Net-(U2-~{SRCLR})
- R21 pad 1: /Player One Display Bank - Red/SEG_F -> /DIGIT_SEL_1
- R21 pad 2: Net-(Q10-G) -> Net-(Q5-G)
- R22 pad 1: /Player One Display Bank - Red/SEG_G -> /DIGIT_SEL_2
- R22 pad 2: Net-(Q11-G) -> Net-(Q6-G)
- R23 pad 1: /Player One Display Bank - Red/SEG_DP -> /DIGIT_SEL_3
- R23 pad 2: Net-(Q12-G) -> Net-(Q7-G)
- R24 pad 1: Net-(Q9-S) -> /DIGIT_SEL_4
- R24 pad 2: /Player One Display Bank - Red/ANODE_E -> Net-(Q8-G)
- R25 pad 1: Net-(Q10-S) -> /Player Two Display Bank - Green/AA
- R25 pad 2: /Player One Display Bank - Red/ANODE_F -> /Player Two Display Bank - Green/SA
- R26 pad 1: Net-(Q11-S) -> /Player Two Display Bank - Green/AB
- R26 pad 2: /Player One Display Bank - Red/ANODE_G -> /Player Two Display Bank - Green/SB
- R27 pad 1: Net-(Q12-S) -> /Player Two Display Bank - Green/AC
- R27 pad 2: /Player One Display Bank - Red/ANODE_DP -> /Player Two Display Bank - Green/SC
- R28 pad 1: /DIGIT_SEL_1 -> /Player Two Display Bank - Green/AD
- R28 pad 2: Net-(Q13-G) -> /Player Two Display Bank - Green/SD
- R29 pad 1: /DIGIT_SEL_2 -> /Player Two Display Bank - Green/AE
- R29 pad 2: Net-(Q14-G) -> /Player Two Display Bank - Green/SE
- R30 pad 1: /DIGIT_SEL_3 -> /Player Two Display Bank - Green/AF
- R30 pad 2: Net-(Q15-G) -> /Player Two Display Bank - Green/SF
- R31 pad 1: /DIGIT_SEL_4 -> /Player Two Display Bank - Green/AG
- R31 pad 2: Net-(Q16-G) -> /Player Two Display Bank - Green/SG
- R32 pad 1: /Player Two Display Bank - Green/SEG_A -> /Player Two Display Bank - Green/ADP
- R32 pad 2: Net-(Q17-G) -> /Player Two Display Bank - Green/SDP
- R33 pad 1: /Player Two Display Bank - Green/SEG_B -> +5V
- R33 pad 2: Net-(Q18-G) -> Net-(U3-~{SRCLR})
- R34 pad 1: /Player Two Display Bank - Green/SEG_C -> /DIGIT_SEL_1
- R34 pad 2: Net-(Q19-G) -> Net-(Q9-G)
- R35 pad 1: /Player Two Display Bank - Green/SEG_D -> /DIGIT_SEL_2
- R35 pad 2: Net-(Q20-G) -> Net-(Q10-G)
- R36 pad 1: Net-(Q17-S) -> /DIGIT_SEL_3
- R36 pad 2: /Player Two Display Bank - Green/ANODE_A -> Net-(Q11-G)
- R37 pad 1: Net-(Q18-S) -> /DIGIT_SEL_4
- R37 pad 2: /Player Two Display Bank - Green/ANODE_B -> Net-(Q12-G)
- R38 pad 1: Net-(Q19-S) -> /Player Three Display Bank - Yellow/AA
- R38 pad 2: /Player Two Display Bank - Green/ANODE_C -> /Player Three Display Bank - Yellow/SA
- R39 pad 1: Net-(Q20-S) -> /Player Three Display Bank - Yellow/AB
- R39 pad 2: /Player Two Display Bank - Green/ANODE_D -> /Player Three Display Bank - Yellow/SB
- R40 pad 1: /Player Two Display Bank - Green/SEG_E -> /Player Three Display Bank - Yellow/AC
- R40 pad 2: Net-(Q21-G) -> /Player Three Display Bank - Yellow/SC
- R41 pad 1: /Player Two Display Bank - Green/SEG_F -> /Player Three Display Bank - Yellow/AD
- R41 pad 2: Net-(Q22-G) -> /Player Three Display Bank - Yellow/SD
- R42 pad 1: /Player Two Display Bank - Green/SEG_G -> /Player Three Display Bank - Yellow/AE
- R42 pad 2: Net-(Q23-G) -> /Player Three Display Bank - Yellow/SE
- R43 pad 1: /Player Two Display Bank - Green/SEG_DP -> /Player Three Display Bank - Yellow/AF
- R43 pad 2: Net-(Q24-G) -> /Player Three Display Bank - Yellow/SF
- R44 pad 1: Net-(Q21-S) -> /Player Three Display Bank - Yellow/AG
- R44 pad 2: /Player Two Display Bank - Green/ANODE_E -> /Player Three Display Bank - Yellow/SG
- R45 pad 1: Net-(Q22-S) -> /Player Three Display Bank - Yellow/ADP
- R45 pad 2: /Player Two Display Bank - Green/ANODE_F -> /Player Three Display Bank - Yellow/SDP
- R46 pad 1: Net-(Q23-S) -> +5V
- R46 pad 2: /Player Two Display Bank - Green/ANODE_G -> Net-(U4-~{SRCLR})
- R47 pad 1: Net-(Q24-S) -> /DIGIT_SEL_1
- R47 pad 2: /Player Two Display Bank - Green/ANODE_DP -> Net-(Q13-G)
- R48 pad 1: /DIGIT_SEL_1 -> /DIGIT_SEL_2
- R48 pad 2: Net-(Q25-G) -> Net-(Q14-G)
- R49 pad 1: /DIGIT_SEL_2 -> /DIGIT_SEL_3
- R49 pad 2: Net-(Q26-G) -> Net-(Q15-G)
- R50 pad 1: /DIGIT_SEL_3 -> /DIGIT_SEL_4
- R50 pad 2: Net-(Q27-G) -> Net-(Q16-G)
- R51 pad 1: /DIGIT_SEL_4 -> /Player Four Display Bank - Blue/AA
- R51 pad 2: Net-(Q28-G) -> /Player Four Display Bank - Blue/SA
- R52 pad 1: /Player Three Display Bank - Yellow/SEG_A -> /Player Four Display Bank - Blue/AB
- R52 pad 2: Net-(Q29-G) -> /Player Four Display Bank - Blue/SB
- R53 pad 1: /Player Three Display Bank - Yellow/SEG_B -> /Player Four Display Bank - Blue/AC
- R53 pad 2: Net-(Q30-G) -> /Player Four Display Bank - Blue/SC
- R54 pad 1: /Player Three Display Bank - Yellow/SEG_C -> /Player Four Display Bank - Blue/AD
- R54 pad 2: Net-(Q31-G) -> /Player Four Display Bank - Blue/SD
- R55 pad 1: /Player Three Display Bank - Yellow/SEG_D -> /Player Four Display Bank - Blue/AE
- R55 pad 2: Net-(Q32-G) -> /Player Four Display Bank - Blue/SE
- R56 pad 1: Net-(Q29-S) -> /Player Four Display Bank - Blue/AF
- R56 pad 2: /Player Three Display Bank - Yellow/ANODE_A -> /Player Four Display Bank - Blue/SF
- R57 pad 1: Net-(Q30-S) -> /Player Four Display Bank - Blue/AG
- R57 pad 2: /Player Three Display Bank - Yellow/ANODE_B -> /Player Four Display Bank - Blue/SG
- R58 pad 1: Net-(Q31-S) -> /Player Four Display Bank - Blue/ADP
- R58 pad 2: /Player Three Display Bank - Yellow/ANODE_C -> /Player Four Display Bank - Blue/SDP
- R59 pad 1: Net-(Q32-S) -> +5V
- R59 pad 2: /Player Three Display Bank - Yellow/ANODE_D -> Net-(U5-~{SRCLR})
- U2 pad 1: /Player One Display Bank - Red/SEG_B -> +5V
- U2 pad 10: +5V -> /LATCH
- U2 pad 11: /SCLK -> /Player One Display Bank - Red/SE
- U2 pad 12: /LATCH -> /Player One Display Bank - Red/SF
- U2 pad 13: GND -> /Player One Display Bank - Red/SG
- U2 pad 14: /SHIFT_CARRY_3 -> /Player One Display Bank - Red/SDP
- U2 pad 15: /Player One Display Bank - Red/SEG_A -> /SCLK
- U2 pad 16: +5V -> GND
- U2 pad 2: /Player One Display Bank - Red/SEG_C -> /SHIFT_CARRY_3
- U2 pad 3: /Player One Display Bank - Red/SEG_D -> /Player One Display Bank - Red/SA
- U2 pad 4: /Player One Display Bank - Red/SEG_E -> /Player One Display Bank - Red/SB
- U2 pad 5: /Player One Display Bank - Red/SEG_F -> /Player One Display Bank - Red/SC
- U2 pad 6: /Player One Display Bank - Red/SEG_G -> /Player One Display Bank - Red/SD
- U2 pad 7: /Player One Display Bank - Red/SEG_DP -> Net-(U2-~{SRCLR})
- U3 pad 1: /Player Two Display Bank - Green/SEG_B -> +5V
- U3 pad 10: +5V -> /LATCH
- U3 pad 11: /SCLK -> /Player Two Display Bank - Green/SE
- U3 pad 12: /LATCH -> /Player Two Display Bank - Green/SF
- U3 pad 13: GND -> /Player Two Display Bank - Green/SG
- U3 pad 14: /SHIFT_CARRY_2 -> /Player Two Display Bank - Green/SDP
- U3 pad 15: /Player Two Display Bank - Green/SEG_A -> /SCLK
- U3 pad 16: +5V -> GND
- U3 pad 2: /Player Two Display Bank - Green/SEG_C -> /SHIFT_CARRY_2
- U3 pad 3: /Player Two Display Bank - Green/SEG_D -> /Player Two Display Bank - Green/SA
- U3 pad 4: /Player Two Display Bank - Green/SEG_E -> /Player Two Display Bank - Green/SB
- U3 pad 5: /Player Two Display Bank - Green/SEG_F -> /Player Two Display Bank - Green/SC
- U3 pad 6: /Player Two Display Bank - Green/SEG_G -> /Player Two Display Bank - Green/SD
- U3 pad 7: /Player Two Display Bank - Green/SEG_DP -> Net-(U3-~{SRCLR})
- U4 pad 1: /Player Three Display Bank - Yellow/SEG_B -> +5V
- U4 pad 10: +5V -> /LATCH
- U4 pad 11: /SCLK -> /Player Three Display Bank - Yellow/SE
- U4 pad 12: /LATCH -> /Player Three Display Bank - Yellow/SF
- U4 pad 13: GND -> /Player Three Display Bank - Yellow/SG
- U4 pad 14: /SHIFT_CARRY_1 -> /Player Three Display Bank - Yellow/SDP
- U4 pad 15: /Player Three Display Bank - Yellow/SEG_A -> /SCLK
- U4 pad 16: +5V -> GND
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
Commit message: continue wip
Parts:
- added C6: 0.1uF, Capacitor_SMD:C_0805_2012Metric_Pad1.18x1.45mm_HandSolder, F.Cu at (82.3, 35.6)
- added C7: 0.1uF, Capacitor_SMD:C_0805_2012Metric_Pad1.18x1.45mm_HandSolder, F.Cu at (193.3, 40.7)
- added C8: 0.1uF, Capacitor_SMD:C_0805_2012Metric_Pad1.18x1.45mm_HandSolder, F.Cu at (175.3, 176.5)
- added C9: 0.1uF, Capacitor_SMD:C_0805_2012Metric_Pad1.18x1.45mm_HandSolder, F.Cu at (106.7, 175.3)
- moved Q5 235.2 mm to (160.6, 30.6)
- moved Q6 235.2 mm to (160.6, 35.2)
- moved Q7 235.2 mm to (160.6, 39.8)
- moved Q8 235.2 mm to (160.6, 44.5)
- moved R21 235.2 mm to (165.4, 29.7)
- moved R22 235.2 mm to (165.4, 32.6)
- moved R23 235.2 mm to (165.4, 35.6)
- moved R24 235.2 mm to (165.4, 38.5)
- moved R26 235.2 mm to (170.2, 29.7)
- moved R27 235.2 mm to (170.2, 32.6)
- moved R28 235.2 mm to (170.2, 35.6)
- moved R29 235.2 mm to (170.2, 38.5)
- moved R31 235.2 mm to (174.9, 29.7)
- moved R32 235.2 mm to (174.9, 32.6)
- moved R33 235.2 mm to (174.9, 35.6)
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Connections:
- net /Player Four Display Bank - Blue/AA renamed /P4/AA
- net /Player Four Display Bank - Blue/AB renamed /P4/AB
- net /Player Four Display Bank - Blue/AC renamed /P4/AC
- net /Player Four Display Bank - Blue/AD renamed /P4/AD
- net /Player Four Display Bank - Blue/ADP renamed /P4/ADP
- net /Player Four Display Bank - Blue/AE renamed /P4/AE
- net /Player Four Display Bank - Blue/AF renamed /P4/AF
- net /Player Four Display Bank - Blue/AG renamed /P4/AG
- net /Player Four Display Bank - Blue/CA1 renamed /P4/CA1
- net /Player Four Display Bank - Blue/CA2 renamed /P4/CA2
- net /Player Four Display Bank - Blue/CA3 renamed /P4/CA3
- net /Player Four Display Bank - Blue/CA4 renamed /P4/CA4
- net /Player Four Display Bank - Blue/SA renamed /P4/SA
- net /Player Four Display Bank - Blue/SB renamed /P4/SB
- net /Player Four Display Bank - Blue/SC renamed /P4/SC
- net /Player Four Display Bank - Blue/SD renamed /P4/SD
- net /Player Four Display Bank - Blue/SDP renamed /P4/SDP
- net /Player Four Display Bank - Blue/SE renamed /P4/SE
- net /Player Four Display Bank - Blue/SF renamed /P4/SF
- net /Player Four Display Bank - Blue/SG renamed /P4/SG
- net /Player One Display Bank - Red/AA renamed /P1/AA
- net /Player One Display Bank - Red/AB renamed /P1/AB
- net /Player One Display Bank - Red/AC renamed /P1/AC
- net /Player One Display Bank - Red/AD renamed /P1/AD
- net /Player One Display Bank - Red/ADP renamed /P1/ADP
- net /Player One Display Bank - Red/AE renamed /P1/AE
- net /Player One Display Bank - Red/AF renamed /P1/AF
- net /Player One Display Bank - Red/AG renamed /P1/AG
- net /Player One Display Bank - Red/CA1 renamed /P1/CA1
- net /Player One Display Bank - Red/CA2 renamed /P1/CA2
- net /Player One Display Bank - Red/CA3 renamed /P1/CA3
- net /Player One Display Bank - Red/CA4 renamed /P1/CA4
- net /Player One Display Bank - Red/SA renamed /P1/SA
- net /Player One Display Bank - Red/SB renamed /P1/SB
- net /Player One Display Bank - Red/SC renamed /P1/SC
- net /Player One Display Bank - Red/SD renamed /P1/SD
- net /Player One Display Bank - Red/SDP renamed /P1/SDP
- net /Player One Display Bank - Red/SE renamed /P1/SE
- net /Player One Display Bank - Red/SF renamed /P1/SF
- net /Player One Display Bank - Red/SG renamed /P1/SG
- net /Player One Display Bank - Red/SHIFT_OUT renamed /P1/SHIFT_OUT
- net /Player Three Display Bank - Yellow/AA renamed /P3/AA
- net /Player Three Display Bank - Yellow/AB renamed /P3/AB
- net /Player Three Display Bank - Yellow/AC renamed /P3/AC
- net /Player Three Display Bank - Yellow/AD renamed /P3/AD
- net /Player Three Display Bank - Yellow/ADP renamed /P3/ADP
- net /Player Three Display Bank - Yellow/AE renamed /P3/AE
- net /Player Three Display Bank - Yellow/AF renamed /P3/AF
- net /Player Three Display Bank - Yellow/AG renamed /P3/AG
- net /Player Three Display Bank - Yellow/CA1 renamed /P3/CA1
- net /Player Three Display Bank - Yellow/CA2 renamed /P3/CA2
- net /Player Three Display Bank - Yellow/CA3 renamed /P3/CA3
- net /Player Three Display Bank - Yellow/CA4 renamed /P3/CA4
- net /Player Three Display Bank - Yellow/SA renamed /P3/SA
- net /Player Three Display Bank - Yellow/SB renamed /P3/SB
- net /Player Three Display Bank - Yellow/SC renamed /P3/SC
- net /Player Three Display Bank - Yellow/SD renamed /P3/SD
- net /Player Three Display Bank - Yellow/SDP renamed /P3/SDP
- net /Player Three Display Bank - Yellow/SE renamed /P3/SE
- net /Player Three Display Bank - Yellow/SF renamed /P3/SF
- net /Player Three Display Bank - Yellow/SG renamed /P3/SG
- net /Player Two Display Bank - Green/AA renamed /P2/AA
- net /Player Two Display Bank - Green/AB renamed /P2/AB
- net /Player Two Display Bank - Green/AC renamed /P2/AC
- net /Player Two Display Bank - Green/AD renamed /P2/AD
- net /Player Two Display Bank - Green/ADP renamed /P2/ADP
- net /Player Two Display Bank - Green/AE renamed /P2/AE
- net /Player Two Display Bank - Green/AF renamed /P2/AF
- net /Player Two Display Bank - Green/AG renamed /P2/AG
- net /Player Two Display Bank - Green/CA1 renamed /P2/CA1
- net /Player Two Display Bank - Green/CA2 renamed /P2/CA2
- net /Player Two Display Bank - Green/CA3 renamed /P2/CA3
- net /Player Two Display Bank - Green/CA4 renamed /P2/CA4
- net /Player Two Display Bank - Green/SA renamed /P2/SA
- net /Player Two Display Bank - Green/SB renamed /P2/SB
- net /Player Two Display Bank - Green/SC renamed /P2/SC
- net /Player Two Display Bank - Green/SD renamed /P2/SD
- net /Player Two Display Bank - Green/SDP renamed /P2/SDP
- net /Player Two Display Bank - Green/SE renamed /P2/SE
- net /Player Two Display Bank - Green/SF renamed /P2/SF
- net /Player Two Display Bank - Green/SG renamed /P2/SG
